File: Motor-Controller-Board_2022_Prototype/Roboteq_Board_V1.1.sch (EAGLE design)
At the start: 53 parts, among them CON1 D-SUB_2-ROW_15-PIN, CON10 TE_4-PIN, CON11 TE_3-PIN, CON12 1X08, CON13 1X08, CON14 1X08, CON15 1X08, CON16 1X08, CON4 1X08, CON5 1X08, CON6 1X08, CON8 1X08, IC1 TLV272, IC2 RS232-TTL_MAX232E, Y1 16MHz

Commit message: Added labels
Parts:
- renumbered CON1 to ROBOTEQ-CON, CON10 to POWER-BYPASS, CON11 to HALL-SENSOR, DEADMAN-SWITCH-IN to DEADMAN-SWITCH
