File: Fuel-Cell-Controller-Board_2022_Prototype/ARCHIVED/Fuel_Cell_Controller_may2022.brd (EAGLE design)
At the start: 203.2 x 163.8 mm, 164 parts, among them J1 BLUETOOTH, Q1 5.8A/30V/35mΩ, U1 MAX232PTH

Commit message: Updates to FCCB
Routing:
- net FC12V: track 452.3 -> 450.4 mm
Changed lines of the file:
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@@
 </element>
 <element name="JP6" library="jumper" library_urn="urn:adsk.eagle:library:252" package="JP1" package3d_urn="urn:adsk.eagle:package:15455/1" value="" x="67.818" y="139.7" smashed="yes" rot="R180">
-<attribute name="NAME" x="69.469" y="142.24" size="1.27" layer="25" ratio="10" rot="R270"/>
+<attribute name="NAME" x="69.469" y="142.367" size="1.27" layer="25" ratio="10" rot="R270"/>
 <attribute name="VALUE" x="64.897" y="142.24" size="1.27" layer="27" ratio="10" rot="R270"/>
 </element>
@@
 <contactref element="R4" pad="1"/>
 <contactref element="U$22" pad="CATHODE"/>
-<contactref element="C9" pad="1"/>
 <contactref element="C13" pad="1"/>
 <contactref element="C12" pad="1"/>
@@
 <wire x1="156.972" y1="117.972" x2="156.972" y2="116.332" width="0.762" layer="1"/>
 <wire x1="154.686" y1="114.438" x2="154.686" y2="116.332" width="0.762" layer="1"/>
-<wire x1="156.972" y1="114.438" x2="156.972" y2="116.332" width="0.762" layer="1"/>
 <contactref element="U$15" pad="S"/>
 <wire x1="151.81" y1="125.73" x2="152.13" y2="125.41" width="0.762" layer="1"/>
@@
 <wire x1="68.758" y1="146.889" x2="62.992" y2="141.123" width="0.762" layer="1"/>
 <wire x1="62.992" y1="141.123" x2="62.992" y2="140.97" width="0.762" layer="1"/>
+<contactref element="C9" pad="1"/>
 <wire x1="77.089" y1="146.685" x2="77.038" y2="146.889" width="0" layer="19" extent="1-1"/>
+<wire x1="156.972" y1="114.438" x2="154.686" y2="114.438" width="0" layer="19" extent="1-1"/>
 </signal>
 <signal name="N$3">
@@
 <wire x1="42.164" y1="134.112" x2="14.351" y2="134.112" width="0.254" layer="1"/>
 <via x="14.351" y="134.112" extent="1-16" drill="0.5"/>
-<wire x1="12.573" y1="135.763" x2="12.573" y2="152.4" width="0.254" layer="16"/>
-<wire x1="12.573" y1="152.4" x2="10.16" y2="152.4" width="0.254" layer="16"/>
+<wire x1="12.446" y1="135.89" x2="12.446" y2="152.4" width="0.254" layer="16"/>
+<wire x1="12.446" y1="152.4" x2="10.16" y2="152.4" width="0.254" layer="16"/>
 <wire x1="10.16" y1="152.4" x2="9.144" y2="153.416" width="0.254" layer="16"/>
 <wire x1="9.144" y1="154.964" x2="10.39" y2="156.21" width="0.254" layer="16"/>
@@
 <wire x1="40.524" y1="119.38" x2="42.164" y2="119.38" width="0.254" layer="16"/>
 <wire x1="62.7218375" y1="80.822125" x2="61.7381625" y2="80.822125" width="0.254" layer="1"/>
-<wire x1="61.7381625" y1="80.822125" x2="61.04259375" y2="80.12655625" width="0.254" layer="1"/>
+<wire x1="61.7381625" y1="80.822125" x2="60.1640375" y2="79.248" width="0.254" layer="1"/>
 <wire x1="64.77" y1="79.634715625" x2="63.909246875" y2="79.634715625" width="0.254" layer="1"/>
-<wire x1="61.04259375" y1="80.12655625" x2="61.04259375" y2="79.83859375" width="0.254" layer="1"/>
 <wire x1="63.909246875" y1="79.634715625" x2="62.7218375" y2="80.822125" width="0.254" layer="1"/>
-<wire x1="61.04259375" y1="79.83859375" x2="60.452" y2="79.248" width="0.254" layer="1"/>
-<wire x1="60.452" y1="79.248" x2="43.18" y2="79.248" width="0.254" layer="1"/>
-<wire x1="14.224" y1="134.112" x2="12.573" y2="135.763" width="0.254" layer="16"/>
+<wire x1="60.1640375" y1="79.248" x2="43.18" y2="79.248" width="0.254" layer="1"/>
+<wire x1="14.224" y1="134.112" x2="12.446" y2="135.89" width="0.254" layer="16"/>
 <wire x1="14.351" y1="134.112" x2="14.224" y2="134.112" width="0.254" layer="16"/>
 </signal>
