File: Fuel-Cell-Controller-Board_2022_Prototype/Fuel_Cell_Controller.sch (EAGLE design)
At the start: 164 parts, among them J1 BLUETOOTH, Q1 5.8A/30V/35mΩ, U1 MAX232PTH

Commit message: Updates to FCCB
Parts:
- removed AUX12VLED, AUX5VLED, FC12VLED, FC5VLED: (no value), led:LEDCHIP-LED0805
- removed AUX_PWR, FC_PWR: TE_6-PIN, EcoCar-Connectors:TE_6-PIN
- removed C1, C2, C27, C3, C4, C5: 1µF, SparkFun-Passives:CAP0805
- removed C10, C11, C12, C13, C25, C26, C9: 10µF, SparkFun-Capacitors:CAP0805
- removed C14, C15: 0.1µF, SparkFun-Passives:CAP0805
- removed C16, C6, C7: 0.1µF, SparkFun-Capacitors:CAP0805
- removed C23, C24, C8: 1µF, SparkFun-Capacitors:CAP0805
- removed D7, D8, D9: (no value), diode:DIODE-DO214AC
- removed J2: (no value), SparkFun-Connectors:CONN_05SCREW
- removed JP5, JP6: (no value), jumper:JP1E
- removed PRESSURE, RELAYBOARD1, RELAYBOARD2, TEMPERATURE: ETHERNET, ETHERNET:ETHERNET
- removed R1, R2, R22, R23, R38: 1kΩ, SparkFun-Passives:RESISTOR0805-RES
- removed R13, R18, R19, R20, R21: 324Ω, SparkFun-Passives:RESISTOR0805-RES
- removed R14, R15, R16, R17, R24, R39, R4, R40, R41, R42, R43, R44, R45, R53, R54, R55, R56, R57, R58, R59, R60, R61: 10kΩ, SparkFun-Passives:RESISTOR0805-RES
- removed R28: 604Ω, resistor:R-US_R0805
- removed R3: 470Ω, SparkFun-Passives:RESISTOR0805-RES
- removed R30, R31: 324Ω, resistor:R-US_R0805
- removed R46, R47, R48, R49, R50, R51, R52: 100kΩ, SparkFun-Passives:RESISTOR0805-RES
- removed U$26: EG4621CT-ND, EG4621CT-ND:EG4621CT-ND
- removed U$27, U$28, U$32: 1µF, 100uF_Cap:CAP-VS-SERIES-PACKAGE-E(ELECT)VS-SERIES-PACKAGE-E
- removed U$29: 10µF, 100uF_Cap:CAP-VS-SERIES-PACKAGE-E(ELECT)VS-SERIES-PACKAGE-E
- removed U$4: H11L1H11L1, FCC_parts:H11L1H11L1
- removed U$7, U$8, U$9: DMP3056L-7DMP3056L-7, FCC_parts:DMP3056L-7DMP3056L-7
- removed U1: MAX232PTH, SparkFun-DigitalIC:MAX232PTH
- removed X1, X2: (no value), con-subd:F09HP
- added AUX_PWR1, FC_PWR1: TE_6-PIN, EcoCar-Connectors:TE_6-PIN
- added C101, C102, C103: 0.1µF, SparkFun-Capacitors:CAP0805
- added C104, C106, C114: 1µF, 100uF_Cap:CAP-VS-SERIES-PACKAGE-E(ELECT)VS-SERIES-PACKAGE-E
- added C105, C113, C115: 1µF, SparkFun-Capacitors:CAP0805
- added C107, C108, C109, C110, C111, C116, C117: 10µF, SparkFun-Capacitors:CAP0805
- added C112: 10µF, 100uF_Cap:CAP-VS-SERIES-PACKAGE-E(ELECT)VS-SERIES-PACKAGE-E
- added C119, C120: 0.1µF, SparkFun-Passives:CAP0805
- added C201: 1µF, SparkFun-Passives:CAP0805
- added D201, D202, D203: (no value), diode:DIODE-DO214AC
- added LED1, LED2, LED3, LED4: (no value), led:LEDCHIP-LED0805
- added PRESSURE1, RELAYBOARD3, RELAYBOARD4, TEMPERATURE1: ETHERNET, ETHERNET:ETHERNET
- added R101, R103, R220: 1kΩ, SparkFun-Passives:RESISTOR0805-RES
- added R102, R104, R105, R106, R107, R108, R109, R110, R112, R113, R114, R115, R205, R206, R207, R208, R209, R210, R211, R212: 10kΩ, SparkFun-Passives:RESISTOR0805-RES
- added R116, R117, R118, R119, R120: 324Ω, SparkFun-Passives:RESISTOR0805-RES
- added R201, R202: 604Ω, resistor:R-US_R0805
- added R203, R204: 324Ω, resistor:R-US_R0805
- added R213, R214, R215, R216, R217, R218, R219: 100kΩ, SparkFun-Passives:RESISTOR0805-RES
- added R221: 470Ω, SparkFun-Passives:RESISTOR0805-RES
- added U$23, U$24: DMP3056L-7DMP3056L-7, FCC_parts:DMP3056L-7DMP3056L-7
- JP1: device jumper:JP2E -> jumper:JP1E
- JP2: device jumper:JP4Q -> jumper:JP1E
- R29: value 604Ω -> 10kΩ; device resistor:R-US_R0805 -> SparkFun-Passives:RESISTOR0805-RES
- U$10: value UMFT234XF -> H11L1H11L1; device FCC_parts:UMFT234XFUMFT234XF -> FCC_parts:H11L1H11L1
- U$19: value ADS1015 -> DMP3056L-7DMP3056L-7; device FCC_parts:ADS1015 -> FCC_parts:DMP3056L-7DMP3056L-7
Connections:
- removed net ADC_A2: J2.4, U$19.A2
- removed net ADC_A3: J2.5, U$19.A3
- removed net ADC_ADDR: JP2.1, JP2.3, JP2.5, JP2.7, U$19.ADDR
- removed net ADC_ALERT: U$1.PD_14(D10/SERIAL8_CTS/PWM4/3), U$19.ALRT
- removed net AUX3V3: SHTSENSOR.VIN, U$30.3.3VO
- removed net BUTTON: R24.2, U$1.PF_2, U$26.P$2
- removed net FROM_FTDI: U$1.PE_7(SERIAL7_RX), U$10.TXD
- removed net FROM_MOTOR: U1.R1IN, X2.2
- removed net I2C4_SCL: JP2.2, U$1.PF_14(D4/I2C4_SCL), U$19.SCL
- removed net I2C4_SDA: JP2.4, U$1.PF_15(D2/I2C4_SDA), U$19.SDA
- removed net MASS_FLOW: R22.1, R23.2, U$19.A0
- removed net MOTOR_RX: U$1.PB_11(SERIAL3_RX/I2C2_SDA/PWM2/4), U1.R1OUT
- removed net MOTOR_TX: U$1.PB_10(SERIAL3_TX/I2C2_SCL/SPI2_SCLK/PWM2/3), U1.T1IN
- removed net N$12: R3.2, U$4.ANODE
- removed net N$15: R22.2, X1.4
- removed net N$21: FC5VLED.A, R28.1
- removed net N$23: FC12VLED.A, R29.1
- removed net N$25: AUX5VLED.A, R30.1
- removed net N$28: AUX12VLED.A, R31.1
- removed net N$8: C5.2, U1.V-
- removed net NUC_3V3: C16.1, C6.1, C7.1, JP1.3, JP2.6, R38.2, R46.1, R47.1, R48.1, R49.1, R50.2, R51.2, R52.2, U$1.3V3, U$18.3.3V, U$19.VDD, U$20.VDD, U$26.P$1, U$27.+
- removed net TO_FTDI: U$1.PE_8(SERIAL7_TX/PWM1/1), U$10.RXD
- removed net TO_MOTOR: U1.T1OUT, X2.3
- removed net VIN: JP3.1, JP5.1, U$1.VIN
- new net FC3V3: C101.1, C102.1, C103.1, C104.+, JP4.1, R213.2, R214.2, R215.2, R216.1, R217.1, R218.1, R219.1, R220.2, SHTSENSOR.VIN, U$18.3.3V, U$20.VDD, U$30.3.3VO
- new net TO_JP3: JP3.2, U$1.5V
- new net TO_JP4: JP4.2, U$1.3V3
- net ALARM_LED: now also R116.1; no longer R13.1
- net AUX12V: now also AUX_PWR1.1, AUX_PWR1.3, C116.1, C117.1, JP1.2, R204.2; no longer AUX_PWR.1, AUX_PWR.3, C25.1, C26.1, JP5.2, R31.2, X1.2
- net AUX5V: now also AUX_PWR1.4, AUX_PWR1.6, C113.1, C114.+, C115.1, JP2.2, R203.2; no longer AUX_PWR.4, AUX_PWR.6, C23.1, C24.1, J1.VCC, JP6.1, R30.2, U$2.RAW, U$30.VIN, U$32.+
- net CAP_CURR: no longer J2.3, U$19.A1
- net CAP_RELAY: now also RELAYBOARD3.3; no longer RELAYBOARD1.3
- net CAP_VOLT: now also RELAYBOARD4.3; no longer RELAYBOARD2.3
- net CHARGE_RELAY: now also RELAYBOARD3.6; no longer RELAYBOARD1.6
- net DEBUG_LED: now also R117.1; no longer R18.1
- net FAN1_PWR: now also D201.C, U$19.DRAIN; no longer D7.C, U$7.DRAIN
- net FAN2_PWR: now also D202.C, U$23.DRAIN; no longer D8.C, U$8.DRAIN
- net FAN3_PWR: now also D203.C, U$24.DRAIN; no longer D9.C, U$9.DRAIN
- net FANS_GATE: now also R29.2, U$10.VO, U$19.GATE, U$23.GATE, U$24.GATE; no longer R4.2, U$4.VO, U$7.GATE, U$8.GATE, U$9.GATE
- net FANS_SWITCH_ALL: now also R221.1; no longer R3.1
- net FC12V: now also C107.1, C108.1, C109.1, C110.1, C111.1, C112.+, FC_PWR1.1, FC_PWR1.3, JP1.1, PRESSURE1.1, R202.2, R29.1, U$1.VIN, U$10.VCC, U$19.SOURCE, U$23.SOURCE, U$24.SOURCE; no longer C10.1, C11.1, C12.1, C13.1, C9.1, FC_PWR.1, FC_PWR.3, JP3.2, PRESSURE.1, R29.2, R4.1, U$29.+, U$4.VCC, U$7.SOURCE, U$8.SOURCE, U$9.SOURCE
- net FC5V: now also C105.1, C106.+, C119.1, C120.1, FC_PWR1.4, FC_PWR1.6, J1.VCC, JP2.1, JP3.1, R101.1, R102.2, R103.1, R104.2, R201.2, U$2.RAW, U$30.VIN; no longer C14.1, C15.1, C3.1, C4.2, C8.1, FC_PWR.4, FC_PWR.6, JP4.1, JP6.2, R1.1, R14.2, R15.2, R2.1, R28.2, U$28.+, U1.VCC
- net FCC_RELAY: now also RELAYBOARD3.2; no longer RELAYBOARD1.2
- net FCTEMP_1: now also R219.2, TEMPERATURE1.1; no longer R46.2, TEMPERATURE.1
- net FCTEMP_2: now also R218.2, TEMPERATURE1.2; no longer R47.2, TEMPERATURE.2
- net FC_VOLT: now also RELAYBOARD4.1; no longer RELAYBOARD2.1
- net GND: now also AUX_PWR1.2, AUX_PWR1.5, C101.2, C102.2, C103.2, C104.-, C105.2, C106.-, C107.2, C108.2, C109.2, C110.2, C111.2, C112.-, C113.2, C114.-, C115.2, C116.2, C117.2, C119.2, C120.2, C201.2, D201.A, D202.A, D203.A, FC_PWR1.2, FC_PWR1.5, LED1.C, LED2.C, LED3.C, LED4.C, PRESSURE1.7, PRESSURE1.8, PRESSURE1.SHD1, PRESSURE1.SHD2, R105.2, R106.2, R107.2, R108.2, R109.2, R110.2, R112.2, R113.2, R114.2, R115.1, R206.1, R208.1, R210.1, R212.1, RELAYBOARD3.7, RELAYBOARD3.8, RELAYBOARD3.SHD1, RELAYBOARD3.SHD2, RELAYBOARD4.8, RELAYBOARD4.SHD1, RELAYBOARD4.SHD2, TEMPERATURE1.8, TEMPERATURE1.SHD1, TEMPERATURE1.SHD2, U$10.CATHODE; no longer AUX12VLED.C, AUX5VLED.C, AUX_PWR.2, AUX_PWR.5, C10.2, C11.2, C12.2, C13.2, C14.2, C15.2, C16.2, C23.2, C24.2, C25.2, C26.2, C27.2, C3.2, C5.1, C6.2, C7.2, C8.2, C9.2, D7.A, D8.A, D9.A, FC12VLED.C, FC5VLED.C, FC_PWR.2, FC_PWR.5, J2.1, JP1.1, JP2.8, PRESSURE.7, PRESSURE.8, PRESSURE.SHD1, PRESSURE.SHD2, R17.1, R23.1, R24.1, R39.1, R41.1, R43.1, R45.1, R53.2, R54.2, R55.2, R56.2, R57.2, R58.2, R59.2, R60.2, R61.2, RELAYBOARD1.7, RELAYBOARD1.8, RELAYBOARD1.SHD1, RELAYBOARD1.SHD2, RELAYBOARD2.8, RELAYBOARD2.SHD1, RELAYBOARD2.SHD2, TEMPERATURE.8, TEMPERATURE.SHD1, TEMPERATURE.SHD2, U$19.GND, U$27.-, U$28.-, U$29.-, U$32.-, U$4.CATHODE, U$4.GND, U1.GND, X1.1, X1.3, X2.5
- net MOTOR_RELAY: now also RELAYBOARD3.4; no longer RELAYBOARD1.4
- net MOTOR_VOLT: now also RELAYBOARD4.2; no longer RELAYBOARD2.2
- net N$1: now also LED1.A, R201.1; no longer JP4.2, U$1.5V
- net N$10: now also R103.2; no longer R2.2
- net N$11: now also R101.2; no longer R1.2
- net N$16: now also R116.2; no longer R13.2
- net N$17: now also R117.2; no longer R18.2
- net N$18: now also R118.2; no longer R19.2
- net N$19: now also R119.2; no longer R20.2
- net N$20: now also R120.2; no longer R21.2
- net N$3: now also LED2.A, R202.1; no longer C1.1, U1.C1+
- net N$4: now also LED3.A, R203.1; no longer C1.2, U1.C1-
- net N$5: now also LED4.A, R204.1; no longer C2.1, U1.C2+
- net N$6: now also RELAYBOARD4.LED2P; no longer C2.2, U1.C2-
- net N$7: now also R221.2, U$10.ANODE; no longer C4.1, U1.V+
- net OE*: now also R102.1, R104.1; no longer R14.1, R15.1
- net PRESSURE_1: now also R205.1, R206.2; no longer R16.1, R17.2
- net PRESSURE_2: now also R207.1, R208.2; no longer R40.1, R41.2
- net PRESSURE_3: now also R209.1, R210.2; no longer R42.1, R43.2
- net PRESSURE_4: now also R211.1, R212.2; no longer R44.1, R45.2
- net RUN_LED: now also R118.1; no longer R19.1
- net SHT_ADR: no longer JP1.2
- net SHUT_LED: now also R119.1; no longer R20.1
- net START_LED: now also R120.1; no longer R21.1
- net START_RELAY: now also RELAYBOARD3.5; no longer RELAYBOARD1.5
- net STOP: now also C201.1, R115.2; no longer C27.1, R39.2
- net TEMP_1: now also R217.2, TEMPERATURE1.3; no longer R48.2, TEMPERATURE.3
- net TEMP_2: now also R216.2, TEMPERATURE1.4; no longer R49.2, TEMPERATURE.4
- net TEMP_3: now also R215.1, TEMPERATURE1.5; no longer R50.1, TEMPERATURE.5
- net TEMP_4: now also R214.1, TEMPERATURE1.6; no longer R51.1, TEMPERATURE.6
- net TEMP_5: now also R213.1, TEMPERATURE1.7; no longer R52.1, TEMPERATURE.7
- net _CAP_CURR: now also RELAYBOARD4.6; no longer RELAYBOARD2.6
- net _CAP_RELAY: now also R106.1; no longer R54.1
- net _CHARGE_RELAY: now also R108.1; no longer R56.1
- net _FCC_RELAY: now also R105.1; no longer R53.1
- net _FC_CURR: now also RELAYBOARD4.4; no longer RELAYBOARD2.4
- net _MOTOR_CURR: now also RELAYBOARD4.5; no longer RELAYBOARD2.5
- net _MOTOR_RELAY: now also R107.1; no longer R55.1
- net _OUTPUT_1: now also R113.1; no longer R60.1
- net _OUTPUT_2: now also R114.1; no longer R61.1
- net _PRESSURE_1: now also PRESSURE1.2, R205.2; no longer PRESSURE.2, R16.2
- net _PRESSURE_2: now also PRESSURE1.3, R207.2; no longer PRESSURE.3, R40.2
- net _PRESSURE_3: now also PRESSURE1.4, R209.2; no longer PRESSURE.4, R42.2
- net _PRESSURE_4: now also PRESSURE1.5, R211.2; no longer PRESSURE.5, R44.2
- net _PURGE_VALVE: now also R112.1; no longer R59.1
- net _START: now also R220.1; no longer R38.1
- net _START_RELAY: now also R109.1; no longer R57.1
- net _SUPPLY_VALVE: now also R110.1; no longer R58.1
Other:
- note added: "JUMPERS"
- note added: "N-MOSFET INVERTER"
- note added: "PULLDOWN RESISTORS"
- note added: "Temperature Sensor Pull Up Resistors"
- note removed: "12-bit Adafruit ADC"
- note removed: "12V to 7V regulator to lighten the load on the nucleo regulator"
- note removed: "A0-A4 are temporarily connected to screw terminals."
- note removed: "A0: Mass Flow Meter"
- note removed: "A1:"
- note removed: "A2:"
- note removed: "A3:"
- note removed: "Can this be NUC3V3?"
- note removed: "DUAL RS232 CONVERTER"
- note removed: "Ethernet I/O"
- note removed: "FTDI CHIP"
- note removed: "Feel free to route to Ethernet connectors or anything else"
- note removed: "Jumpers for selecting power"
- note removed: "Make sure this is a male connector"
- note removed: "N-Mosfet to invert signal"
- note removed: "PUSH BUTTON (ACTIVE HIGH)"
- note removed: "PullDown Resistor's"
- note removed: "RS232 TO MASS FLOW METER"
- note removed: "RS232 TO MOTOR CONTROLLER"
- note removed: "Screw Terminals"

Commit message: Updates to FCC board
Parts:
- removed C17, C18, C19, C20, C21, C22: (no value), SparkFun-Capacitors:CAP0805
- removed H1, H2, H3, H4, H5, H6, H7, H8: MOUNT-PAD-ROUND3.6, holes:MOUNT-PAD-ROUND3.6
- removed J1: BLUETOOTH, FCC_parts:BLUETOOTH
- removed LP_FILTER_OP_AMP: TLV2404TLV2404, FCC_parts:TLV2404TLV2404
- removed R10, R12, R6, R8: 10kΩ, SparkFun-Passives:RESISTOR0805-RES
- removed R11, R5, R7, R9: 470Ω, SparkFun-Passives:RESISTOR0805-RES
- removed R25, R26, R27: (no value), SparkFun-Resistors:RESISTOR0402
- removed R32, R33, R34, R35, R36, R37: (no value), resistor:R-US_R0805
- removed SHTSENSOR: SHT31-DIS, FCC_parts:SHT31-DIS
- removed U$18: DS3231, DS3231:DS3231
- removed U$2: OPENLOG, openlog:OPENLOG
- removed U$20: CD143A-SR3.3CT-ND, 3_3V TVS:CD143A-SR3.3CT-ND
- removed U$21, U$31: 641-1198-1-ND, 5V TVS:641-1198-1-ND
- removed U$22: P6KE15A-E3/54GICT-ND, 12V TVS:P6KE15A-E3/54GICT-ND
- removed U$30: ADAFRUITOLED, FCC_parts:ADAFRUITOLED
- added C301, C302, C303, C304, C305, C306: (no value), SparkFun-Capacitors:CAP0805
- added D301, D302: 641-1198-1-ND, 5V TVS:641-1198-1-ND
- added D303: P6KE15A-E3/54GICT-ND, 12V TVS:P6KE15A-E3/54GICT-ND
- added H10, H11, H12, H13, H14, H15, H16, H9: MOUNT-PAD-ROUND3.6, holes:MOUNT-PAD-ROUND3.6
- added J2: BLUETOOTH, FCC_parts:BLUETOOTH
- added LP_FILTER_OP_AMP1: TLV2404TLV2404, FCC_parts:TLV2404TLV2404
- added R301, R302, R305, R306: 470Ω, SparkFun-Passives:RESISTOR0805-RES
- added R303, R304, R307, R308: 10kΩ, SparkFun-Passives:RESISTOR0805-RES
- added R309, R310, R311, R312, R313, R314: (no value), resistor:R-US_R0805
- added R315, R316, R317: (no value), SparkFun-Resistors:RESISTOR0402
- added SHTSENSOR1: SHT31-DIS, FCC_parts:SHT31-DIS
- added U$27: ADAFRUITOLED, FCC_parts:ADAFRUITOLED
- added U$4: OPENLOG, openlog:OPENLOG
- added U$7: DS3231, DS3231:DS3231
- added U$8: CD143A-SR3.3CT-ND, 3_3V TVS:CD143A-SR3.3CT-ND
Connections:
- removed net N$24: LP_FILTER_OP_AMP.1IN-, LP_FILTER_OP_AMP.1OUT, R25.2
- removed net N$26: LP_FILTER_OP_AMP.2IN-, LP_FILTER_OP_AMP.2OUT, R26.2
- removed net N$27: LP_FILTER_OP_AMP.3IN-, LP_FILTER_OP_AMP.3OUT, R27.1
- new net N$12: LP_FILTER_OP_AMP1.2IN-, LP_FILTER_OP_AMP1.2OUT, R316.2
- new net N$15: LP_FILTER_OP_AMP1.3IN-, LP_FILTER_OP_AMP1.3OUT, R317.1
- new net N$8: LP_FILTER_OP_AMP1.1IN-, LP_FILTER_OP_AMP1.1OUT, R315.2
- net AUX12V: now also R307.1; no longer R6.1
- net AUX5V: now also D302.C; no longer U$31.C
- net CAP_CURR: now also C303.1, R313.2, R314.1; no longer C17.1, R36.2, R37.1
- net CAP_VOLT: now also LP_FILTER_OP_AMP1.3IN+; no longer LP_FILTER_OP_AMP.3IN+
- net FC12V: now also D303.C, R303.1, R304.1, R308.1; no longer R10.1, R12.1, R8.1, U$22.C
- net FC3V3: now also SHTSENSOR1.VIN, U$27.3.3VO, U$7.3.3V, U$8.VDD; no longer SHTSENSOR.VIN, U$18.3.3V, U$20.VDD, U$30.3.3VO
- net FC5V: now also D301.C, J2.VCC, LP_FILTER_OP_AMP1.VCC, U$27.VIN, U$4.RAW; no longer J1.VCC, LP_FILTER_OP_AMP.VCC, U$2.RAW, U$21.C, U$30.VIN
- net FC_CURR: now also C301.1, R309.2, R310.1; no longer C19.1, R32.2, R33.1
- net FC_VOLT: now also LP_FILTER_OP_AMP1.1IN+; no longer LP_FILTER_OP_AMP.1IN+
- net FROM_BLUE: now also J2.TXO; no longer J1.TXO
- net FROM_OPEN: now also U$4.TXO; no longer U$2.TXO
- net GND: now also C301.2, C302.2, C303.2, C304.2, C305.2, C306.2, D301.A, D302.A, D303.A, H10.MOUNT, H11.MOUNT, H12.MOUNT, H13.MOUNT, H14.MOUNT, H15.MOUNT, H16.MOUNT, H9.MOUNT, J2.GND, LP_FILTER_OP_AMP1.4IN+, LP_FILTER_OP_AMP1.4IN-, LP_FILTER_OP_AMP1.GND, R310.2, R312.2, R314.2, SHTSENSOR1.GND, U$27.GND, U$4.GND, U$4.GND2, U$7.GND, U$8.GND; no longer C17.2, C18.2, C19.2, C20.2, C21.2, C22.2, H1.MOUNT, H2.MOUNT, H3.MOUNT, H4.MOUNT, H5.MOUNT, H6.MOUNT, H7.MOUNT, H8.MOUNT, J1.GND, LP_FILTER_OP_AMP.4IN+, LP_FILTER_OP_AMP.4IN-, LP_FILTER_OP_AMP.GND, R33.2, R35.2, R37.2, SHTSENSOR.GND, U$18.GND, U$2.GND, U$2.GND2, U$20.GND, U$21.A, U$22.A, U$30.GND, U$31.A
- net HUMID_RST: now also SHTSENSOR1.RST; no longer SHTSENSOR.RST
- net I2C1_SCL: now also SHTSENSOR1.SCL, U$7.SCL; no longer SHTSENSOR.SCL, U$18.SCL
- net I2C1_SDA: now also SHTSENSOR1.SDA, U$7.SDA; no longer SHTSENSOR.SDA, U$18.SDA
- net MOTOR_CURR: now also C302.1, R311.2, R312.1; no longer C18.1, R34.2, R35.1
- net MOTOR_VOLT: now also LP_FILTER_OP_AMP1.2IN+; no longer LP_FILTER_OP_AMP.2IN+
- net N$13: now also R302.2; no longer R9.2
- net N$14: now also R306.2; no longer R11.2
- net N$2: now also R305.2; no longer R5.2
- net N$9: now also R301.2; no longer R7.2
- net OLED_CLK: now also U$27.CLK; no longer U$30.CLK
- net OLED_MISO: now also U$27.DC; no longer U$30.DC
- net OLED_MOSI: now also U$27.DATA; no longer U$30.DATA
- net OLED_SEL: now also U$27.CS; no longer U$30.CS
- net OPEN_RST: now also U$4.DTR; no longer U$2.DTR
- net OUTPUT_1: now also R302.1; no longer R9.1
- net OUTPUT_1_GATE: now also R304.2; no longer R10.2
- net OUTPUT_2: now also R306.1; no longer R11.1
- net OUTPUT_2_GATE: now also R308.2; no longer R12.2
- net PURGE_VALVE: now also R301.1; no longer R7.1
- net PURGE_VALVE_GATE: now also R303.2; no longer R8.2
- net SHT31_ALERT: now also SHTSENSOR1.ALR; no longer SHTSENSOR.ALR, U$1.PD_15(D9/SERIAL8_RTS/PWM4/4)
- net SHT_ADR: now also SHTSENSOR1.ADR; no longer SHTSENSOR.ADR
- net SUPPLY_VALVE: now also R305.1; no longer R5.1
- net SUPPLY_VALVE_GATE: now also R307.2; no longer R6.2
- net TO_BLUE: now also J2.RXI; no longer J1.RXI
- net TO_OPEN: now also U$4.RXI; no longer U$2.RXI
- net _CAP_CURR: now also R313.1; no longer R36.1
- net _CAP_VOLT: now also C306.1, R317.2; no longer C22.1, R27.2
- net _FC_CURR: now also R309.1; no longer R32.1
- net _FC_VOLT: now also C304.1, R315.1; no longer C20.1, R25.1
- net _MOTOR_CURR: now also R311.1; no longer R34.1
- net _MOTOR_VOLT: now also C305.1, R316.1; no longer C21.1, R26.1
Other:
- note removed: "ALARM"
- note removed: "DEBUG"
- note removed: "Double check these"
- note removed: "RUN"
- note removed: "SHUTDOWN"
- note removed: "STARTUP"
