File: Fuel-Cell-Controller-Board_2022_Prototype/Prototype_FCC_Board_82022.sch (EAGLE design)
At the start: 152 parts, among them IC1 MAX232ECWE, IC2 TLV2404IN, IC3 TLV2404IN, J2 BLUETOOTH, Q1 5.8A/30V/35mΩ

Commit message: update
Parts:
- added JP5: (no value), adafruit:PINHD-1X8CLEANBIG
- C301, C302, C303, C304, C305, C306: value (none) -> 47uF
- R309, R312, R314: value (none) -> 145Ω
- R310, R311, R313: value (none) -> 75Ω
- R315, R316, R317: value (none) -> 220Ω; device SparkFun-Resistors:RESISTOR0402 -> resistor:R-US_R0805
- renumbered D3 to D307, D4 to D306, D5 to D305, D6 to D304
Connections:
- removed net N$12: IC3.3IN-, IC3.3OUT
- new net N$25: C301.2, IC3.1IN+, R309.2, R310.2
- net CAP_CURR: now also IC3.3IN-, IC3.3OUT; no longer C303.1, IC3.3IN+, R313.1, R314.1
- net FC_CURR: now also IC3.1IN-, IC3.1OUT; no longer C301.2, IC3.1IN+, R309.2, R310.2
- net GND: now also R314.2; no longer R313.2
- net MOTOR_CURR: now also IC3.2IN-, IC3.2OUT; no longer C302.2, IC3.2IN+, R311.2, R312.2
- net N$15: now also C303.1, IC3.3IN+, R313.1, R314.1; no longer IC3.2IN-, IC3.2OUT
- net N$8: now also C302.2, IC3.2IN+, R311.2, R312.2; no longer IC3.1IN-, IC3.1OUT
- net _CAP_CURR: now also R313.2; no longer R314.2
Other:
- moved on the sheet: C304, C305, C306, IC2, R313, R314, R315, R316, R317

Commit message: update
Connections:
- new net N$28: JP5.3
- new net N$30: JP5.4
- new net N$31: JP5.5
- net FC3V3: now also JP5.6
- net FC5V: now also JP5.7
- net GND: now also JP5.8
- net I2C1_SCL: now also JP5.2
- net I2C1_SDA: now also JP5.1
- net RX_RS232: now also CAN.3; no longer CAN.6
- net TX_RS232: now also CAN.6; no longer CAN.3
Other:
- note added: "128x64 OLED Display"
- note added: "X"
- moved on the sheet: JP5
Changed lines of the file:
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@@
 <text x="261.62" y="109.22" size="3.81" layer="94">PULLUP RESISTORS</text>
 <text x="261.62" y="63.5" size="3.81" layer="94">LINEAR REGULATOR</text>
+<text x="360.68" y="76.2" size="1.778" layer="91" align="center">X</text>
+<text x="360.68" y="71.12" size="1.778" layer="91" align="center">X</text>
+<text x="391.16" y="71.12" size="1.778" layer="91" align="center">X</text>
+<text x="391.16" y="76.2" size="1.778" layer="91" align="center">X</text>
+<text x="63.5" y="248.92" size="1.778" layer="91" align="center">X</text>
+<text x="63.5" y="256.54" size="1.778" layer="91" align="center">X</text>
+<text x="63.5" y="259.08" size="1.778" layer="91" align="center">X</text>
+<text x="63.5" y="238.76" size="1.778" layer="91" align="center">X</text>
+<text x="63.5" y="236.22" size="1.778" layer="91" align="center">X</text>
+<text x="205.74" y="251.46" size="1.778" layer="91" align="center">X</text>
+<text x="205.74" y="248.92" size="1.778" layer="91" align="center">X</text>
+<text x="205.74" y="238.76" size="1.778" layer="91" align="center">X</text>
+<text x="205.74" y="236.22" size="1.778" layer="91" align="center">X</text>
+<text x="205.74" y="233.68" size="1.778" layer="91" align="center">X</text>
+<text x="205.74" y="231.14" size="1.778" layer="91" align="center">X</text>
+<text x="205.74" y="228.6" size="1.778" layer="91" align="center">X</text>
+<text x="205.74" y="223.52" size="1.778" layer="91" align="center">X</text>
+<text x="205.74" y="220.98" size="1.778" layer="91" align="center">X</text>
+<text x="205.74" y="215.9" size="1.778" layer="91" align="center">X</text>
+<text x="205.74" y="213.36" size="1.778" layer="91" align="center">X</text>
+<text x="205.74" y="210.82" size="1.778" layer="91" align="center">X</text>
+<text x="205.74" y="203.2" size="1.778" layer="91" align="center">X</text>
+<text x="205.74" y="200.66" size="1.778" layer="91" align="center">X</text>
+<text x="205.74" y="193.04" size="1.778" layer="91" align="center">X</text>
+<text x="205.74" y="187.96" size="1.778" layer="91" align="center">X</text>
+<text x="205.74" y="182.88" size="1.778" layer="91" align="center">X</text>
+<text x="205.74" y="160.02" size="1.778" layer="91" align="center">X</text>
+<text x="205.74" y="157.48" size="1.778" layer="91" align="center">X</text>
+<text x="205.74" y="154.94" size="1.778" layer="91" align="center">X</text>
+<text x="205.74" y="132.08" size="1.778" layer="91" align="center">X</text>
+<text x="205.74" y="129.54" size="1.778" layer="91" align="center">X</text>
 </plain>
 <instances>
@@
 <net name="TX_RS232" class="0">
 <segment>
-<pinref part="CAN" gate="G$1" pin="3"/>
-<wire x1="401.32" y1="246.38" x2="391.16" y2="246.38" width="0.1524" layer="91"/>
-<label x="391.16" y="246.38" size="1.778" layer="95" rot="R180" xref="yes"/>
+<pinref part="CAN" gate="G$1" pin="6"/>
+<wire x1="401.32" y1="238.76" x2="388.62" y2="238.76" width="0.1524" layer="91"/>
+<label x="388.62" y="238.76" size="1.778" layer="95" rot="R180" xref="yes"/>
 </segment>
 </net>
 <net name="RX_RS232" class="0">
 <segment>
-<pinref part="CAN" gate="G$1" pin="6"/>
-<wire x1="401.32" y1="238.76" x2="391.16" y2="238.76" width="0.1524" layer="91"/>
-<label x="391.16" y="238.76" size="1.778" layer="95" rot="R180" xref="yes"/>
+<pinref part="CAN" gate="G$1" pin="3"/>
+<wire x1="401.32" y1="246.38" x2="388.62" y2="246.38" width="0.1524" layer="91"/>
+<label x="388.62" y="246.38" size="1.778" layer="95" rot="R180" xref="yes"/>
 </segment>
 </net>
@@
 <text x="129.54" y="187.96" size="3.81" layer="94">Valve Cntrl</text>
 <text x="20.32" y="187.96" size="3.81" layer="94">Valve Cntrl</text>
+<text x="320.04" y="190.5" size="3.81" layer="94">128x64 OLED Display</text>
+<text x="337.82" y="175.26" size="1.778" layer="91" align="center">X</text>
+<text x="337.82" y="172.72" size="1.778" layer="91" align="center">X</text>
+<text x="337.82" y="170.18" size="1.778" layer="91" align="center">X</text>
+<text x="347.98" y="218.44" size="1.778" layer="91" align="center">X</text>
+<text x="43.18" y="109.22" size="1.778" layer="91" align="center">X</text>
+<text x="25.4" y="83.82" size="1.778" layer="91" align="center">X</text>
+<text x="208.28" y="88.9" size="1.778" layer="91" align="center">X</text>
+<text x="208.28" y="91.44" size="1.778" layer="91" align="center">X</text>
+<text x="208.28" y="93.98" size="1.778" layer="91" align="center">X</text>
+<text x="353.06" y="91.44" size="1.778" layer="91" align="center">X</text>
+<text x="353.06" y="93.98" size="1.778" layer="91" align="center">X</text>
+<text x="353.06" y="96.52" size="1.778" layer="91" align="center">X</text>
+<text x="269.24" y="180.34" size="1.778" layer="91" align="center">X</text>
+<text x="269.24" y="170.18" size="1.778" layer="91" align="center">X</text>
 </plain>
 <instances>
@@
 <attribute name="VALUE" x="367.03" y="80.518" size="1.778" layer="96"/>
 </instance>
-<instance part="JP5" gate="G$1" x="360.68" y="180.34" smashed="yes">
-<attribute name="NAME" x="354.33" y="191.135" size="1.778" layer="95"/>
-<attribute name="VALUE" x="354.33" y="165.1" size="1.778" layer="96"/>
+<instance part="JP5" gate="G$1" x="325.12" y="172.72" smashed="yes" rot="R180">
+<attribute name="NAME" x="331.47" y="161.925" size="1.778" layer="95" rot="R180"/>
+<attribute name="VALUE" x="331.47" y="187.96" size="1.778" layer="96" rot="R180"/>
 </instance>
 </instances>
@@
 <pinref part="R314" gate="G$1" pin="2"/>
 </segment>
+<segment>
+<pinref part="JP5" gate="G$1" pin="8"/>
+<wire x1="327.66" y1="182.88" x2="337.82" y2="182.88" width="0.1524" layer="91"/>
+<label x="337.82" y="182.88" size="1.778" layer="95"/>
+</segment>
 </net>
 <net name="FC12V" class="0">
@@
 <junction x="340.36" y="248.92"/>
 </segment>
+<segment>
+<pinref part="JP5" gate="G$1" pin="6"/>
+<wire x1="327.66" y1="177.8" x2="337.82" y2="177.8" width="0.1524" layer="91"/>
+<label x="337.82" y="177.8" size="1.778" layer="95"/>
+</segment>
 </net>
 <net name="OPEN_RST" class="0">
@@
 <label x="330.2" y="238.76" size="1.778" layer="95" rot="R180" xref="yes"/>
 </segment>
+<segment>
+<pinref part="JP5" gate="G$1" pin="2"/>
+<wire x1="327.66" y1="167.64" x2="337.82" y2="167.64" width="0.1524" layer="91"/>
+<label x="337.82" y="167.64" size="1.778" layer="95" xref="yes"/>
+</segment>
 </net>
 <net name="I2C1_SDA" class="0">
@@
 <label x="330.2" y="233.68" size="1.778" layer="95" rot="R180" xref="yes"/>
 </segment>
+<segment>
+<pinref part="JP5" gate="G$1" pin="1"/>
+<wire x1="327.66" y1="165.1" x2="358.14" y2="165.1" width="0.1524" layer="91"/>
+<label x="358.14" y="165.1" size="1.778" layer="95" xref="yes"/>
+</segment>
 </net>
 <net name="AUX5V" class="0">
@@
 <label x="175.26" y="106.68" size="1.778" layer="95"/>
 </segment>
+<segment>
+<pinref part="JP5" gate="G$1" pin="7"/>
+<wire x1="327.66" y1="180.34" x2="337.82" y2="180.34" width="0.1524" layer="91"/>
+<label x="337.82" y="180.34" size="1.778" layer="95"/>
+</segment>
 </net>
 <net name="_FC_CURR" class="0">
@@
 </segment>
 </net>
+<net name="N$28" class="0">
+<segment>
+<pinref part="JP5" gate="G$1" pin="3"/>
+<wire x1="327.66" y1="170.18" x2="337.82" y2="170.18" width="0.1524" layer="91"/>
+</segment>
+</net>
+<net name="N$30" class="0">
+<segment>
+<pinref part="JP5" gate="G$1" pin="4"/>
+<wire x1="327.66" y1="172.72" x2="337.82" y2="172.72" width="0.1524" layer="91"/>
+<wire x1="327.66" y1="172.72" x2="337.82" y2="172.72" width="0.1524" layer="91"/>
+</segment>
+</net>
+<net name="N$31" class="0">
+<segment>
+<pinref part="JP5" gate="G$1" pin="5"/>
+<wire x1="327.66" y1="175.26" x2="337.82" y2="175.26" width="0.1524" layer="91"/>
+</segment>
+</net>

Commit message: update
Parts:
- removed C201: 1µF, SparkFun-Passives:CAP0805
- removed H2_SENSOR: ETHERNET, ETHERNET:ETHERNET
- removed Q1: 5.8A/30V/35mΩ, n-mos switch:MOSFET-NCH-AO3404A
- removed R101, R103: 1kΩ, SparkFun-Passives:RESISTOR0805-RES
- removed R102, R104, R115: 10kΩ, SparkFun-Passives:RESISTOR0805-RES
- added J1: RJ45_LED, EcoCar-Connectors:RJ45_LED
Connections:
- removed net N$10: R103.2, U$3.DIR
- removed net N$11: R101.2, U$5.DIR
- removed net OE*: Q1.D, R102.1, R104.1, U$3.OE*, U$5.OE*
- removed net STOP: C201.1, H2_SENSOR.1, Q1.G, R115.2, U$1.PB_5(CAN2_RD/SPI1_MOSI/PWM3/2)
- new net NEW_BLUE_BUTTON: U$1.PF_13(D7)
- net ESTOP_1: now also J1.3; no longer H2_SENSOR.3
- net ESTOP_2: now also J1.4; no longer H2_SENSOR.4
- net FC3V3: now also R121.2, R122.2
- net FC5V: now also U$3.DIR, U$5.DIR; no longer R101.1, R102.2, R103.1, R104.2, R121.2, R122.2
- net GND: now also J1.5, J1.6, J1.7, J1.8, U$3.OE*, U$5.A6, U$5.A7, U$5.A8, U$5.B6, U$5.B7, U$5.B8, U$5.OE*; no longer C201.2, H2_SENSOR.5, H2_SENSOR.6, H2_SENSOR.7, H2_SENSOR.8, H2_SENSOR.SHD1, H2_SENSOR.SHD2, Q1.S, R115.1
- net H2_OK: now also J1.2; no longer H2_SENSOR.2
Other:
- note removed: "N-MOSFET INVERTER"
- moved on the sheet: C101, C102, C103, C104, C105, C106, C107, C108, C109, C110, C111, C112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

Commit message: update
Parts:
- removed CAN, FANS_1, FANS_2, PRESSURE1, RELAYBOARD3, RELAYBOARD4, TEMPERATURE1, VALVES: ETHERNET, ETHERNET:ETHERNET
- added J10, J3, J4, J5, J6, J7, J8, J9: RJ45_LED, EcoCar-Connectors:RJ45_LED
Connections:
- removed net _START: U$1.PF_12(D8)
- net CAP_RELAY: now also J8.3; no longer RELAYBOARD3.3
- net CAP_VOLT: now also J9.3; no longer RELAYBOARD4.3
- net CHARGE_RELAY: now also J8.6; no longer RELAYBOARD3.6
- net FAN1_PWR: now also J3.1; no longer FANS_1.1
- net FAN2_PWR: now also J3.4; no longer FANS_1.4
- net FAN3_PWR: now also J4.1; no longer FANS_2.1
- net FC12V: now also J5.1; no longer PRESSURE1.1
- net FCC_RELAY: now also J8.2; no longer RELAYBOARD3.2
- net FCTEMP_1: now also J6.1; no longer TEMPERATURE1.1
- net FCTEMP_2: now also J6.2; no longer TEMPERATURE1.2
- net FC_VOLT: now also J9.1; no longer RELAYBOARD4.1
- net GND: now also J1.SHIELD, J10.2, J10.4, J10.6, J10.8, J10.SHIELD, J3.7, J3.8, J3.SHIELD, J4.6, J4.7, J4.8, J4.SHIELD, J5.7, J5.8, J5.SHIELD, J6.8, J6.SHIELD, J7.4, J7.5, J7.SHIELD, J8.7, J8.8, J8.SHIELD, J9.8, J9.SHIELD; no longer CAN.4, CAN.5, CAN.SHD1, CAN.SHD2, FANS_1.7, FANS_1.8, FANS_1.SHD1, FANS_1.SHD2, FANS_2.6, FANS_2.7, FANS_2.8, FANS_2.SHD1, FANS_2.SHD2, PRESSURE1.7, PRESSURE1.8, PRESSURE1.SHD1, PRESSURE1.SHD2, RELAYBOARD3.7, RELAYBOARD3.8, RELAYBOARD3.SHD1, RELAYBOARD3.SHD2, RELAYBOARD4.8, RELAYBOARD4.SHD1, RELAYBOARD4.SHD2, TEMPERATURE1.8, TEMPERATURE1.SHD1, TEMPERATURE1.SHD2, VALVES.2, VALVES.4, VALVES.6, VALVES.8, VALVES.SHD1, VALVES.SHD2
- net MOTOR_RELAY: now also J8.4; no longer RELAYBOARD3.4
- net MOTOR_VOLT: now also J9.2; no longer RELAYBOARD4.2
- net N$6: now also J9.LED1N; no longer RELAYBOARD4.LED2P
- net OUTPUT_1_ENET: now also J10.5; no longer VALVES.5
- net OUTPUT_2_ENET: now also J10.7; no longer VALVES.7
- net PURGE_VALVE_ENET: now also J10.3; no longer VALVES.3
- net PWM_1: now also J3.3; no longer FANS_1.3
- net PWM_2: now also J3.6; no longer FANS_1.6
- net PWM_3: now also J4.3; no longer FANS_2.3
- net RX_RS232: now also J7.3; no longer CAN.3
- net START_RELAY: now also J8.5; no longer RELAYBOARD3.5
- net SUPPLY_VALVE_ENET: now also J10.1; no longer VALVES.1
- net TACH_1: now also J3.2; no longer FANS_1.2
- net TACH_2: now also J3.5; no longer FANS_1.5
- net TACH_3: now also J4.2; no longer FANS_2.2
- net TEMP_1: now also J6.3; no longer TEMPERATURE1.3
- net TEMP_2: now also J6.4; no longer TEMPERATURE1.4
- net TEMP_3: now also J6.5; no longer TEMPERATURE1.5
- net TEMP_4: now also J6.6; no longer TEMPERATURE1.6
- net TEMP_5: now also J6.7; no longer TEMPERATURE1.7
- net TX_RS232: now also J7.6; no longer CAN.6
- net _CAP_CURR: now also J9.6; no longer RELAYBOARD4.6
- net _FC_CURR: now also J9.4; no longer RELAYBOARD4.4
- net _MOTOR_CURR: now also J9.5; no longer RELAYBOARD4.5
- net _PRESSURE_1: now also J5.2; no longer PRESSURE1.2
- net _PRESSURE_2: now also J5.3; no longer PRESSURE1.3
- net _PRESSURE_3: now also J5.4; no longer PRESSURE1.4
- net _PRESSURE_4: now also J5.5; no longer PRESSURE1.5
Other:
- moved on the sheet: R105, R106, R107, R108, R109, R110, R112, R113, R114

Commit message: update
Parts:
- removed U$8: CD143A-SR3.3CT-ND, 3_3V TVS:CD143A-SR3.3CT-ND
- added D308: P6KE15A-E3/54GICT-ND, 12V TVS:P6KE15A-E3/54GICT-ND
- added R123, R124: 4.7kΩ, SparkFun-Passives:RESISTOR0805-RES
Connections:
- net AUX12V: now also D308.C
- net FC3V3: now also R123.1, R124.2, U$3.DIR, U$3.VCC, U$5.DIR, U$5.VCC; no longer U$8.VDD
- net FC5V: no longer U$3.DIR, U$3.VCC, U$5.DIR, U$5.VCC
- net GND: now also D308.A, R123.2, R124.1; no longer U$8.GND
Other:
- note removed: "NC"
- moved on the sheet: D301, D302, D303

Commit message: update
Parts:
- R116, R119: value 324Ω -> 65Ω
- R118, R120: value 324Ω -> 10Ω
Changed lines of the file:
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@@
 <part name="R308" library="SparkFun-Passives" deviceset="RESISTOR" device="0805-RES" value="10kΩ"/>
 <part name="D1" library="SparkFun-LED" library_urn="urn:adsk.eagle:library:529" deviceset="LED" device="1206" package3d_urn="urn:adsk.eagle:package:39352/1" value="RED"/>
-<part name="R116" library="SparkFun-Passives" deviceset="RESISTOR" device="0805-RES" value="324Ω"/>
+<part name="R116" library="SparkFun-Passives" deviceset="RESISTOR" device="0805-RES" value="65Ω"/>
 <part name="C102" library="SparkFun-Capacitors" library_urn="urn:adsk.eagle:library:510" deviceset="CAP" device="0805" value="0.1µF"/>
 <part name="C105" library="SparkFun-Capacitors" library_urn="urn:adsk.eagle:library:510" deviceset="CAP" device="0805" value="1µF"/>
@@
 <part name="U$25" library="FCC_parts" deviceset="5060BRG4" device="5060BRG4"/>
 <part name="GND5" library="E-P-008-R1.2" deviceset="GND" device=""/>
-<part name="R118" library="SparkFun-Passives" deviceset="RESISTOR" device="0805-RES" value="324Ω"/>
-<part name="R119" library="SparkFun-Passives" deviceset="RESISTOR" device="0805-RES" value="324Ω"/>
-<part name="R120" library="SparkFun-Passives" deviceset="RESISTOR" device="0805-RES" value="324Ω"/>
+<part name="R118" library="SparkFun-Passives" deviceset="RESISTOR" device="0805-RES" value="10Ω"/>
+<part name="R119" library="SparkFun-Passives" deviceset="RESISTOR" device="0805-RES" value="65Ω"/>
+<part name="R120" library="SparkFun-Passives" deviceset="RESISTOR" device="0805-RES" value="10Ω"/>
 <part name="C103" library="SparkFun-Capacitors" library_urn="urn:adsk.eagle:library:510" deviceset="CAP" device="0805" value="0.1µF"/>
 <part name="C101" library="SparkFun-Capacitors" library_urn="urn:adsk.eagle:library:510" deviceset="CAP" device="0805" value="0.1µF"/>

Commit message: new resistor
Parts:
- added R1: 145Ω, resistor:R-US_R0805
Changed lines of the file:
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@@
 <part name="GND26" library="E-P-008-R1.2" deviceset="GND" device=""/>
 <part name="D308" library="12V TVS" deviceset="P6KE15A-E3/54GICT-ND" device=""/>
+<part name="R1" library="resistor" library_urn="urn:adsk.eagle:library:348" deviceset="R-US_" device="R0805" package3d_urn="urn:adsk.eagle:package:26059/1" value="145Ω"/>
 </parts>
 <sheets>
@@
 <attribute name="VALUE" x="63.4746" y="81.8642" size="1.778" layer="96"/>
 </instance>
+<instance part="R1" gate="G$1" x="157.48" y="48.26" smashed="yes">
+<attribute name="NAME" x="153.67" y="49.7586" size="1.778" layer="95"/>
+<attribute name="VALUE" x="153.67" y="44.958" size="1.778" layer="96"/>
+</instance>
 </instances>

Commit message: update
Parts:
- removed R1: 145Ω, resistor:R-US_R0805
Changed lines of the file:
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@@
 <part name="GND26" library="E-P-008-R1.2" deviceset="GND" device=""/>
 <part name="D308" library="12V TVS" deviceset="P6KE15A-E3/54GICT-ND" device=""/>
-<part name="R1" library="resistor" library_urn="urn:adsk.eagle:library:348" deviceset="R-US_" device="R0805" package3d_urn="urn:adsk.eagle:package:26059/1" value="145Ω"/>
 </parts>
 <sheets>
@@
 <attribute name="VALUE" x="63.4746" y="81.8642" size="1.778" layer="96"/>
 </instance>
-<instance part="R1" gate="G$1" x="157.48" y="48.26" smashed="yes">
-<attribute name="NAME" x="153.67" y="49.7586" size="1.778" layer="95"/>
-<attribute name="VALUE" x="153.67" y="44.958" size="1.778" layer="96"/>
-</instance>
 </instances>
