File: Fuel-Cell-Controller-Board_2022_Prototype/Prototype_FCC_Board_82022.brd (EAGLE design)
At the start: 160 x 100 mm, 153 parts, among them IC1 MAX232ECWE, IC2 TLV2404IN, IC3 TLV2404IN, J2 BLUETOOTH, Q1 5.8A/30V/35mΩ

Commit message: update
Parts:
- removed C201: 1µF, SparkFun-Passives:0805
- removed H2_SENSOR: ETHERNET, ETHERNET:A122645-ND
- removed Q1: 5.8A/30V/35mΩ, n-mos switch:SOT23-3
- removed R101, R103: 1kΩ, SparkFun-Passives:0805
- removed R102, R104, R115: 10kΩ, SparkFun-Passives:0805
- added J1: RJ45_LED, EcoCar-Connectors:RJ45_LED
Connections:
- removed net N$10: R103.2, U$3.1
- removed net N$11: R101.2, U$5.1
- removed net OE*: Q1.3, R102.1, R104.1, U$3.19, U$5.19
- removed net STOP: C201.1, H2_SENSOR.P$1, Q1.1, R115.2, U$1.PB_5
- new net NEW_BLUE_BUTTON: U$1.PF_13
- net ESTOP_1: now also J1.3; no longer H2_SENSOR.P$3
- net ESTOP_2: now also J1.4; no longer H2_SENSOR.P$4
- net FC3V3: now also R121.2, R122.2
- net FC5V: now also U$3.1, U$5.1; no longer R101.1, R102.2, R103.1, R104.2, R121.2, R122.2
- net GND: now also J1.5, J1.6, J1.7, J1.8, U$3.19, U$5.11, U$5.12, U$5.13, U$5.19, U$5.7, U$5.8, U$5.9; no longer C201.2, H2_SENSOR.P$13, H2_SENSOR.P$14, H2_SENSOR.P$5, H2_SENSOR.P$6, H2_SENSOR.P$7, H2_SENSOR.P$8, Q1.2, R115.1
- net H2_OK: now also J1.2; no longer H2_SENSOR.P$2

Commit message: update
Parts:
- removed CAN, FANS_1, FANS_2, PRESSURE1, RELAYBOARD3, RELAYBOARD4, TEMPERATURE1, VALVES: ETHERNET, ETHERNET:A122645-ND
- added J10, J3, J4, J5, J6, J7, J8, J9: RJ45_LED, EcoCar-Connectors:RJ45_LED
Connections:
- removed net _START: U$1.PF_12
- net CAP_RELAY: now also J8.3; no longer RELAYBOARD3.P$3
- net CAP_VOLT: now also J9.3; no longer RELAYBOARD4.P$3
- net CHARGE_RELAY: now also J8.6; no longer RELAYBOARD3.P$6
- net FAN1_PWR: now also J3.1; no longer FANS_1.P$1
- net FAN2_PWR: now also J3.4; no longer FANS_1.P$4
- net FAN3_PWR: now also J4.1; no longer FANS_2.P$1
- net FC12V: now also J5.1; no longer PRESSURE1.P$1
- net FCC_RELAY: now also J8.2; no longer RELAYBOARD3.P$2
- net FCTEMP_1: now also J6.1; no longer TEMPERATURE1.P$1
- net FCTEMP_2: now also J6.2; no longer TEMPERATURE1.P$2
- net FC_VOLT: now also J9.1; no longer RELAYBOARD4.P$1
- net GND: now also J1.S1, J1.S2, J10.2, J10.4, J10.6, J10.8, J10.S1, J10.S2, J3.7, J3.8, J3.S1, J3.S2, J4.6, J4.7, J4.8, J4.S1, J4.S2, J5.7, J5.8, J5.S1, J5.S2, J6.8, J6.S1, J6.S2, J7.4, J7.5, J7.S1, J7.S2, J8.7, J8.8, J8.S1, J8.S2, J9.8, J9.S1, J9.S2; no longer CAN.P$13, CAN.P$14, CAN.P$4, CAN.P$5, FANS_1.P$13, FANS_1.P$14, FANS_1.P$7, FANS_1.P$8, FANS_2.P$13, FANS_2.P$14, FANS_2.P$6, FANS_2.P$7, FANS_2.P$8, PRESSURE1.P$13, PRESSURE1.P$14, PRESSURE1.P$7, PRESSURE1.P$8, RELAYBOARD3.P$13, RELAYBOARD3.P$14, RELAYBOARD3.P$7, RELAYBOARD3.P$8, RELAYBOARD4.P$13, RELAYBOARD4.P$14, RELAYBOARD4.P$8, TEMPERATURE1.P$13, TEMPERATURE1.P$14, TEMPERATURE1.P$8, VALVES.P$13, VALVES.P$14, VALVES.P$2, VALVES.P$4, VALVES.P$6, VALVES.P$8
- net MOTOR_RELAY: now also J8.4; no longer RELAYBOARD3.P$4
- net MOTOR_VOLT: now also J9.2; no longer RELAYBOARD4.P$2
- net N$6: now also J9.10; no longer RELAYBOARD4.P$12
- net OUTPUT_1_ENET: now also J10.5; no longer VALVES.P$5
- net OUTPUT_2_ENET: now also J10.7; no longer VALVES.P$7
- net PURGE_VALVE_ENET: now also J10.3; no longer VALVES.P$3
- net PWM_1: now also J3.3; no longer FANS_1.P$3
- net PWM_2: now also J3.6; no longer FANS_1.P$6
- net PWM_3: now also J4.3; no longer FANS_2.P$3
- net RX_RS232: now also J7.3; no longer CAN.P$3
- net START_RELAY: now also J8.5; no longer RELAYBOARD3.P$5
- net SUPPLY_VALVE_ENET: now also J10.1; no longer VALVES.P$1
- net TACH_1: now also J3.2; no longer FANS_1.P$2
- net TACH_2: now also J3.5; no longer FANS_1.P$5
- net TACH_3: now also J4.2; no longer FANS_2.P$2
- net TEMP_1: now also J6.3; no longer TEMPERATURE1.P$3
- net TEMP_2: now also J6.4; no longer TEMPERATURE1.P$4
- net TEMP_3: now also J6.5; no longer TEMPERATURE1.P$5
- net TEMP_4: now also J6.6; no longer TEMPERATURE1.P$6
- net TEMP_5: now also J6.7; no longer TEMPERATURE1.P$7
- net TX_RS232: now also J7.6; no longer CAN.P$6
- net _CAP_CURR: now also J9.6; no longer RELAYBOARD4.P$6
- net _FC_CURR: now also J9.4; no longer RELAYBOARD4.P$4
- net _MOTOR_CURR: now also J9.5; no longer RELAYBOARD4.P$5
- net _PRESSURE_1: now also J5.2; no longer PRESSURE1.P$2
- net _PRESSURE_2: now also J5.3; no longer PRESSURE1.P$3
- net _PRESSURE_3: now also J5.4; no longer PRESSURE1.P$4
- net _PRESSURE_4: now also J5.5; no longer PRESSURE1.P$5

Commit message: update
Parts:
- removed U$8: CD143A-SR3.3CT-ND, 3_3V TVS:SOT143_AVAGO
- added D308: P6KE15A-E3/54GICT-ND, 12V TVS:DO-204AC
- added R123, R124: 4.7kΩ, SparkFun-Passives:0805
- moved JP4 34.3 mm to (-6.35, 214.6)
Connections:
- net AUX12V: now also D308.CATHODE
- net FC3V3: now also R123.1, R124.2, U$3.1, U$3.20, U$5.1, U$5.20; no longer U$8.VDD
- net FC5V: no longer U$3.1, U$3.20, U$5.1, U$5.20
- net GND: now also D308.ANODE, R123.2, R124.1; no longer U$8.GND

Commit message: update
Parts:
- R116, R119: value 324Ω -> 65Ω
- R118, R120: value 324Ω -> 10Ω
Changed lines of the file:
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@@
 <attribute name="VALUE" x="-46.736" y="223.393" size="0.4064" layer="27"/>
 </element>
-<element name="R116" library="SparkFun-Passives" package="0805" value="324Ω" x="-53.34" y="224.79" smashed="yes">
+<element name="R116" library="SparkFun-Passives" package="0805" value="65Ω" x="-53.34" y="224.79" smashed="yes">
 <attribute name="NAME" x="-54.102" y="225.6155" size="0.4064" layer="25"/>
 <attribute name="VALUE" x="-54.356" y="223.393" size="0.4064" layer="27"/>
@@
 <attribute name="VALUE" x="-58.166" y="223.393" size="0.4064" layer="27"/>
 </element>
-<element name="R118" library="SparkFun-Passives" package="0805" value="324Ω" x="-60.96" y="224.79" smashed="yes">
+<element name="R118" library="SparkFun-Passives" package="0805" value="10Ω" x="-60.96" y="224.79" smashed="yes">
 <attribute name="NAME" x="-61.722" y="225.6155" size="0.4064" layer="25"/>
 <attribute name="VALUE" x="-61.976" y="223.393" size="0.4064" layer="27"/>
 </element>
-<element name="R119" library="SparkFun-Passives" package="0805" value="324Ω" x="-64.77" y="224.79" smashed="yes">
+<element name="R119" library="SparkFun-Passives" package="0805" value="65Ω" x="-64.77" y="224.79" smashed="yes">
 <attribute name="NAME" x="-65.532" y="225.6155" size="0.4064" layer="25"/>
 <attribute name="VALUE" x="-65.786" y="223.393" size="0.4064" layer="27"/>
 </element>
-<element name="R120" library="SparkFun-Passives" package="0805" value="324Ω" x="-68.58" y="224.79" smashed="yes">
+<element name="R120" library="SparkFun-Passives" package="0805" value="10Ω" x="-68.58" y="224.79" smashed="yes">
 <attribute name="NAME" x="-69.342" y="225.6155" size="0.4064" layer="25"/>
 <attribute name="VALUE" x="-69.596" y="223.393" size="0.4064" layer="27"/>
