File: Sensor-Board_2022_Prototype/Sensor-Board_dev.brd (EAGLE design)
At the start: 355.6 x 253.7 mm, 21 parts

Commit message: Added side signal labels
Connections:
- net N$9: now also UC1.5V; no longer UC1.NC1, UC1.NC2
- net RIGHT_REAR_RX_TTL: now also UC1.PG_9
Changed lines of the file:
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@@
 <wire x1="73.66" y1="146.690715625" x2="25.885" y2="-261.62" width="0" layer="19" extent="1-1"/>
-</signal>
-<signal name="N$9">
-<contactref element="UC1" pad="NC1"/>
-<contactref element="UC1" pad="NC2"/>
-<contactref element="F2" pad="2"/>
-<wire x1="73.66" y1="126.370715625" x2="25.885" y2="-265.43" width="0" layer="19" extent="1-1"/>
-<wire x1="73.66" y1="164.470715625" x2="73.66" y2="126.370715625" width="0" layer="19" extent="1-1"/>
 </signal>
 <signal name="N$25">
@@
 <signal name="RIGHT_REAR_RX_TTL">
 <contactref element="RIGHT_SIG" pad="9"/>
+<contactref element="UC1" pad="PG_9"/>
+<wire x1="41.91" y1="-355.6" x2="121.92" y2="128.910715625" width="0" layer="19" extent="1-1"/>
 </signal>
 <signal name="RIGHT_FWD_TX_TTL">
@@
 <contactref element="UC1" pad="PC_6"/>
 </signal>
+<signal name="N$9">
+<contactref element="UC1" pad="5V"/>
+<contactref element="F2" pad="2"/>
+<wire x1="73.66" y1="154.310715625" x2="25.885" y2="-265.43" width="0" layer="19" extent="1-1"/>
+</signal>
 </signals>
