File: CommsHub_2022_Prototype/board.brd (EAGLE design)
At the start: 100 x 80 mm, 46 parts, among them CON1 TE_6-PIN, CON4 1X02, IC1 MAX3232CSE, IC2 MAX3232CSE, IC3 MAX3232CSE

Commit message: Pushing final schematic
Connections:
- net 3.3V: now also ETH10.P$11, ETH10.P$9, ETH11.P$11, ETH11.P$9, ETH12.P$11, ETH12.P$9, ETH8.P$11, ETH8.P$9, ETH9.P$11, ETH9.P$9
- net RX1: now also ETH8.P$10
- net RX2: now also ETH9.P$10
- net RX3: now also ETH10.P$10
- net RX4: now also ETH11.P$10
- net RX5: now also ETH12.P$10
- net TX1: now also ETH8.P$12
- net TX2: now also ETH9.P$12
- net TX3: now also ETH10.P$12
- net TX4: now also ETH11.P$12
- net TX5: now also ETH12.P$12
Changed lines of the file:
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@@
 <wire x1="10" y1="58.0284" x2="9.8366" y2="57.865" width="0.25" layer="1"/>
 <contactref element="U$1" pad="0-RX1/CS1/CRX2"/>
-<wire x1="23" y1="34" x2="3.06" y2="-108.62" width="0" layer="19" extent="1-1"/>
+<contactref element="ETH8" pad="P$10"/>
+<wire x1="26.43" y1="-4.86" x2="3.06" y2="-108.62" width="0" layer="19" extent="1-1"/>
+<wire x1="23" y1="34" x2="26.43" y2="-4.86" width="0" layer="19" extent="1-1"/>
 </signal>
 <signal name="TX1">
@@
 <wire x1="9.7316" y1="56.7" x2="9.8366" y2="56.595" width="0.25" layer="1"/>
 <contactref element="U$1" pad="1-TX1/MISO1/CTX2"/>
-<wire x1="26" y1="34" x2="5.6" y2="-108.62" width="0" layer="19" extent="1-1"/>
+<contactref element="ETH8" pad="P$12"/>
+<wire x1="37.86" y1="-4.86" x2="5.6" y2="-108.62" width="0" layer="19" extent="1-1"/>
+<wire x1="26" y1="34" x2="37.86" y2="-4.86" width="0" layer="19" extent="1-1"/>
 </signal>
 <signal name="RX3">
@@
 <wire x1="29" y1="35" x2="36.84" y2="35" width="0.25" layer="1"/>
 <contactref element="U$1" pad="15-A1/RX3/SPDIF_IN"/>
-<wire x1="36.84" y1="35" x2="28.46" y2="-93.38" width="0" layer="19" extent="1-1"/>
+<contactref element="ETH10" pad="P$10"/>
+<wire x1="30.43" y1="-27.86" x2="28.46" y2="-93.38" width="0" layer="19" extent="1-1"/>
+<wire x1="36.84" y1="35" x2="30.43" y2="-27.86" width="0" layer="19" extent="1-1"/>
 </signal>
 <signal name="TX3">
@@
 <wire x1="30" y1="40" x2="34.3" y2="40" width="0.25" layer="1"/>
 <contactref element="U$1" pad="14-A0/TX3/SPDIF_OUT"/>
-<wire x1="31" y1="-93.38" x2="34.3" y2="40" width="0" layer="19" extent="1-1"/>
+<contactref element="ETH10" pad="P$12"/>
+<wire x1="41.86" y1="-27.86" x2="34.3" y2="40" width="0" layer="19" extent="1-1"/>
+<wire x1="31" y1="-93.38" x2="41.86" y2="-27.86" width="0" layer="19" extent="1-1"/>
 </signal>
 <signal name="RX2">
@@
 <wire x1="39" y1="39" x2="35.76" y2="39" width="0.25" layer="16"/>
 <contactref element="U$1" pad="7-RX2/OUT1A"/>
-<wire x1="35.76" y1="39" x2="20.84" y2="-108.62" width="0" layer="19" extent="16-16"/>
+<contactref element="ETH9" pad="P$10"/>
+<wire x1="5.43" y1="-27.86" x2="20.84" y2="-108.62" width="0" layer="19" extent="1-1"/>
+<wire x1="35.76" y1="39" x2="5.43" y2="-27.86" width="0" layer="19" extent="16-16"/>
 </signal>
 <signal name="TX2">
@@
 <wire x1="61.6716" y1="56" x2="61.8366" y2="55.835" width="0.25" layer="1"/>
 <contactref element="U$1" pad="8-TX2/IN1"/>
-<wire x1="31.72" y1="37.52" x2="23.38" y2="-108.62" width="0" layer="19" extent="16-16"/>
+<contactref element="ETH9" pad="P$12"/>
+<wire x1="16.86" y1="-27.86" x2="23.38" y2="-108.62" width="0" layer="19" extent="1-1"/>
+<wire x1="31.72" y1="37.52" x2="16.86" y2="-27.86" width="0" layer="19" extent="16-16"/>
 </signal>
 <signal name="RX4">
@@
 <wire x1="35.1816" y1="57" x2="34.8366" y2="57.345" width="0.25" layer="1"/>
 <contactref element="U$1" pad="16-A2/RX4/SCL1"/>
-<wire x1="3.78" y1="38.78" x2="25.92" y2="-93.38" width="0" layer="19" extent="16-16"/>
+<contactref element="ETH11" pad="P$10"/>
+<wire x1="5.43" y1="-46.86" x2="25.92" y2="-93.38" width="0" layer="19" extent="1-1"/>
+<wire x1="3.78" y1="38.78" x2="5.43" y2="-46.86" width="0" layer="19" extent="16-16"/>
 </signal>
 <signal name="TX4">
@@
 <wire x1="34.9116" y1="56" x2="34.8366" y2="56.075" width="0.25" layer="1"/>
 <contactref element="U$1" pad="17-A3/TX4/SDA1"/>
-<wire x1="1.24" y1="40.24" x2="23.38" y2="-93.38" width="0" layer="19" extent="16-16"/>
+<contactref element="ETH11" pad="P$12"/>
+<wire x1="16.86" y1="-46.86" x2="23.38" y2="-93.38" width="0" layer="19" extent="1-1"/>
+<wire x1="1.24" y1="40.24" x2="16.86" y2="-46.86" width="0" layer="19" extent="16-16"/>
 </signal>
 <signal name="RX5">
@@
 <wire x1="8.055" y1="54.055" x2="8" y2="54" width="0.25" layer="1"/>
 <contactref element="U$1" pad="21-A7/RX5/BCLK1"/>
-<wire x1="4" y1="22.48" x2="13.22" y2="-93.38" width="0" layer="19" extent="1-1"/>
+<contactref element="ETH12" pad="P$10"/>
+<wire x1="30.43" y1="-46.86" x2="13.22" y2="-93.38" width="0" layer="19" extent="1-1"/>
+<wire x1="4" y1="22.48" x2="30.43" y2="-46.86" width="0" layer="19" extent="1-1"/>
 </signal>
 <signal name="TX5">
@@
 <wire x1="6.325" y1="55.325" x2="4" y2="53" width="0.25" layer="1"/>
 <contactref element="U$1" pad="20-A6/TX5/LRCLK1"/>
-<wire x1="1" y1="22.5" x2="15.76" y2="-93.38" width="0" layer="19" extent="1-1"/>
+<contactref element="ETH12" pad="P$12"/>
+<wire x1="41.86" y1="-46.86" x2="15.76" y2="-93.38" width="0" layer="19" extent="1-1"/>
+<wire x1="1" y1="22.5" x2="41.86" y2="-46.86" width="0" layer="19" extent="1-1"/>
 </signal>
 <signal name="N$16">
@@
 <contactref element="U$2" pad="5"/>
 <contactref element="C19" pad="1"/>
+<contactref element="ETH12" pad="P$9"/>
+<contactref element="ETH12" pad="P$11"/>
+<contactref element="ETH8" pad="P$9"/>
+<contactref element="ETH8" pad="P$11"/>
+<contactref element="ETH9" pad="P$9"/>
+<contactref element="ETH9" pad="P$11"/>
+<contactref element="ETH11" pad="P$9"/>
+<contactref element="ETH11" pad="P$11"/>
+<contactref element="ETH10" pad="P$9"/>
+<contactref element="ETH10" pad="P$11"/>
 <wire x1="-35.1" y1="-185" x2="-35.1" y2="-197" width="0" layer="19" extent="1-1"/>
 <wire x1="-1.9" y1="-134.7" x2="-35.1" y2="-185" width="0" layer="19" extent="1-1"/>
@@
 <wire x1="36.08" y1="-108.62" x2="5.6" y2="-93.38" width="0" layer="19" extent="1-1"/>
 <wire x1="46.24" y1="-103.54" x2="36.08" y2="-108.62" width="0" layer="19" extent="1-1"/>
-<wire x1="24.1" y1="38.9" x2="8.81" y2="-82.19" width="0" layer="19" extent="16-16"/>
+<wire x1="3.14" y1="-46.86" x2="8.81" y2="-82.19" width="0" layer="19" extent="1-1"/>
+<wire x1="14.57" y1="-46.86" x2="3.14" y2="-46.86" width="0" layer="19" extent="1-1"/>
+<wire x1="28.14" y1="-46.86" x2="14.57" y2="-46.86" width="0" layer="19" extent="1-1"/>
+<wire x1="39.57" y1="-46.86" x2="28.14" y2="-46.86" width="0" layer="19" extent="1-1"/>
+<wire x1="3.14" y1="-27.86" x2="3.14" y2="-46.86" width="0" layer="19" extent="1-1"/>
+<wire x1="14.57" y1="-27.86" x2="3.14" y2="-27.86" width="0" layer="19" extent="1-1"/>
+<wire x1="28.14" y1="-27.86" x2="14.57" y2="-27.86" width="0" layer="19" extent="1-1"/>
+<wire x1="39.57" y1="-27.86" x2="28.14" y2="-27.86" width="0" layer="19" extent="1-1"/>
+<wire x1="35.57" y1="-4.86" x2="39.57" y2="-27.86" width="0" layer="19" extent="1-1"/>
+<wire x1="24.14" y1="-4.86" x2="35.57" y2="-4.86" width="0" layer="19" extent="1-1"/>
+<wire x1="24.1" y1="38.9" x2="24.14" y2="-4.86" width="0" layer="19" extent="16-16"/>
 <wire x1="61.7116" y1="48.34" x2="59" y2="47.82" width="0" layer="19" extent="1-1"/>
 </signal>

Commit message: test
Parts:
- moved D2 346.1 mm to (-38.1, 99.1)
- moved D1 341.1 mm to (-30.5, 99.1)
- moved C21 299.2 mm to (-26.7, 85.1)
- moved R5 299.0 mm to (-77.5, 99.1)
- moved LED5 293.9 mm to (-58.4, 99.1)
- moved R4 292.5 mm to (-73.7, 99.1)
- moved C18 289.5 mm to (-17.8, 85.1)
- moved LED4 287.7 mm to (-54.6, 99.1)
- moved R3 286.1 mm to (-69.8, 99.1)
- moved LED3 281.4 mm to (-50.8, 99.1)
- moved R2 279.7 mm to (-66.0, 99.1)
- moved LED2 275.3 mm to (-47.0, 99.1)
- moved LED1 272.2 mm to (-43.2, 99.1)
- moved R1 270.3 mm to (-62.2, 99.1)
- moved C20 248.3 mm to (-17.8, 100.3)
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Routing:
- net 3.3V: track 111.1 -> 0.00 mm, vias 5 -> 0
- net TX1: track 92.2 -> 0.00 mm, vias 4 -> 0
- net RX1: track 78.6 -> 0.00 mm, vias 3 -> 0
- net RS_RX4: track 73.5 -> 0.00 mm, vias 2 -> 0
- net RS_TX2: track 59.1 -> 0.00 mm
- net RS_TX4: track 58.5 -> 0.00 mm, vias 2 -> 0
- net RS_TX3: track 53.3 -> 0.00 mm, vias 1 -> 0
- net RX4: track 52.2 -> 0.00 mm, vias 1 -> 0
- net TX4: track 50.7 -> 0.00 mm, vias 1 -> 0
- net RS_RX3: track 46.7 -> 0.00 mm, vias 2 -> 0
- net TX2: track 44.0 -> 0.00 mm, vias 1 -> 0
- net RX2: track 41.8 -> 0.00 mm, vias 1 -> 0
- net TX5: track 38.5 -> 0.00 mm
- net RX3: track 37.5 -> 0.00 mm, vias 2 -> 0
- net RX5: track 35.3 -> 0.00 mm
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- removed copper zone on layer 1, net GND
- removed copper zone on layer 16, net GND
Other:
- board size 100 x 80 mm -> 163.8 x 136.8 mm
- board text removed: "CAN"
- board text removed: "FAST SERIAL"
- board text removed: "SERIAL"
