File: FCBoard/FCBoard.kicad_sch (KiCad schematic)
At the start: 97 parts, among them CON4 1X01, CON5 1X01, CON6 1X02, CON7 1X01, CON8 1X02, CON9 1X01, U1 ADP2302ARDZ-5.0-R7, U2 LTC4412HVIS6TRMPBF, U3 LTC4412HVIS6TRMPBF, U4 SI9433BDY-T1-E3, U5 SI9433BDY-T1-E3, U6 SI9433BDY-T1-E3

Commit message: Updates
Parts:
- removed C1, C18, C19, C2, C9: 10uF, FCC Power Board Aug 2022_OW:C1210, symbol FCC Power Board Aug 2022_OW-eagle-import:C-EUC1210
- removed C10, C20, C3: 1uF, FCC Power Board Aug 2022_OW:C0805, symbol FCC Power Board Aug 2022_OW-eagle-import:C-EUC0805
- removed C11, C12, C21, C4: 0.1uF, FCC Power Board Aug 2022_OW:C0603, symbol FCC Power Board Aug 2022_OW-eagle-import:C-EUC0603
- removed C13, C14, C15: EEU-FC2A221, FCC Power Board Aug 2022_OW:CAP_16_X_25, symbol FCC Power Board Aug 2022_OW-eagle-import:EEU-FC2A221
- removed C16, C17, C22, C7, C8: EEUFR1H221B, FCC Power Board Aug 2022_OW:CAP_PAN_10X16, symbol FCC Power Board Aug 2022_OW-eagle-import:EEUFR1H221B
- removed C23, C28, C31, C32, C37, C40: 220uF, FCC Power Board Aug 2022_OW:CAPACITOR_220UF_63V, symbol FCC Power Board Aug 2022_OW-eagle-import:CAPACITOR_ELECTROLYTIC_220UF
- removed C24, C33: 0.1uF, FCC Power Board Aug 2022_OW:0805, symbol FCC Power Board Aug 2022_OW-eagle-import:CAPACITOR_0805
- removed C25, C26, C27, C34, C35, C36: 10uF, FCC Power Board Aug 2022_OW:0805, symbol FCC Power Board Aug 2022_OW-eagle-import:CAPACITOR_0805
- removed C29, C38: 1nF/50V, FCC Power Board Aug 2022_OW:0805, symbol FCC Power Board Aug 2022_OW-eagle-import:CAPACITOR_0805
- removed C30, C39: 1uF/50V, FCC Power Board Aug 2022_OW:0805, symbol FCC Power Board Aug 2022_OW-eagle-import:CAPACITOR_0805
- removed C5, C6: 1uF, FCC Power Board Aug 2022_OW:C1210, symbol FCC Power Board Aug 2022_OW-eagle-import:C-EUC1210
- removed CON4, CON5, CON7, CON9: 1X01, FCC Power Board Aug 2022_OW:1X01, symbol FCC Power Board Aug 2022_OW-eagle-import:1X01
- removed CON6, CON8: 1X02, FCC Power Board Aug 2022_OW:1X02, symbol FCC Power Board Aug 2022_OW-eagle-import:1X02
- removed D7: SMBJ12A, FCC Power Board Aug 2022_OW:DO214AA, symbol FCC Power Board Aug 2022_OW-eagle-import:DIODE_TVS_UNI_DO-214AA
- removed D8: SMBJ5.0A, FCC Power Board Aug 2022_OW:DO214AA, symbol FCC Power Board Aug 2022_OW-eagle-import:DIODE_TVS_UNI_DO-214AA
- removed E1, E2, E3: 5555140-6, FCC Power Board Aug 2022_OW:1734723-1_RJ11, symbol FCC Power Board Aug 2022_OW-eagle-import:5555140-6
- removed F2, F3: 7.5A, FCC Power Board Aug 2022_OW:FUSEHOLDER_VERTICAL, symbol FCC Power Board Aug 2022_OW-eagle-import:FUSEHOLDER_VERTICAL
- removed JP1: JP1E, FCC Power Board Aug 2022_OW:JP1, symbol FCC Power Board Aug 2022_OW-eagle-import:JP1E
- removed LED1: Amber 1.9V, FCC Power Board Aug 2022_OW:CHIPLED_0805, symbol FCC Power Board Aug 2022_OW-eagle-import:LEDCHIPLED_0805
- removed LED2: Blue 3.3V, FCC Power Board Aug 2022_OW:CHIPLED_0805, symbol FCC Power Board Aug 2022_OW-eagle-import:LEDCHIPLED_0805
- removed LED3, LED4, LED5: LEDCHIPLED_0805, FCC Power Board Aug 2022_OW:CHIPLED_0805, symbol FCC Power Board Aug 2022_OW-eagle-import:LEDCHIPLED_0805
- removed LED6, LED7: RED, FCC Power Board Aug 2022_OW:0805_LED, symbol FCC Power Board Aug 2022_OW-eagle-import:LED_0805
- removed MOD1, MOD2: i3A, FCC Power Board Aug 2022_OW:CONVERTER_I3A, symbol FCC Power Board Aug 2022_OW-eagle-import:CONVERTER_I3A
- removed R1: R-US_R0603, FCC Power Board Aug 2022_OW:R0603, symbol FCC Power Board Aug 2022_OW-eagle-import:R-US_R0603
- removed R10: 8.2k, FCC Power Board Aug 2022_OW:0805, symbol FCC Power Board Aug 2022_OW-eagle-import:RESISTOR_0805
- removed R11, R9: 10k, FCC Power Board Aug 2022_OW:TRIMPOT, symbol FCC Power Board Aug 2022_OW-eagle-import:RESISTOR_TRIMPOT
- removed R12: 2k, FCC Power Board Aug 2022_OW:0805, symbol FCC Power Board Aug 2022_OW-eagle-import:RESISTOR_0805
- removed R13: 560, FCC Power Board Aug 2022_OW:0805, symbol FCC Power Board Aug 2022_OW-eagle-import:RESISTOR_0805
- removed R8: 1.6k, FCC Power Board Aug 2022_OW:0805, symbol FCC Power Board Aug 2022_OW-eagle-import:RESISTOR_0805
- removed SV1, SV2: MA03-1, FCC Power Board Aug 2022_OW:MA03-1, symbol FCC Power Board Aug 2022_OW-eagle-import:MA03-1
- removed TP1, TP2, TP3: TEST-POINT3X5, FCC Power Board Aug 2022_OW:PAD.03X.05, symbol FCC Power Board Aug 2022_OW-eagle-import:TEST-POINT3X5
- removed U$1: RPA60-2412SFW_P, FCC Power Board Aug 2022_OW:RPA60-2412SFW_P, symbol FCC Power Board Aug 2022_OW-eagle-import:RPA60-2412SFW_P
- removed U$10: SMAJ12A, FCC Power Board Aug 2022_OW:SMA-DO214AC, symbol FCC Power Board Aug 2022_OW-eagle-import:SMAJ12A
- removed U$11: SMAJ5.0A, FCC Power Board Aug 2022_OW:SMA-DO214AC, symbol FCC Power Board Aug 2022_OW-eagle-import:SMAJ5.0A
- removed U$12, U$13: NSI45020AT1G, FCC Power Board Aug 2022_OW:SOD123, symbol FCC Power Board Aug 2022_OW-eagle-import:NSI45020AT1G
- removed U$18, U$20: 2X1-CONN, FCC Power Board Aug 2022_OW:2X1-MATE-N-LOCK, symbol FCC Power Board Aug 2022_OW-eagle-import:2X1-CONN
- removed U$2: 47uH, FCC Power Board Aug 2022_OW:INDUCTOR_SMD_FOOTPRINT, symbol FCC Power Board Aug 2022_OW-eagle-import:PA4320
- removed U$21: M3_SCREW_TERMINAL, FCC Power Board Aug 2022_OW:M3_SCREW_TERMINAL, symbol FCC Power Board Aug 2022_OW-eagle-import:M3_SCREW_TERMINAL
- removed U$3: 744770112, FCC Power Board Aug 2022_OW:INDUCTOR_SMD_FOOTPRINT, symbol FCC Power Board Aug 2022_OW-eagle-import:744770112
- removed U$4: DB2460500L, FCC Power Board Aug 2022_OW:SOD123, symbol FCC Power Board Aug 2022_OW-eagle-import:DB2460500L
- removed U$5, U$6, U$7: SHELL2013_FUSEMINI-BLADE, FCC Power Board Aug 2022_OW:SHELL2013_MINI-BLADE-FUSE, symbol FCC Power Board Aug 2022_OW-eagle-import:SHELL2013_FUSEMINI-BLADE
- removed U$8: P4SMA51A, FCC Power Board Aug 2022_OW:SMA-DO214AC, symbol FCC Power Board Aug 2022_OW-eagle-import:P4SMA51A
- removed U$9: VS-15EWL06FNTR-M3, FCC Power Board Aug 2022_OW:TO252, symbol FCC Power Board Aug 2022_OW-eagle-import:VS-15EWL06FNTR-M3
- removed U1: ADP2302ARDZ-5.0-R7, FCC Power Board Aug 2022_OW:RD_8_1, symbol FCC Power Board Aug 2022_OW-eagle-import:ADP2302ARDZ-5.0-R7
- removed U2, U3: LTC4412HVIS6TRMPBF, FCC Power Board Aug 2022_OW:TSOT-23_S6, symbol FCC Power Board Aug 2022_OW-eagle-import:LTC4412HVIS6TRMPBF
- removed U4, U5, U6: SI9433BDY-T1-E3, FCC Power Board Aug 2022_OW:SOIC-N-8_SI, symbol FCC Power Board Aug 2022_OW-eagle-import:SI9433BDY-T1-E3
- added C41, C42, C43: EEU-FC2A221, FCC Power Board Aug 2022_OW:CAP_16_X_25, symbol FCC Power Board Aug 2022_OW-eagle-import:EEU-FC2A221
- added C44, C45: 1uF, FCC Power Board Aug 2022_OW:C1210, symbol FCC Power Board Aug 2022_OW-eagle-import:C-EUC1210
- added C46, C47, C53, C66, C67: EEUFR1H221B, FCC Power Board Aug 2022_OW:CAP_PAN_10X16, symbol FCC Power Board Aug 2022_OW-eagle-import:EEUFR1H221B
- added C48, C49, C62, C68, C69: 10uF, FCC Power Board Aug 2022_OW:C1210, symbol FCC Power Board Aug 2022_OW-eagle-import:C-EUC1210
- added C50, C63, C70: 1uF, FCC Power Board Aug 2022_OW:C0805, symbol FCC Power Board Aug 2022_OW-eagle-import:C-EUC0805
- added C51, C64, C65, C71: 0.1uF, FCC Power Board Aug 2022_OW:C0603, symbol FCC Power Board Aug 2022_OW-eagle-import:C-EUC0603
- added C52, C72: 1nF/50V, FCC Power Board Aug 2022_OW:0805, symbol FCC Power Board Aug 2022_OW-eagle-import:CAPACITOR_0805
- added C54, C73: 1uF/50V, FCC Power Board Aug 2022_OW:0805, symbol FCC Power Board Aug 2022_OW-eagle-import:CAPACITOR_0805
- added C55, C60, C61, C74, C79, C80: 220uF, FCC Power Board Aug 2022_OW:CAPACITOR_220UF_63V, symbol FCC Power Board Aug 2022_OW-eagle-import:CAPACITOR_ELECTROLYTIC_220UF
- added C56, C75: 0.1uF, FCC Power Board Aug 2022_OW:0805, symbol FCC Power Board Aug 2022_OW-eagle-import:CAPACITOR_0805
- added C57, C58, C59, C76, C77, C78: 10uF, FCC Power Board Aug 2022_OW:0805, symbol FCC Power Board Aug 2022_OW-eagle-import:CAPACITOR_0805
- added CON1, CON10: 1X02, FCC Power Board Aug 2022_OW:1X02, symbol FCC Power Board Aug 2022_OW-eagle-import:1X02
- added CON11, CON12, CON2, CON3: 1X01, FCC Power Board Aug 2022_OW:1X01, symbol FCC Power Board Aug 2022_OW-eagle-import:1X01
- added D1: SMBJ12A, FCC Power Board Aug 2022_OW:DO214AA, symbol FCC Power Board Aug 2022_OW-eagle-import:DIODE_TVS_UNI_DO-214AA
- added D2: SMBJ5.0A, FCC Power Board Aug 2022_OW:DO214AA, symbol FCC Power Board Aug 2022_OW-eagle-import:DIODE_TVS_UNI_DO-214AA
- added E4, E5, E6: 5555140-6, FCC Power Board Aug 2022_OW:1734723-1_RJ11, symbol FCC Power Board Aug 2022_OW-eagle-import:5555140-6
- added F1, F4: 7.5A, FCC Power Board Aug 2022_OW:FUSEHOLDER_VERTICAL, symbol FCC Power Board Aug 2022_OW-eagle-import:FUSEHOLDER_VERTICAL
- added JP2: JP1E, FCC Power Board Aug 2022_OW:JP1, symbol FCC Power Board Aug 2022_OW-eagle-import:JP1E
- added LED10, LED13, LED14: LEDCHIPLED_0805, FCC Power Board Aug 2022_OW:CHIPLED_0805, symbol FCC Power Board Aug 2022_OW-eagle-import:LEDCHIPLED_0805
- added LED11: Amber 1.9V, FCC Power Board Aug 2022_OW:CHIPLED_0805, symbol FCC Power Board Aug 2022_OW-eagle-import:LEDCHIPLED_0805
- added LED12: Blue 3.3V, FCC Power Board Aug 2022_OW:CHIPLED_0805, symbol FCC Power Board Aug 2022_OW-eagle-import:LEDCHIPLED_0805
- added LED8, LED9: RED, FCC Power Board Aug 2022_OW:0805_LED, symbol FCC Power Board Aug 2022_OW-eagle-import:LED_0805
- added MOD3, MOD4: i3A, FCC Power Board Aug 2022_OW:CONVERTER_I3A, symbol FCC Power Board Aug 2022_OW-eagle-import:CONVERTER_I3A
- added R14: 560, FCC Power Board Aug 2022_OW:0805, symbol FCC Power Board Aug 2022_OW-eagle-import:RESISTOR_0805
- added R2: 1.6k, FCC Power Board Aug 2022_OW:0805, symbol FCC Power Board Aug 2022_OW-eagle-import:RESISTOR_0805
- added R3, R7: 10k, FCC Power Board Aug 2022_OW:TRIMPOT, symbol FCC Power Board Aug 2022_OW-eagle-import:RESISTOR_TRIMPOT
- added R4: 2k, FCC Power Board Aug 2022_OW:0805, symbol FCC Power Board Aug 2022_OW-eagle-import:RESISTOR_0805
- added R5: R-US_R0603, FCC Power Board Aug 2022_OW:R0603, symbol FCC Power Board Aug 2022_OW-eagle-import:R-US_R0603
- added R6: 8.2k, FCC Power Board Aug 2022_OW:0805, symbol FCC Power Board Aug 2022_OW-eagle-import:RESISTOR_0805
- added SV3, SV4: MA03-1, FCC Power Board Aug 2022_OW:MA03-1, symbol FCC Power Board Aug 2022_OW-eagle-import:MA03-1
- added U$14, U$22, U$28: SHELL2013_FUSEMINI-BLADE, FCC Power Board Aug 2022_OW:SHELL2013_MINI-BLADE-FUSE, symbol FCC Power Board Aug 2022_OW-eagle-import:SHELL2013_FUSEMINI-BLADE
- added U$15: VS-15EWL06FNTR-M3, FCC Power Board Aug 2022_OW:TO252, symbol FCC Power Board Aug 2022_OW-eagle-import:VS-15EWL06FNTR-M3
- added U$16: P4SMA51A, FCC Power Board Aug 2022_OW:SMA-DO214AC, symbol FCC Power Board Aug 2022_OW-eagle-import:P4SMA51A
- added U$17: 47uH, FCC Power Board Aug 2022_OW:INDUCTOR_SMD_FOOTPRINT, symbol FCC Power Board Aug 2022_OW-eagle-import:PA4320
- added U$19: RPA60-2412SFW_P, FCC Power Board Aug 2022_OW:RPA60-2412SFW_P, symbol FCC Power Board Aug 2022_OW-eagle-import:RPA60-2412SFW_P
- added U$23, U$24: 2X1-CONN, FCC Power Board Aug 2022_OW:2X1-MATE-N-LOCK, symbol FCC Power Board Aug 2022_OW-eagle-import:2X1-CONN
- added U$25: M3_SCREW_TERMINAL, FCC Power Board Aug 2022_OW:M3_SCREW_TERMINAL, symbol FCC Power Board Aug 2022_OW-eagle-import:M3_SCREW_TERMINAL
- added U$26: DB2460500L, FCC Power Board Aug 2022_OW:SOD123, symbol FCC Power Board Aug 2022_OW-eagle-import:DB2460500L
- added U$27: 744770112, FCC Power Board Aug 2022_OW:INDUCTOR_SMD_FOOTPRINT, symbol FCC Power Board Aug 2022_OW-eagle-import:744770112
- added U$29, U$30: NSI45020AT1G, FCC Power Board Aug 2022_OW:SOD123, symbol FCC Power Board Aug 2022_OW-eagle-import:NSI45020AT1G
- added U7: ADP2302ARDZ-5.0-R7, FCC Power Board Aug 2022_OW:RD_8_1, symbol FCC Power Board Aug 2022_OW-eagle-import:ADP2302ARDZ-5.0-R7
Connections:
- net 12V: now also C53.1 (11), C62.1, C63.1, C64.1, D1.C, E5.2, E5.5, E6.2, E6.5, F1.3 (2), F1.4 (2), LED10.A, LED8.1 (A), R5.1, U$24.CIRCUIT1 (P$1), U7.2 (VIN), U7.3 (EN)
- net 12V_PRE_FUSE: now also C56.1, C57.1, C58.1, C59.1, C60.+, C61.+, CON2.1, F1.1, F1.2 (1), MOD3.7 (SENSE+), MOD3.8 (VOUT)
- net 12V_REG: now also U$22.IN
- net 5V: now also D2.C, E5.3, E5.4, E6.3, E6.4, F4.3 (2), F4.4 (2), LED11.A, LED9.1 (A), U$23.CIRCUIT1 (P$1)
- net 5V_PRE_FUSE: now also C75.1, C76.1, C77.1, C78.1, C79.+, C80.+, CON11.1, F4.1, F4.2 (1), MOD4.7 (SENSE+), MOD4.8 (VOUT)
- net FEEDBACK: now also C66.1 (11), C67.1 (11), C68.1, C69.1, C70.1, C71.1, U$27.1 (+), U$28.IN, U7.5 (FB)
- net GND: now also C46.2 (22), C47.2 (22), C48.2, C49.2, C50.2, C51.2, C52.2, C53.2 (22), C54.2, C55.-, C56.2, C57.2, C58.2, C59.2, C60.-, C61.-, C62.2, C63.2, C64.2, C66.2 (22), C67.2 (22), C68.2, C69.2, C70.2, C71.2, C72.2, C73.2, C74.-, C75.2, C76.2, C77.2, C78.2, C79.-, C80.-, CON1.1, CON10.1, CON12.1, CON3.1, D1.A, D2.A, E5.1, E5.6, E5.SH1, E5.SH2, E6.1, E6.6, E6.SH1, E6.SH2, MOD3.3 (GND), MOD3.4 (GND), MOD4.3 (GND), MOD4.4 (GND), R14.1, R3.3 (CW), R4.1, R7.3 (CW), SV3.1, SV3.2, SV4.1, SV4.2, U$19.P$5 (GNDOUT), U$23.GND, U$24.GND, U$25.P$1 (1), U$25.P$2 (2), U$25.P$3 (3), U$25.P$4 (4), U$26.A, U$29.C, U$30.C, U7.6 (NC), U7.7 (GND), U7.EPAD
- net VIN: now also C41.1 (11), C52.1, C54.1, C55.+, C72.1, C73.1, C74.+, MOD3.1 (VIN), MOD4.1 (VIN), U$14.IN, U$15.3 (C), U$16.K (C), U$17.2 (-)
- new net: CON1.2, MOD3.2 (ON/OFF)
- new net: C65.1, U7.1 (BST)
- new net: C65.2, U$26.C, U$27.2 (-), U7.8 (SW)
- new net: CON10.2, MOD4.2 (ON/OFF)
- new net: C42.1 (11), C43.1 (11), C44.1, C45.1, JP2.2, U$17.1 (+), U$19.P$1 (VIN)
- new net: C46.1 (11), C47.1 (11), C48.1, C49.1, C50.1, C51.1, U$19.P$6 (VOUT), U$22.OUT
- new net: MOD4.6 (TRIM), R6.1
- new net: R5.2, U7.4 (PGOOD)
- new net: LED9.2 (C), R14.2
- new net: LED11.C, LED13.A
- new net: LED13.C, U$29.A
- new net: LED10.C, LED12.A
- new net: LED12.C, LED14.A
- new net: MOD3.6 (TRIM), R2.1
- new net: R2.2, R3.1 (CCW), R3.2 (WIPER)
- new net: LED8.2 (C), R4.2
- new net: LED14.C, U$30.A
- new net: JP2.1, U$19.P$3 (CRTL)
- new net: R6.2, R7.1 (CCW), R7.2 (WIPER)
- new net 5V_REG: U$28.OUT
- new net FC_IN: E4.2, E4.3, E4.4, E4.5, U$14.OUT
- new net GND_IN: C41.2 (22), C42.2 (22), C43.2 (22), C44.2, C45.2, E4.1, E4.6, E4.SH1, E4.SH2, SV3.3, SV4.3, U$15.1 (A), U$15.2 (A), U$16.A, U$19.P$2 (GNDIN)
Other:
- note added: "12V DC-DC Converter"
- note added: "5V DC-DC Converter"
- note added: "Input Connector"
- note added: "LED Test"
- note added: "Output Connectors"
- note added: "Protection System"
- note removed: "1"
- note removed: "12V DC-DC"
- note removed: "2"
- note removed: "3"
- note removed: "4"
- note removed: "5"
- note removed: "6"
- note removed: "7"
- note removed: "8"
- note removed: "A"
- note removed: "B"
- note removed: "C"
- note removed: "D"
- note removed: "E"
- note removed: "INPUT"
- note removed: "LED TEST"

Commit message: Organization
Other:
- note removed: "OUTPUT"
- moved on the sheet: C44, C45, C48, C49, C50, C51, C52, C54, C55, C56, C57, C58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
