File: LoRa_Tranciever_sch-DESKTOP-UUV004C.kicad_sch (KiCad schematic)
At the start: 16 parts, among them J3 Conn_Coaxial, U3 SX1280IMLTRT, Y1 52MHz

Commit message: Made minor changes
Other:
- moved on the sheet: J3
Changed lines of the file:
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@@
     (stroke (width 0) (type default))
   )
-  (wire (pts (xy 185.42 69.85) (xy 189.23 69.85))
+  (wire (pts (xy 185.42 69.85) (xy 218.44 69.85))
     (stroke (width 0) (type default))
   )
@@
     (stroke (width 0) (type default))
   )
-  (wire (pts (xy 194.31 74.93) (xy 194.31 80.01))
+  (wire (pts (xy 223.52 74.93) (xy 223.52 80.01))
     (stroke (width 0) (type default))
   )
@@
     (effects (font (size 1.27 1.27)) (justify right))
   )
-  (hierarchical_label "SX1280_NRESET" (shape input) (at 46.99 67.31 180) (fields_autoplaced)
-    (effects (font (size 1.27 1.27)) (justify right))
-  )
   (hierarchical_label "DIO1" (shape bidirectional) (at 58.42 81.28 180) (fields_autoplaced)
     (effects (font (size 1.27 1.27)) (justify right))
@@
     )
   )
-  (symbol (lib_id "power:GND") (at 194.31 80.01 0) (unit 1)
-    (in_bom yes) (on_board yes) (dnp no) (fields_autoplaced)
-    (property "Reference" "#PWR042" (at 194.31 86.36 0)
-      (effects (font (size 1.27 1.27)) hide)
-    )
-    (property "Value" "GND" (at 194.31 85.09 0)
+  (symbol (lib_id "power:GND") (at 223.52 80.01 0) (unit 1)
+    (in_bom yes) (on_board yes) (dnp no) (fields_autoplaced)
+    (property "Reference" "#PWR042" (at 223.52 86.36 0)
+      (effects (font (size 1.27 1.27)) hide)
+    )
+    (property "Value" "GND" (at 223.52 85.09 0)
       (effects (font (size 1.27 1.27)))
     )
-    (property "Footprint" "" (at 194.31 80.01 0)
-      (effects (font (size 1.27 1.27)) hide)
-    )
-    (property "Datasheet" "" (at 194.31 80.01 0)
+    (property "Footprint" "" (at 223.52 80.01 0)
+      (effects (font (size 1.27 1.27)) hide)
+    )
+    (property "Datasheet" "" (at 223.52 80.01 0)
       (effects (font (size 1.27 1.27)) hide)
     )
@@
     )
   )
-  (symbol (lib_id "Connector:Conn_Coaxial") (at 194.31 69.85 0) (unit 1)
-    (in_bom yes) (on_board yes) (dnp no) (fields_autoplaced)
-    (property "Reference" "J3" (at 198.12 68.8732 0)
+  (symbol (lib_id "Connector:Conn_Coaxial") (at 223.52 69.85 0) (unit 1)
+    (in_bom yes) (on_board yes) (dnp no) (fields_autoplaced)
+    (property "Reference" "J3" (at 227.33 68.8732 0)
       (effects (font (size 1.27 1.27)) (justify left))
     )
-    (property "Value" "Conn_Coaxial" (at 198.12 71.4132 0)
+    (property "Value" "Conn_Coaxial" (at 227.33 71.4132 0)
       (effects (font (size 1.27 1.27)) (justify left))
     )
-    (property "Footprint" "footprints:TAOGLAS_EMPCB.SMAFSTJ.B.HT" (at 194.31 69.85 0)
-      (effects (font (size 1.27 1.27)) hide)
-    )
-    (property "Datasheet" " ~" (at 194.31 69.85 0)
-      (effects (font (size 1.27 1.27)) hide)
-    )
+    (property "Footprint" "footprints:TAOGLAS_EMPCB.SMAFSTJ.B.HT" (at 223.52 69.85 0)
+      (effects (font (size 1.27 1.27)) hide)
+    )
+    (property "Datasheet" " ~" (at 223.52 69.85 0)
+      (effects (font (size 1.27 1.27)) hide)
+    )
