File: usb_interface.kicad_sch (KiCad schematic)
At the start: 13 parts, among them J4 USB_B_Micro, U5 FT234XD-R

Commit message: Ready to order added all part numbers
Parts:
- C14, C16, C?: JLC # C327414 -> (none); LCSC # (none) -> C1525
- C15: LCSC # (none) -> C307423
- C? (x2): LCSC # (none) -> C1567
- D10: JLC # C510024 -> (none); JLC Link https://jlcpcb.com/partdetail/RohmSemicon-SMLD12D8WT86/C510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 -> (none)
- D?: JLC # C7519 -> (none)
- J4: JLC # C132562 -> (none)
- R17: LCSC # (none) -> C22966
- R18, R19: LCSC # (none) -> C2933185
- U5: JLC # C132158 -> (none)
Changed lines of the file:
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@@
       (effects (font (size 1.524 1.524)) (justify left) hide)
-    )
-    (property "JLC #" "C7519" (at 127 86.36 0)
-      (effects (font (size 1.27 1.27)) hide)
-    )
-    (property "JLC Link" "" (at 127 86.36 0)
-      (effects (font (size 1.27 1.27)) hide)
-    )
-    (property "DK Link" "" (at 127 86.36 0)
-      (effects (font (size 1.27 1.27)) hide)
     )
     (property "MPN" "" (at 127 86.36 0)
@@
       (effects (font (size 1.27 1.27)) hide)
     )
-    (property "JLC #" "C327414" (at 62.23 104.14 0)
-      (effects (font (size 1.27 1.27)) hide)
-    )
-    (property "JLC Link" "" (at 62.23 104.14 0)
-      (effects (font (size 1.27 1.27)) hide)
-    )
-    (property "DK Link" "" (at 62.23 104.14 0)
-      (effects (font (size 1.27 1.27)) hide)
-    )
     (property "MPN" "" (at 62.23 104.14 0)
       (effects (font (size 1.27 1.27)) hide)
     )
-    (property "LCSC #" "" (at 62.23 104.14 0)
+    (property "LCSC #" "C1525" (at 62.23 104.14 0)
       (effects (font (size 1.27 1.27)) hide)
     )
@@
       (effects (font (size 1.27 1.27)) hide)
     )
-    (property "JLC Link" "" (at 69.85 66.04 0)
-      (effects (font (size 1.27 1.27)) hide)
-    )
-    (property "DK Link" "" (at 69.85 66.04 0)
-      (effects (font (size 1.27 1.27)) hide)
-    )
     (property "MPN" "" (at 69.85 66.04 0)
       (effects (font (size 1.27 1.27)) hide)
     )
-    (property "LCSC #" "" (at 69.85 66.04 0)
+    (property "LCSC #" "C22966" (at 69.85 66.04 0)
       (effects (font (size 1.27 1.27)) hide)
     )
@@
       (effects (font (size 1.27 1.27)) hide)
     )
-    (property "JLC #" "C327414" (at 39.37 105.41 0)
-      (effects (font (size 1.27 1.27)) hide)
-    )
-    (property "JLC Link" "" (at 39.37 105.41 0)
-      (effects (font (size 1.27 1.27)) hide)
-    )
-    (property "DK Link" "" (at 39.37 105.41 0)
-      (effects (font (size 1.27 1.27)) hide)
-    )
     (property "MPN" "" (at 39.37 105.41 0)
       (effects (font (size 1.27 1.27)) hide)
     )
-    (property "LCSC #" "" (at 39.37 105.41 0)
+    (property "LCSC #" "C1525" (at 39.37 105.41 0)
       (effects (font (size 1.27 1.27)) hide)
     )
@@
       (effects (font (size 1.27 1.27)) hide)
     )
-    (property "JLC Link" "" (at 76.2 86.36 0)
-      (effects (font (size 1.27 1.27)) hide)
-    )
-    (property "DK Link" "" (at 76.2 86.36 0)
-      (effects (font (size 1.27 1.27)) hide)
-    )
     (property "MPN" "" (at 76.2 86.36 0)
       (effects (font (size 1.27 1.27)) hide)
     )
-    (property "LCSC #" "" (at 76.2 86.36 0)
+    (property "LCSC #" "C2933185" (at 76.2 86.36 0)
       (effects (font (size 1.27 1.27)) hide)
     )
@@
       (effects (font (size 1.27 1.27)) hide)
     )
-    (property "JLC Link" "" (at 167.64 85.09 0)
-      (effects (font (size 1.27 1.27)) hide)
-    )
-    (property "DK Link" "" (at 167.64 85.09 0)
-      (effects (font (size 1.27 1.27)) hide)
-    )
     (property "MPN" "" (at 167.64 85.09 0)
       (effects (font (size 1.27 1.27)) hide)
     )
     (property "Description" "USB 2.0 1 Surface Mount 5P Female -30℃~+80℃ Micro-B SMD  USB Connectors ROHS" (at 167.64 85.09 0)
-      (effects (font (size 1.27 1.27)) hide)
-    )
-    (property "JLC #" "C132562" (at 167.64 85.09 0)
       (effects (font (size 1.27 1.27)) hide)
     )
@@
     (property "Description" "IC USB SERIAL BASIC UART 12DFN" (at 48.26 111.76 0)
       (effects (font (size 1.524 1.524)) (justify left) hide)
-    )
-    (property "JLC #" "C132158" (at 53.34 86.36 0)
-      (effects (font (size 1.27 1.27)) hide)
-    )
-    (property "JLC Link" "" (at 53.34 86.36 0)
-      (effects (font (size 1.27 1.27)) hide)
-    )
-    (property "DK Link" "" (at 53.34 86.36 0)
-      (effects (font (size 1.27 1.27)) hide)
     )
     (property "MPN" "" (at 53.34 86.36 0)
@@
       (effects (font (size 1.27 1.27)) hide)
     )
-    (property "JLC Link" "https://jlcpcb.com/partdetail/RohmSemicon-SMLD12D8WT86/C510024" (at 78.74 66.04 0)
-      (effects (font (size 1.27 1.27)) hide)
-    )
-    (property "DK Link" "" (at 78.74 66.04 0)
-      (effects (font (size 1.27 1.27)) hide)
-    )
     (property "MPN" "" (at 78.74 66.04 0)
       (effects (font (size 1.27 1.27)) hide)
@@
       (effects (font (size 1.27 1.27)) hide)
     )
-    (property "JLC #" "C510024" (at 78.74 66.04 0)
-      (effects (font (size 1.27 1.27)) hide)
-    )
     (pin "1")
     (pin "2")
@@
       (effects (font (size 1.27 1.27)) hide)
     )
-    (property "JLC #" "C327414" (at 106.68 104.14 0)
-      (effects (font (size 1.27 1.27)) hide)
-    )
-    (property "JLC Link" "" (at 106.68 104.14 0)
-      (effects (font (size 1.27 1.27)) hide)
-    )
-    (property "DK Link" "" (at 106.68 104.14 0)
-      (effects (font (size 1.27 1.27)) hide)
-    )
     (property "MPN" "" (at 106.68 104.14 0)
       (effects (font (size 1.27 1.27)) hide)
     )
-    (property "LCSC #" "" (at 106.68 104.14 0)
+    (property "LCSC #" "C1525" (at 106.68 104.14 0)
       (effects (font (size 1.27 1.27)) hide)
     )
@@
       (effects (font (size 1.27 1.27)) hide)
     )
-    (property "JLC Link" "" (at 82.55 104.14 0)
-      (effects (font (size 1.27 1.27)) hide)
-    )
-    (property "DK Link" "" (at 82.55 104.14 0)
-      (effects (font (size 1.27 1.27)) hide)
-    )
     (property "MPN" "" (at 82.55 104.14 0)
       (effects (font (size 1.27 1.27)) hide)
     )
-    (property "LCSC #" "" (at 82.55 104.14 0)
+    (property "LCSC #" "C1567" (at 82.55 104.14 0)
       (effects (font (size 1.27 1.27)) hide)
     )
@@
       (effects (font (size 1.27 1.27)) hide)
     )
-    (property "JLC Link" "" (at 90.17 104.14 0)
-      (effects (font (size 1.27 1.27)) hide)
-    )
-    (property "DK Link" "" (at 90.17 104.14 0)
-      (effects (font (size 1.27 1.27)) hide)
-    )
     (property "MPN" "" (at 90.17 104.14 0)
       (effects (font (size 1.27 1.27)) hide)
     )
-    (property "LCSC #" "" (at 90.17 104.14 0)
+    (property "LCSC #" "C1567" (at 90.17 104.14 0)
       (effects (font (size 1.27 1.27)) hide)
     )
@@
       (effects (font (size 1.27 1.27)) hide)
     )
-    (property "JLC Link" "" (at 54.61 104.14 0)
-      (effects (font (size 1.27 1.27)) hide)
-    )
-    (property "DK Link" "" (at 54.61 104.14 0)
-      (effects (font (size 1.27 1.27)) hide)
-    )
     (property "MPN" "" (at 54.61 104.14 0)
       (effects (font (size 1.27 1.27)) hide)
     )
-    (property "LCSC #" "" (at 54.61 104.14 0)
+    (property "LCSC #" "C307423" (at 54.61 104.14 0)
       (effects (font (size 1.27 1.27)) hide)
     )
@@
       (effects (font (size 1.27 1.27)) hide)
     )
-    (property "JLC Link" "" (at 76.2 88.9 0)
-      (effects (font (size 1.27 1.27)) hide)
-    )
-    (property "DK Link" "" (at 76.2 88.9 0)
-      (effects (font (size 1.27 1.27)) hide)
-    )
     (property "MPN" "" (at 76.2 88.9 0)
       (effects (font (size 1.27 1.27)) hide)
     )
-    (property "LCSC #" "" (at 76.2 88.9 0)
-      (effects (font (size 1.27 1.27)) hide)
-    )
+    (property "LCSC #" "C2933185" (at 76.2 88.9 0)
+      (effects (font (size 1.27 1.27)) hide)
+    )
