File: Fuel_Cell_Controller_Prototype/sensors.kicad_sch (KiCad schematic)
At the start: 11 parts, among them U6 SHT31-DIS, U8 ADA4898-2

Commit message: Big overall changes. Check git project board to ensure work is not repeated
Parts:
- renumbered U6 to U7
Changed lines of the file:
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@@
         )
         (path "/f651cec9-411c-4a4e-a163-5c49adbe6a12/26245637-81d1-4f60-832a-3f71fed7a491"
-          (reference "#PWR042") (unit 1)
+          (reference "#PWR058") (unit 1)
         )
       )
@@
         )
         (path "/f651cec9-411c-4a4e-a163-5c49adbe6a12/26245637-81d1-4f60-832a-3f71fed7a491"
-          (reference "#PWR035") (unit 1)
+          (reference "#PWR054") (unit 1)
         )
       )
@@
         )
         (path "/f651cec9-411c-4a4e-a163-5c49adbe6a12/26245637-81d1-4f60-832a-3f71fed7a491"
-          (reference "#PWR036") (unit 1)
+          (reference "#PWR057") (unit 1)
         )
       )
@@
         )
         (path "/f651cec9-411c-4a4e-a163-5c49adbe6a12/26245637-81d1-4f60-832a-3f71fed7a491"
-          (reference "R23") (unit 1)
+          (reference "R33") (unit 1)
         )
       )
@@
         )
         (path "/f651cec9-411c-4a4e-a163-5c49adbe6a12/26245637-81d1-4f60-832a-3f71fed7a491"
-          (reference "#PWR033") (unit 1)
+          (reference "#PWR051") (unit 1)
         )
       )
@@
   (symbol (lib_id "power:GND") (at 49.53 111.76 0) (unit 1)
     (in_bom yes) (on_board yes) (dnp no) (fields_autoplaced)
-    (property "Reference" "#PWR043" (at 49.53 118.11 0)
+    (property "Reference" "#PWR055" (at 49.53 118.11 0)
       (effects (font (size 1.27 1.27)) hide)
     )
@@
       (project "Fuel_Cell_Controller_Prototype"
         (path "/f651cec9-411c-4a4e-a163-5c49adbe6a12/26245637-81d1-4f60-832a-3f71fed7a491"
-          (reference "#PWR043") (unit 1)
+          (reference "#PWR055") (unit 1)
         )
       )
@@
         )
         (path "/f651cec9-411c-4a4e-a163-5c49adbe6a12/26245637-81d1-4f60-832a-3f71fed7a491"
-          (reference "R21") (unit 1)
+          (reference "R29") (unit 1)
         )
       )
@@
         )
         (path "/f651cec9-411c-4a4e-a163-5c49adbe6a12/26245637-81d1-4f60-832a-3f71fed7a491"
-          (reference "#PWR037") (unit 1)
+          (reference "#PWR059") (unit 1)
         )
       )
@@
         )
         (path "/f651cec9-411c-4a4e-a163-5c49adbe6a12/26245637-81d1-4f60-832a-3f71fed7a491"
-          (reference "#PWR039") (unit 1)
+          (reference "#PWR056") (unit 1)
         )
       )
@@
         )
         (path "/f651cec9-411c-4a4e-a163-5c49adbe6a12/26245637-81d1-4f60-832a-3f71fed7a491"
-          (reference "R25") (unit 1)
+          (reference "R31") (unit 1)
         )
       )
@@
         )
         (path "/f651cec9-411c-4a4e-a163-5c49adbe6a12/26245637-81d1-4f60-832a-3f71fed7a491"
-          (reference "R24") (unit 1)
+          (reference "R34") (unit 1)
         )
       )
@@
         )
         (path "/f651cec9-411c-4a4e-a163-5c49adbe6a12/26245637-81d1-4f60-832a-3f71fed7a491"
-          (reference "#PWR038") (unit 1)
+          (reference "#PWR060") (unit 1)
         )
       )
@@
   (symbol (lib_id "Sensor_Humidity:SHT31-DIS") (at 49.53 104.14 0) (unit 1)
     (in_bom yes) (on_board yes) (dnp no) (fields_autoplaced)
-    (property "Reference" "U6" (at 51.4859 93.98 0)
+    (property "Reference" "U7" (at 51.4859 93.98 0)
       (effects (font (size 1.27 1.27)) (justify left))
     )
@@
       (project "Fuel_Cell_Controller_Prototype"
         (path "/f651cec9-411c-4a4e-a163-5c49adbe6a12/26245637-81d1-4f60-832a-3f71fed7a491"
-          (reference "U6") (unit 1)
+          (reference "U7") (unit 1)
         )
       )
@@
   (symbol (lib_id "power:GND") (at 36.83 111.76 0) (unit 1)
     (in_bom yes) (on_board yes) (dnp no) (fields_autoplaced)
-    (property "Reference" "#PWR044" (at 36.83 118.11 0)
+    (property "Reference" "#PWR053" (at 36.83 118.11 0)
       (effects (font (size 1.27 1.27)) hide)
     )
@@
       (project "Fuel_Cell_Controller_Prototype"
         (path "/f651cec9-411c-4a4e-a163-5c49adbe6a12/26245637-81d1-4f60-832a-3f71fed7a491"
+          (reference "#PWR053") (unit 1)
+        )
+      )
+    )
+  )
+  (symbol (lib_id "Diode:BZV55C3V3") (at 74.93 58.42 270) (unit 1)
+    (in_bom yes) (on_board yes) (dnp no) (fields_autoplaced)
+    (property "Reference" "D8" (at 77.47 57.15 90)
+      (effects (font (size 1.27 1.27)) (justify left))
+    )
+    (property "Value" "BZV55C3V3" (at 77.47 59.69 90)
+      (effects (font (size 1.27 1.27)) (justify left))
+    )
+    (property "Footprint" "Diode_SMD:D_MiniMELF" (at 70.485 58.42 0)
+      (effects (font (size 1.27 1.27)) hide)
+    )
+    (property "Datasheet" "https://assets.nexperia.com/documents/data-sheet/BZV55_SER.pdf" (at 74.93 58.42 0)
+      (effects (font (size 1.27 1.27)) hide)
+    )
+    (pin "1")
+    (pin "2")
+    (instances
+      (project "Fuel_Cell_Controller_Prototype"
+        (path "/f651cec9-411c-4a4e-a163-5c49adbe6a12"
+          (reference "D8") (unit 1)
+        )
+        (path "/f651cec9-411c-4a4e-a163-5c49adbe6a12/26245637-81d1-4f60-832a-3f71fed7a491"
+          (reference "D11") (unit 1)
+        )
+      )
+    )
+  )
+  (symbol (lib_id "power:GND") (at 33.02 64.77 0) (unit 1)
+    (in_bom yes) (on_board yes) (dnp no) (fields_autoplaced)
+    (property "Reference" "#PWR044" (at 33.02 71.12 0)
+      (effects (font (size 1.27 1.27)) hide)
+    )
+    (property "Value" "GND" (at 33.02 69.85 0)
+      (effects (font (size 1.27 1.27)))
+    )
+    (property "Footprint" "" (at 33.02 64.77 0)
+      (effects (font (size 1.27 1.27)) hide)
+    )
+    (property "Datasheet" "" (at 33.02 64.77 0)
+      (effects (font (size 1.27 1.27)) hide)
+    )
+    (pin "1")
+    (instances
+      (project "Fuel_Cell_Controller_Prototype"
+        (path "/f651cec9-411c-4a4e-a163-5c49adbe6a12"
           (reference "#PWR044") (unit 1)
         )
-      )
-    )
-  )
-  (symbol (lib_id "Diode:BZV55C3V3") (at 74.93 58.42 270) (unit 1)
-    (in_bom yes) (on_board yes) (dnp no) (fields_autoplaced)
-    (property "Reference" "D8" (at 77.47 57.15 90)
-      (effects (font (size 1.27 1.27)) (justify left))
-    )
-    (property "Value" "BZV55C3V3" (at 77.47 59.69 90)
-      (effects (font (size 1.27 1.27)) (justify left))
-    )
-    (property "Footprint" "Diode_SMD:D_MiniMELF" (at 70.485 58.42 0)
-      (effects (font (size 1.27 1.27)) hide)
-    )
-    (property "Datasheet" "https://assets.nexperia.com/documents/data-sheet/BZV55_SER.pdf" (at 74.93 58.42 0)
-      (effects (font (size 1.27 1.27)) hide)
-    )
-    (pin "1")
-    (pin "2")
-    (instances
-      (project "Fuel_Cell_Controller_Prototype"
-        (path "/f651cec9-411c-4a4e-a163-5c49adbe6a12"
-          (reference "D8") (unit 1)
-        )
-        (path "/f651cec9-411c-4a4e-a163-5c49adbe6a12/26245637-81d1-4f60-832a-3f71fed7a491"
-          (reference "D9") (unit 1)
-        )
-      )
-    )
-  )
-  (symbol (lib_id "power:GND") (at 33.02 64.77 0) (unit 1)
-    (in_bom yes) (on_board yes) (dnp no) (fields_autoplaced)
-    (property "Reference" "#PWR044" (at 33.02 71.12 0)
-      (effects (font (size 1.27 1.27)) hide)
-    )
-    (property "Value" "GND" (at 33.02 69.85 0)
-      (effects (font (size 1.27 1.27)))
-    )
-    (property "Footprint" "" (at 33.02 64.77 0)
-      (effects (font (size 1.27 1.27)) hide)
-    )
-    (property "Datasheet" "" (at 33.02 64.77 0)
-      (effects (font (size 1.27 1.27)) hide)
-    )
-    (pin "1")
-    (instances
-      (project "Fuel_Cell_Controller_Prototype"
-        (path "/f651cec9-411c-4a4e-a163-5c49adbe6a12"
-          (reference "#PWR044") (unit 1)
-        )
-        (path "/f651cec9-411c-4a4e-a163-5c49adbe6a12/26245637-81d1-4f60-832a-3f71fed7a491"
-          (reference "#PWR034") (unit 1)
+        (path "/f651cec9-411c-4a4e-a163-5c49adbe6a12/26245637-81d1-4f60-832a-3f71fed7a491"
+          (reference "#PWR052") (unit 1)
         )
       )
@@
         )
         (path "/f651cec9-411c-4a4e-a163-5c49adbe6a12/26245637-81d1-4f60-832a-3f71fed7a491"
-          (reference "D10") (unit 1)
+          (reference "D12") (unit 1)
         )
       )
@@
         )
         (path "/f651cec9-411c-4a4e-a163-5c49adbe6a12/26245637-81d1-4f60-832a-3f71fed7a491"
-          (reference "#PWR045") (unit 1)
+          (reference "#PWR050") (unit 1)
         )
       )
@@
         )
         (path "/f651cec9-411c-4a4e-a163-5c49adbe6a12/26245637-81d1-4f60-832a-3f71fed7a491"
-          (reference "R22") (unit 1)
+          (reference "R30") (unit 1)
         )
       )
@@
         )
         (path "/f651cec9-411c-4a4e-a163-5c49adbe6a12/26245637-81d1-4f60-832a-3f71fed7a491"
-          (reference "#PWR040") (unit 1)
+          (reference "#PWR061") (unit 1)
         )
       )
@@
         )
         (path "/f651cec9-411c-4a4e-a163-5c49adbe6a12/26245637-81d1-4f60-832a-3f71fed7a491"
-          (reference "R26") (unit 1)
-        )
-      )
+          (reference "R32") (unit 1)
+        )
+      )

Commit message: Sensors Update
Parts:
- removed D6, D8: BZV55C3V3, Diode_SMD:D_MiniMELF, symbol Diode:BZV55C3V3
- removed U8: ADA4898-2, Package_SO:SOIC-8-1EP_3.9x4.9mm_P1.27mm_EP2.41x3.81mm, symbol Amplifier_Operational:ADA4898-2
- added C39: 10uF, symbol Device:C
- added D7, D8: BZV55B3V6, Diode_SMD:D_MiniMELF, symbol Diode:BZV55B3V6
- added U9: MCP602-E/SN, Package_SO:SOIC-8_3.9x4.9mm_P1.27mm, symbol Device:Opamp_Dual
- R25, R26: value ~ -> 100k
- R27: value ~ -> 52.3k
- R28: value ~ -> 13.7k
Connections:
- net +3V3: now also C39.1
- net +5V: now also U9.8 (V+)
- net 12V_Ref: now also D7.1 (K), U9.1, U9.2 (-)
- net 5V_Ref: now also D8.1 (K), U9.6 (-), U9.7
- net GND: now also C39.2, D7.2 (A), D8.2 (A), U9.4 (V-)
- net at R25.2, R26.1: now also U9.5 (+)
- net at R27.2, R28.1: now also U9.3 (+)
Other:
- note added: "V_{in} = V_{s}[R_{2}/(R_{1}+R_{2})] = 2.5V R_{2} = 0.26R_{1}"
- note added: "Voltage Sensors"
- note removed: "MIKAEL: - Concered the zener diodes you chose above have V_{r} too low. We want to have range up to and probably a bit over 3.3V for good measure. Just as long as the max never exceeds 4.5 to 5V - Datasheet for the SHT31D you included doesn't seem to work for me (might just be my end) let me know if its working for you. - Maybe leave a note on any unfinished circuits so that I don't point stuff o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"
- note removed: "Single supply opamp (5V good) Needs to be unity gain stable (also known as a compensated opamp) Standard V+ V- IN+ IN- and one out (Look at dual SOIC-8 packaging)"
- moved on the sheet: R25, R26, R27, U7
