File: Rev 2/usb_interface.kicad_sch (KiCad schematic)
At the start: 13 parts, among them J4 USB_B_Micro, U7 FT234XD-R

Commit message: added GPSW and HW DB
Parts:
- D?: JLCPCB Part#(optional) C7519 -> (none); LCSC # C7519 -> (none)
- J4: JLCPCB Part#(optional) C428495 -> (none); LCSC # C428495 -> (none)
Changed lines of the file:
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@@
       (effects (font (size 1.27 1.27)) hide)
     )
-    (property "LCSC #" "C7519" (at 127 86.36 0)
-      (effects (font (size 1.27 1.27)) hide)
-    )
-    (property "JLCPCB Part#(optional)" "C7519" (at 127 86.36 0)
+    (property "LCSC #" "" (at 127 86.36 0)
+      (effects (font (size 1.27 1.27)) hide)
+    )
+    (property "JLCPCB Part#(optional)" "" (at 127 86.36 0)
       (effects (font (size 1.27 1.27)) hide)
     )
@@
       (effects (font (size 1.27 1.27)) hide)
     )
-    (property "LCSC #" "C428495" (at 167.64 85.09 0)
-      (effects (font (size 1.27 1.27)) hide)
-    )
-    (property "JLCPCB Part#(optional)" "C428495" (at 167.64 85.09 0)
-      (effects (font (size 1.27 1.27)) hide)
-    )
+    (property "LCSC #" "" (at 167.64 85.09 0)
+      (effects (font (size 1.27 1.27)) hide)
+    )
+    (property "JLCPCB Part#(optional)" "" (at 167.64 85.09 0)
+      (effects (font (size 1.27 1.27)) hide)
+    )
