File: Rev 2/power_regulator.kicad_sch (KiCad schematic)
At the start: 28 parts, among them J2 Fuel Cell Connector, J3 USB JMPR, Q1 NMOS, U3 TPS2596, U4 BAT54CTA, U5 AZ1117-3.3, U6 AZ1117-5.0

Commit message: added GPSW and HW DB
Parts:
- J2: JLCPCB Part#(optional) C476812 -> (none); LCSC # C476812 -> (none)
- J3, JP?: JLCPCB Part#(optional) C5116482 -> (none); LCSC # C5116482 -> (none)
- Q1: JLCPCB Part#(optional) C475757 -> (none); LCSC # C475757 -> (none)
- U3: JLCPCB Part#(optional) C2155774 -> (none); LCSC # C2155774 -> (none)
- U4: JLCPCB Part#(optional) C460164 -> (none); LCSC # C460164 -> (none)
- U5: JLCPCB Part#(optional) C110474 -> (none); LCSC # C110474 -> (none)
- U6: JLCPCB Part#(optional) C99343 -> (none); LCSC # C99343 -> (none)
Changed lines of the file:
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@@
       (effects (font (size 1.27 1.27)) hide)
     )
-    (property "LCSC #" "C475757" (at 132.08 83.82 0)
-      (effects (font (size 1.27 1.27)) hide)
-    )
-    (property "JLCPCB Part#(optional)" "C475757" (at 132.08 83.82 0)
+    (property "LCSC #" "" (at 132.08 83.82 0)
+      (effects (font (size 1.27 1.27)) hide)
+    )
+    (property "JLCPCB Part#(optional)" "" (at 132.08 83.82 0)
       (effects (font (size 1.27 1.27)) hide)
     )
@@
       (effects (font (size 1.27 1.27)) hide)
     )
-    (property "LCSC #" "C476812" (at 168.91 138.43 0)
-      (effects (font (size 1.27 1.27)) hide)
-    )
-    (property "JLCPCB Part#(optional)" "C476812" (at 168.91 138.43 0)
+    (property "LCSC #" "" (at 168.91 138.43 0)
+      (effects (font (size 1.27 1.27)) hide)
+    )
+    (property "JLCPCB Part#(optional)" "" (at 168.91 138.43 0)
       (effects (font (size 1.27 1.27)) hide)
     )
@@
       (effects (font (size 1.27 1.27)) hide)
     )
-    (property "LCSC #" "C110474" (at 185.42 44.45 0)
-      (effects (font (size 1.27 1.27)) hide)
-    )
-    (property "JLCPCB Part#(optional)" "C110474" (at 185.42 44.45 0)
+    (property "LCSC #" "" (at 185.42 44.45 0)
+      (effects (font (size 1.27 1.27)) hide)
+    )
+    (property "JLCPCB Part#(optional)" "" (at 185.42 44.45 0)
       (effects (font (size 1.27 1.27)) hide)
     )
@@
       (effects (font (size 1.27 1.27)) hide)
     )
-    (property "LCSC #" "C2155774" (at 77.47 57.15 0)
-      (effects (font (size 1.27 1.27)) hide)
-    )
-    (property "JLCPCB Part#(optional)" "C2155774" (at 77.47 57.15 0)
+    (property "LCSC #" "" (at 77.47 57.15 0)
+      (effects (font (size 1.27 1.27)) hide)
+    )
+    (property "JLCPCB Part#(optional)" "" (at 77.47 57.15 0)
       (effects (font (size 1.27 1.27)) hide)
     )
@@
       (effects (font (size 1.27 1.27)) hide)
     )
-    (property "LCSC #" "C5116482" (at 208.28 134.62 0)
-      (effects (font (size 1.27 1.27)) hide)
-    )
-    (property "JLCPCB Part#(optional)" "C5116482" (at 208.28 134.62 0)
+    (property "LCSC #" "" (at 208.28 134.62 0)
+      (effects (font (size 1.27 1.27)) hide)
+    )
+    (property "JLCPCB Part#(optional)" "" (at 208.28 134.62 0)
       (effects (font (size 1.27 1.27)) hide)
     )
@@
       (effects (font (size 1.27 1.27)) hide)
     )
-    (property "LCSC #" "C460164" (at 128.27 44.45 0)
-      (effects (font (size 1.27 1.27)) hide)
-    )
-    (property "JLCPCB Part#(optional)" "C460164" (at 128.27 44.45 0)
+    (property "LCSC #" "" (at 128.27 44.45 0)
+      (effects (font (size 1.27 1.27)) hide)
+    )
+    (property "JLCPCB Part#(optional)" "" (at 128.27 44.45 0)
       (effects (font (size 1.27 1.27)) hide)
     )
@@
       (effects (font (size 1.27 1.27)) hide)
     )
-    (property "LCSC #" "C5116482" (at 35.56 46.99 0)
-      (effects (font (size 1.27 1.27)) hide)
-    )
-    (property "JLCPCB Part#(optional)" "C5116482" (at 35.56 46.99 0)
+    (property "LCSC #" "" (at 35.56 46.99 0)
+      (effects (font (size 1.27 1.27)) hide)
+    )
+    (property "JLCPCB Part#(optional)" "" (at 35.56 46.99 0)
       (effects (font (size 1.27 1.27)) hide)
     )
@@
       (effects (font (size 1.27 1.27)) hide)
     )
-    (property "LCSC #" "C99343" (at 259.08 43.18 0)
-      (effects (font (size 1.27 1.27)) hide)
-    )
-    (property "JLCPCB Part#(optional)" "C99343" (at 259.08 43.18 0)
-      (effects (font (size 1.27 1.27)) hide)
-    )
+    (property "LCSC #" "" (at 259.08 43.18 0)
+      (effects (font (size 1.27 1.27)) hide)
+    )
+    (property "JLCPCB Part#(optional)" "" (at 259.08 43.18 0)
+      (effects (font (size 1.27 1.27)) hide)
+    )

Commit message: S
Parts:
- R6: JLCPCB Part#(optional) C25815 -> (none)
- R7: JLCPCB Part#(optional) C228086 -> (none); LCSC # C228086 -> C170688; PCBA - -> (none)
Other:
- moved on the sheet: C21
Changed lines of the file:
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@@
   (junction (at 128.27 53.34) (diameter 0) (color 0 0 0 0)
   )
+  (junction (at 78.74 68.58) (diameter 0) (color 0 0 0 0)
+  )
   (junction (at 198.12 44.45) (diameter 0) (color 0 0 0 0)
   )
   (junction (at 171.45 44.45) (diameter 0) (color 0 0 0 0)
   )
-  (junction (at 77.47 68.58) (diameter 0) (color 0 0 0 0)
-  )
   (junction (at 163.83 44.45) (diameter 0) (color 0 0 0 0)
   )
@@
     (stroke (width 0) (type default))
   )
-  (wire (pts (xy 72.39 81.28) (xy 77.47 81.28))
+  (wire (pts (xy 73.66 81.28) (xy 77.47 81.28))
     (stroke (width 0) (type default))
   )
@@
     (stroke (width 0) (type default))
   )
+  (wire (pts (xy 78.74 68.58) (xy 77.47 68.58))
+    (stroke (width 0) (type default))
+  )
   (wire (pts (xy 134.62 53.34) (xy 134.62 54.61))
     (stroke (width 0) (type default))
@@
     (stroke (width 0) (type default))
   )
+  (wire (pts (xy 78.74 68.58) (xy 80.01 68.58))
+    (stroke (width 0) (type default))
+  )
   (wire (pts (xy 128.27 49.53) (xy 128.27 53.34))
     (stroke (width 0) (type default))
@@
     (stroke (width 0) (type default))
   )
-  (wire (pts (xy 72.39 68.58) (xy 74.93 68.58))
-    (stroke (width 0) (type default))
-  )
-  (wire (pts (xy 72.39 78.74) (xy 72.39 81.28))
-    (stroke (width 0) (type default))
-  )
-  (wire (pts (xy 77.47 68.58) (xy 80.01 68.58))
+  (wire (pts (xy 73.66 68.58) (xy 74.93 68.58))
+    (stroke (width 0) (type default))
+  )
+  (wire (pts (xy 73.66 78.74) (xy 73.66 81.28))
     (stroke (width 0) (type default))
   )
@@
     (stroke (width 0) (type default))
   )
-  (wire (pts (xy 72.39 68.58) (xy 72.39 71.12))
+  (wire (pts (xy 73.66 68.58) (xy 73.66 71.12))
     (stroke (width 0) (type default))
   )
@@
     (stroke (width 0) (type default))
   )
+  (wire (pts (xy 78.74 81.28) (xy 77.47 81.28))
+    (stroke (width 0) (type default))
+  )
   (wire (pts (xy 134.62 66.04) (xy 134.62 62.23))
     (stroke (width 0) (type default))
@@
     (stroke (width 0) (type default))
   )
-  (wire (pts (xy 77.47 68.58) (xy 77.47 81.28))
+  (wire (pts (xy 78.74 68.58) (xy 78.74 81.28))
     (stroke (width 0) (type default))
   )
@@
     )
   )
-  (symbol (lib_id "Device:C") (at 72.39 74.93 0) (unit 1)
-    (in_bom yes) (on_board yes) (dnp no)
-    (property "Reference" "C21" (at 67.31 69.85 0)
-      (effects (font (size 1.27 1.27)) (justify left))
-    )
-    (property "Value" "2n2" (at 67.31 72.39 0)
-      (effects (font (size 1.27 1.27)) (justify left))
-    )
-    (property "Footprint" "Capacitor_SMD:C_0603_1608Metric" (at 73.3552 78.74 0)
-      (effects (font (size 1.27 1.27)) hide)
-    )
-    (property "Datasheet" "~" (at 72.39 74.93 0)
-      (effects (font (size 1.27 1.27)) hide)
-    )
-    (property "JLCPCB Part#(optional)" "C1604" (at 72.39 74.93 0)
-      (effects (font (size 1.27 1.27)) hide)
-    )
-    (property "LCSC #" "C1604" (at 72.39 74.93 0)
-      (effects (font (size 1.27 1.27)) hide)
-    )
-    (property "DK #" "1276-1000-1-ND" (at 72.39 74.93 0)
-      (effects (font (size 1.27 1.27)) hide)
-    )
-    (property "PCBA" "-" (at 72.39 74.93 0)
+  (symbol (lib_id "Device:C") (at 73.66 74.93 0) (unit 1)
+    (in_bom yes) (on_board yes) (dnp no)
+    (property "Reference" "C21" (at 66.04 73.66 0)
+      (effects (font (size 1.27 1.27)) (justify left))
+    )
+    (property "Value" "2n2" (at 66.04 76.2 0)
+      (effects (font (size 1.27 1.27)) (justify left))
+    )
+    (property "Footprint" "Capacitor_SMD:C_0603_1608Metric" (at 74.6252 78.74 0)
+      (effects (font (size 1.27 1.27)) hide)
+    )
+    (property "Datasheet" "~" (at 73.66 74.93 0)
+      (effects (font (size 1.27 1.27)) hide)
+    )
+    (property "JLCPCB Part#(optional)" "C1604" (at 73.66 74.93 0)
+      (effects (font (size 1.27 1.27)) hide)
+    )
+    (property "LCSC #" "C1604" (at 73.66 74.93 0)
+      (effects (font (size 1.27 1.27)) hide)
+    )
+    (property "DK #" "1276-1000-1-ND" (at 73.66 74.93 0)
+      (effects (font (size 1.27 1.27)) hide)
+    )
+    (property "PCBA" "-" (at 73.66 74.93 0)
       (effects (font (size 1.27 1.27)) hide)
     )
@@
       (effects (font (size 1.27 1.27)) hide)
     )
-    (property "JLCPCB Part#(optional)" "C228086" (at 59.69 68.58 0)
-      (effects (font (size 1.27 1.27)) hide)
-    )
-    (property "LCSC #" "C228086" (at 59.69 68.58 0)
+    (property "JLCPCB Part#(optional)" "" (at 59.69 68.58 0)
+      (effects (font (size 1.27 1.27)) hide)
+    )
+    (property "LCSC #" "C170688" (at 59.69 68.58 0)
       (effects (font (size 1.27 1.27)) hide)
     )
@@
       (effects (font (size 1.27 1.27)) hide)
     )
-    (property "PCBA" "-" (at 59.69 68.58 0)
+    (property "PCBA" "" (at 59.69 68.58 0)
       (effects (font (size 1.27 1.27)) hide)
     )
@@
       (effects (font (size 1.27 1.27)) hide)
     )
-    (property "JLCPCB Part#(optional)" "C25815" (at 59.69 58.42 0)
+    (property "JLCPCB Part#(optional)" "" (at 59.69 58.42 0)
       (effects (font (size 1.27 1.27)) hide)
     )
@@
   (symbol (lib_id "Device:R") (at 90.17 76.2 0) (unit 1)
     (in_bom yes) (on_board yes) (dnp no)
-    (property "Reference" "R9" (at 82.55 74.93 0)
-      (effects (font (size 1.27 1.27)) (justify left))
-    )
-    (property "Value" "1k1" (at 82.55 77.47 0)
-      (effects (font (size 1.27 1.27)) (justify left))
-    )
+    (property "Reference" "R9" (at 83.82 74.93 0)
+      (effects (font (size 1.27 1.27)) (justify left))
+    )
+    (property "Value" "1k1" (at 83.82 77.47 0)
+      (effects (font (size 1.27 1.27)) (justify left))
+    )
