File: H2-Sensor-Board2022_Lucy/H2 Sensor Board Lucy Rev 1/CAN_MOD.kicad_sch (KiCad schematic)
At the start: 0 parts

Commit message: Telem, FTDI, MCU, CAN
Added basic components for FTDI, on board telemetry,  & CAN transceiver.

Cleaned up some wiring, added STLink connector with ESD.
Parts:
- added C? (x2): 100n, Capacitor_SMD:C_0603_1608Metric, symbol Device:C
- added J6: Conn_01x09_Socket, Connector_Dsub:DSUB-9_Female_Horizontal_P2.77x2.84mm_EdgePinOffset7.70mm_Housed_MountingHolesOffset9.12mm, symbol Connector:Conn_01x09_Socket
- added U10: MCP2542FD-E/SN, Package_SO:SOIC-8-1EP_3.9x4.9mm_P1.27mm_EP2.29x3mm, symbol Interface_CAN_LIN:MCP2542FDxMF
Connections:
- new net +3V3: C?.2, U10.5 (VIO)
- new net +5V: C?.2, U10.3 (VDD)
- new net CAN_RX: U10.4 (RXD)
- new net CAN_STBY: U10.8 (STBY)
- new net CAN_TX: U10.1 (TXD)
- new net CD+: J6.7 (Pin_7), U10.7 (CANH)
- new net CD-: J6.2 (Pin_2), U10.6 (CANL)
- new net GND: C?.1, C?.1, U10.2 (VSS), U10.9 (VSS)
- no-connect marks 0 -> 7
Other:
- note added: "CAN Tranciever with ESD protection IC"
- note added: "ESD Protected CAN Tranciever"
- note added: "Vdd is 5v and Vio is 3v3"
