File: H2-Sensor-Board2022_Lucy/H2 Sensor Board Lucy Rev 1/USB_mod.kicad_sch (KiCad schematic)
At the start: 0 parts

Commit message: Telem, FTDI, MCU, CAN
Added basic components for FTDI, on board telemetry,  & CAN transceiver.

Cleaned up some wiring, added STLink connector with ESD.
Parts:
- added U9: FT230XS, Package_SO:SSOP-16_3.9x4.9mm_P0.635mm, symbol Interface_USB:FT230XS
Changed lines of the file:
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@@
 (kicad_sch (version 20230121) (generator eeschema)
   (paper "A4")
+  (symbol (lib_id "Interface_USB:FT230XS") (at 99.06 52.705 0) (unit 1)
+    (in_bom yes) (on_board yes) (dnp no) (fields_autoplaced)
+    (property "Reference" "U9" (at 103.7941 34.29 0)
+      (effects (font (size 1.27 1.27)) (justify left))
+    )
+    (property "Value" "FT230XS" (at 103.7941 36.83 0)
+      (effects (font (size 1.27 1.27)) (justify left))
+    )
+    (property "Footprint" "Package_SO:SSOP-16_3.9x4.9mm_P0.635mm" (at 124.46 67.945 0)
+      (effects (font (size 1.27 1.27)) hide)
+    )
+    (property "Datasheet" "https://www.ftdichip.com/Support/Documents/DataSheets/ICs/DS_FT230X.pdf" (at 99.06 52.705 0)
+      (effects (font (size 1.27 1.27)) hide)
+    )
+    (pin "1")
+    (pin "10")
+    (pin "11")
+    (pin "12")
+    (pin "13")
+    (pin "14")
+    (pin "15")
+    (pin "16")
+    (pin "2")
+    (pin "3")
+    (pin "4")
+    (pin "5")
+    (pin "6")
+    (pin "7")
+    (pin "8")
+    (pin "9")
+    (instances
+      (project "H2 Sensor Board Lucy Rev 1"
+        (path "/61fdd4a1-2d1e-44dc-8644-252e12d35745/2e2857d1-75ac-46cb-bf4a-c9d81a36e813"
+          (reference "U9") (unit 1)
+        )
+      )
+    )
+  )
 )
