File: H2-Sensor-Board2022_Lucy/H2 Sensor Board Lucy Rev 1/Preheater.kicad_sch (KiCad schematic)
At the start: 2 parts

Commit message: Humiditiy sensor and other small cahnges
Parts:
- removed D11: BAT54C, Package_TO_SOT_SMD:SOT-23, symbol Diode:BAT54C
- removed U10: ~, symbol H2_Parts:H2_Simon_Sensor_Breakout
Changed lines of the file:
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@@
 (kicad_sch (version 20230121) (generator eeschema)
   (paper "A4")
-  (wire (pts (xy 35.56 73.66) (xy 53.34 73.66))
-    (stroke (width 0) (type default))
-  )
-  (wire (pts (xy 25.4 52.07) (xy 27.94 52.07))
-    (stroke (width 0) (type default))
-  )
-  (wire (pts (xy 35.56 57.15) (xy 35.56 73.66))
-    (stroke (width 0) (type default))
-  )
-  (wire (pts (xy 88.9 73.66) (xy 83.82 73.66))
-    (stroke (width 0) (type default))
-  )
-  (wire (pts (xy 25.4 50.8) (xy 25.4 52.07))
-    (stroke (width 0) (type default))
-  )
-  (global_label "VBAT_5V" (shape input) (at 43.18 52.07 0) (fields_autoplaced)
-    (effects (font (size 1.27 1.27)) (justify left))
-    (property "Intersheetrefs" "${INTERSHEET_REFS}" (at 53.8457 52.07 0)
-      (effects (font (size 1.27 1.27)) (justify left) hide)
-    )
-  )
-  (global_label "V_SENSE" (shape input) (at 88.9 73.66 0) (fields_autoplaced)
-    (effects (font (size 1.27 1.27)) (justify left))
-    (property "Intersheetrefs" "${INTERSHEET_REFS}" (at 99.9889 73.66 0)
-      (effects (font (size 1.27 1.27)) (justify left) hide)
-    )
-  )
-  (symbol (lib_id "power:GND") (at 68.58 88.9 0) (unit 1)
-    (in_bom yes) (on_board yes) (dnp no) (fields_autoplaced)
-    (property "Reference" "#PWR056" (at 68.58 95.25 0)
-      (effects (font (size 1.27 1.27)) hide)
-    )
-    (property "Value" "GND" (at 68.58 93.98 0)
-      (effects (font (size 1.27 1.27)))
-    )
-    (property "Footprint" "" (at 68.58 88.9 0)
-      (effects (font (size 1.27 1.27)) hide)
-    )
-    (property "Datasheet" "" (at 68.58 88.9 0)
-      (effects (font (size 1.27 1.27)) hide)
-    )
-    (pin "1")
-    (instances
-      (project "H2 Sensor Board Lucy Rev 1"
-        (path "/61fdd4a1-2d1e-44dc-8644-252e12d35745/59a3a015-89fd-412e-9533-cfe88d3d6cb5"
-          (reference "#PWR056") (unit 1)
-        )
-      )
-    )
-  )
-  (symbol (lib_id "power:+5V") (at 25.4 50.8 0) (unit 1)
-    (in_bom yes) (on_board yes) (dnp no) (fields_autoplaced)
-    (property "Reference" "#PWR055" (at 25.4 54.61 0)
-      (effects (font (size 1.27 1.27)) hide)
-    )
-    (property "Value" "+5V" (at 25.4 45.72 0)
-      (effects (font (size 1.27 1.27)))
-    )
-    (property "Footprint" "" (at 25.4 50.8 0)
-      (effects (font (size 1.27 1.27)) hide)
-    )
-    (property "Datasheet" "" (at 25.4 50.8 0)
-      (effects (font (size 1.27 1.27)) hide)
-    )
-    (pin "1")
-    (instances
-      (project "H2 Sensor Board Lucy Rev 1"
-        (path "/61fdd4a1-2d1e-44dc-8644-252e12d35745/59a3a015-89fd-412e-9533-cfe88d3d6cb5"
-          (reference "#PWR055") (unit 1)
-        )
-      )
-    )
-  )
-  (symbol (lib_id "Diode:BAT54C") (at 35.56 52.07 0) (unit 1)
-    (in_bom yes) (on_board yes) (dnp no) (fields_autoplaced)
-    (property "Reference" "D11" (at 35.56 45.72 0)
-      (effects (font (size 1.27 1.27)))
-    )
-    (property "Value" "BAT54C" (at 35.56 48.26 0)
-      (effects (font (size 1.27 1.27)))
-    )
-    (property "Footprint" "Package_TO_SOT_SMD:SOT-23" (at 37.465 48.895 0)
-      (effects (font (size 1.27 1.27)) (justify left) hide)
-    )
-    (property "Datasheet" "http://www.diodes.com/_files/datasheets/ds11005.pdf" (at 33.528 52.07 0)
-      (effects (font (size 1.27 1.27)) hide)
-    )
-    (pin "1")
-    (pin "2")
-    (pin "3")
-    (instances
-      (project "H2 Sensor Board Lucy Rev 1"
-        (path "/61fdd4a1-2d1e-44dc-8644-252e12d35745/59a3a015-89fd-412e-9533-cfe88d3d6cb5"
-          (reference "D11") (unit 1)
-        )
-      )
-    )
-  )
-  (symbol (lib_id "H2_Parts:H2_Simon_Sensor_Breakout") (at 68.58 73.66 0) (unit 1)
-    (in_bom yes) (on_board yes) (dnp no) (fields_autoplaced)
-    (property "Reference" "U10" (at 68.58 58.42 0)
-      (effects (font (size 1.27 1.27)))
-    )
-    (property "Value" "~" (at 68.58 73.66 0)
-      (effects (font (size 1.27 1.27)))
-    )
-    (property "Footprint" "" (at 68.58 73.66 0)
-      (effects (font (size 1.27 1.27)) hide)
-    )
-    (property "Datasheet" "" (at 68.58 73.66 0)
-      (effects (font (size 1.27 1.27)) hide)
-    )
-    (pin "1")
-    (pin "2")
-    (pin "3")
-    (instances
-      (project "H2 Sensor Board Lucy Rev 1"
-        (path "/61fdd4a1-2d1e-44dc-8644-252e12d35745/59a3a015-89fd-412e-9533-cfe88d3d6cb5"
-          (reference "U10") (unit 1)
-        )
-      )
-    )
-  )
 )

Commit message: Added Simon board and eddited the dimentions
Parts:
- added D11: BAT54C, Package_TO_SOT_SMD:SOT-23, symbol Diode:BAT54C
- added U10: ~, symbol H2_Parts:H2_Simon_Sensor_Breakout
Connections:
- new net: D11.3, U10.3 (V_HEAT)
- new net +5V: D11.1
- new net GND: U10.1 (GND)
- new net VBAT_5V: D11.2
- new net V_SENSE: U10.2 (V_SENSE)
Changed lines of the file:
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@@
 (kicad_sch (version 20230121) (generator eeschema)
   (paper "A4")
+  (wire (pts (xy 35.56 73.66) (xy 53.34 73.66))
+    (stroke (width 0) (type default))
+  )
+  (wire (pts (xy 25.4 52.07) (xy 27.94 52.07))
+    (stroke (width 0) (type default))
+  )
+  (wire (pts (xy 35.56 57.15) (xy 35.56 73.66))
+    (stroke (width 0) (type default))
+  )
+  (wire (pts (xy 88.9 73.66) (xy 83.82 73.66))
+    (stroke (width 0) (type default))
+  )
+  (wire (pts (xy 25.4 50.8) (xy 25.4 52.07))
+    (stroke (width 0) (type default))
+  )
+  (global_label "VBAT_5V" (shape input) (at 43.18 52.07 0) (fields_autoplaced)
+    (effects (font (size 1.27 1.27)) (justify left))
+    (property "Intersheetrefs" "${INTERSHEET_REFS}" (at 53.8457 52.07 0)
+      (effects (font (size 1.27 1.27)) (justify left) hide)
+    )
+  )
+  (global_label "V_SENSE" (shape input) (at 88.9 73.66 0) (fields_autoplaced)
+    (effects (font (size 1.27 1.27)) (justify left))
+    (property "Intersheetrefs" "${INTERSHEET_REFS}" (at 99.9889 73.66 0)
+      (effects (font (size 1.27 1.27)) (justify left) hide)
+    )
+  )
+  (symbol (lib_id "power:GND") (at 68.58 88.9 0) (unit 1)
+    (in_bom yes) (on_board yes) (dnp no) (fields_autoplaced)
+    (property "Reference" "#PWR056" (at 68.58 95.25 0)
+      (effects (font (size 1.27 1.27)) hide)
+    )
+    (property "Value" "GND" (at 68.58 93.98 0)
+      (effects (font (size 1.27 1.27)))
+    )
+    (property "Footprint" "" (at 68.58 88.9 0)
+      (effects (font (size 1.27 1.27)) hide)
+    )
+    (property "Datasheet" "" (at 68.58 88.9 0)
+      (effects (font (size 1.27 1.27)) hide)
+    )
+    (pin "1")
+    (instances
+      (project "H2 Sensor Board Lucy Rev 1"
+        (path "/61fdd4a1-2d1e-44dc-8644-252e12d35745/59a3a015-89fd-412e-9533-cfe88d3d6cb5"
+          (reference "#PWR056") (unit 1)
+        )
+      )
+    )
+  )
+  (symbol (lib_id "power:+5V") (at 25.4 50.8 0) (unit 1)
+    (in_bom yes) (on_board yes) (dnp no) (fields_autoplaced)
+    (property "Reference" "#PWR055" (at 25.4 54.61 0)
+      (effects (font (size 1.27 1.27)) hide)
+    )
+    (property "Value" "+5V" (at 25.4 45.72 0)
+      (effects (font (size 1.27 1.27)))
+    )
+    (property "Footprint" "" (at 25.4 50.8 0)
+      (effects (font (size 1.27 1.27)) hide)
+    )
+    (property "Datasheet" "" (at 25.4 50.8 0)
+      (effects (font (size 1.27 1.27)) hide)
+    )
+    (pin "1")
+    (instances
+      (project "H2 Sensor Board Lucy Rev 1"
+        (path "/61fdd4a1-2d1e-44dc-8644-252e12d35745/59a3a015-89fd-412e-9533-cfe88d3d6cb5"
+          (reference "#PWR055") (unit 1)
+        )
+      )
+    )
+  )
+  (symbol (lib_id "Diode:BAT54C") (at 35.56 52.07 0) (unit 1)
+    (in_bom yes) (on_board yes) (dnp no) (fields_autoplaced)
+    (property "Reference" "D11" (at 35.56 45.72 0)
+      (effects (font (size 1.27 1.27)))
+    )
+    (property "Value" "BAT54C" (at 35.56 48.26 0)
+      (effects (font (size 1.27 1.27)))
+    )
+    (property "Footprint" "Package_TO_SOT_SMD:SOT-23" (at 37.465 48.895 0)
+      (effects (font (size 1.27 1.27)) (justify left) hide)
+    )
+    (property "Datasheet" "http://www.diodes.com/_files/datasheets/ds11005.pdf" (at 33.528 52.07 0)
+      (effects (font (size 1.27 1.27)) hide)
+    )
+    (pin "1")
+    (pin "2")
+    (pin "3")
+    (instances
+      (project "H2 Sensor Board Lucy Rev 1"
+        (path "/61fdd4a1-2d1e-44dc-8644-252e12d35745/59a3a015-89fd-412e-9533-cfe88d3d6cb5"
+          (reference "D11") (unit 1)
+        )
+      )
+    )
+  )
+  (symbol (lib_id "H2_Parts:H2_Simon_Sensor_Breakout") (at 68.58 73.66 0) (unit 1)
+    (in_bom yes) (on_board yes) (dnp no) (fields_autoplaced)
+    (property "Reference" "U10" (at 68.58 58.42 0)
+      (effects (font (size 1.27 1.27)))
+    )
+    (property "Value" "~" (at 68.58 73.66 0)
+      (effects (font (size 1.27 1.27)))
+    )
+    (property "Footprint" "" (at 68.58 73.66 0)
+      (effects (font (size 1.27 1.27)) hide)
+    )
+    (property "Datasheet" "" (at 68.58 73.66 0)
+      (effects (font (size 1.27 1.27)) hide)
+    )
+    (pin "1")
+    (pin "2")
+    (pin "3")
+    (instances
+      (project "H2 Sensor Board Lucy Rev 1"
+        (path "/61fdd4a1-2d1e-44dc-8644-252e12d35745/59a3a015-89fd-412e-9533-cfe88d3d6cb5"
+          (reference "U10") (unit 1)
+        )
+      )
+    )
+  )
 )
