File: H2-Sensor-Board2022_Lucy/H2 Sensor Board Lucy Rev 1/H2_Sensor.kicad_sch (KiCad schematic)
At the start: 4 parts, among them J3 Conn_01x03_Socket

Commit message: Update some Telem
Parts:
- added C1: 100n, Capacitor_SMD:C_0402_1005Metric, symbol Device:C
- added SW2: TARE, Button_Switch_SMD:SW_SPST_PTS810, symbol Switch:SW_Push
Connections:
- net GND: now also C1.1, SW2.1
- new net TARE: C1.2, SW2.2
Changed lines of the file:
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@@
   (junction (at 112.776 41.91) (diameter 0) (color 0 0 0 0)
   )
+  (junction (at 39.878 84.074) (diameter 0) (color 0 0 0 0)
+  )
+  (junction (at 25.908 90.424) (diameter 0) (color 0 0 0 0)
+  )
   (wire (pts (xy 40.64 36.83) (xy 45.72 36.83))
     (stroke (width 0) (type default))
@@
     (stroke (width 0) (type default))
   )
+  (wire (pts (xy 38.608 84.074) (xy 39.878 84.074))
+    (stroke (width 0) (type default))
+  )
   (wire (pts (xy 59.69 44.45) (xy 59.69 66.04))
     (stroke (width 0) (type default))
   )
+  (wire (pts (xy 39.878 84.074) (xy 52.832 84.074))
+    (stroke (width 0) (type default))
+  )
   (wire (pts (xy 45.72 31.75) (xy 45.72 36.83))
     (stroke (width 0) (type default))
@@
     (stroke (width 0) (type default))
   )
+  (wire (pts (xy 39.878 84.074) (xy 39.878 90.424))
+    (stroke (width 0) (type default))
+  )
+  (wire (pts (xy 29.718 90.424) (xy 25.908 90.424))
+    (stroke (width 0) (type default))
+  )
   (wire (pts (xy 45.72 41.91) (xy 45.72 46.99))
     (stroke (width 0) (type default))
@@
     (stroke (width 0) (type default))
   )
+  (wire (pts (xy 25.908 90.424) (xy 25.908 92.964))
+    (stroke (width 0) (type default))
+  )
+  (wire (pts (xy 39.878 90.424) (xy 37.338 90.424))
+    (stroke (width 0) (type default))
+  )
   (wire (pts (xy 77.47 66.04) (xy 90.17 66.04))
     (stroke (width 0) (type default))
   )
+  (wire (pts (xy 25.908 84.074) (xy 25.908 90.424))
+    (stroke (width 0) (type default))
+  )
   (wire (pts (xy 68.58 44.45) (xy 59.69 44.45))
     (stroke (width 0) (type default))
+  )
+  (wire (pts (xy 28.448 84.074) (xy 25.908 84.074))
+    (stroke (width 0) (type default))
+  )
+  (label "TARE" (at 39.878 84.074 0) (fields_autoplaced)
+    (effects (font (size 1.27 1.27)) (justify left bottom))
   )
   (label "H2Conc" (at 58.42 39.37 0) (fields_autoplaced)
@@
     (effects (font (size 1.27 1.27)) (justify left bottom))
   )
-  (hierarchical_label "H2Conc_3.3V" (shape input) (at 136.398 41.91 0) (fields_autoplaced)
+  (hierarchical_label "H2Conc_3.3V" (shape output) (at 136.398 41.91 0) (fields_autoplaced)
     (effects (font (size 1.27 1.27)) (justify left))
   )
+  (hierarchical_label "TARE" (shape output) (at 52.832 84.074 0) (fields_autoplaced)
+    (effects (font (size 1.27 1.27)) (justify left))
+  )
   (symbol (lib_id "power:+5V") (at 45.72 31.75 0) (unit 1)
     (in_bom yes) (on_board yes) (dnp no) (fields_autoplaced)
@@
         (path "/61fdd4a1-2d1e-44dc-8644-252e12d35745/7173564b-4ce8-4fe4-9cf3-378e96487dfe"
           (reference "#PWR02") (unit 1)
+        )
+      )
+    )
+  )
+  (symbol (lib_id "power:GND") (at 25.908 92.964 0) (unit 1)
+    (in_bom yes) (on_board yes) (dnp no) (fields_autoplaced)
+    (property "Reference" "#PWR02" (at 25.908 99.314 0)
+      (effects (font (size 1.27 1.27)) hide)
+    )
+    (property "Value" "GND" (at 25.908 97.409 0)
+      (effects (font (size 1.27 1.27)) hide)
+    )
+    (property "Footprint" "" (at 25.908 92.964 0)
+      (effects (font (size 1.27 1.27)) hide)
+    )
+    (property "Datasheet" "" (at 25.908 92.964 0)
+      (effects (font (size 1.27 1.27)) hide)
+    )
+    (pin "1")
+    (instances
+      (project "CAN-USB RF Module"
+        (path "/05ffaa46-4df3-4c93-a015-882eb69d3f55"
+          (reference "#PWR02") (unit 1)
+        )
+      )
+      (project "H2 Sensor Board Lucy Rev 1"
+        (path "/61fdd4a1-2d1e-44dc-8644-252e12d35745"
+          (reference "#PWR041") (unit 1)
+        )
+        (path "/61fdd4a1-2d1e-44dc-8644-252e12d35745/7173564b-4ce8-4fe4-9cf3-378e96487dfe"
+          (reference "#PWR042") (unit 1)
         )
       )
@@
     )
   )
+  (symbol (lib_id "Switch:SW_Push") (at 33.528 84.074 0) (unit 1)
+    (in_bom yes) (on_board yes) (dnp no)
+    (property "Reference" "SW2" (at 33.528 86.614 0)
+      (effects (font (size 1.27 1.27)))
+    )
+    (property "Value" "TARE" (at 33.528 77.089 0)
+      (effects (font (size 1.27 1.27)))
+    )
+    (property "Footprint" "Button_Switch_SMD:SW_SPST_PTS810" (at 33.528 78.994 0)
+      (effects (font (size 1.27 1.27)) hide)
+    )
+    (property "Datasheet" "~" (at 33.528 78.994 0)
+      (effects (font (size 1.27 1.27)) hide)
+    )
+    (property "MPN" "" (at 33.528 84.074 0)
+      (effects (font (size 1.27 1.27)) hide)
+    )
+    (property "LCSC #" "C221896" (at 33.528 84.074 0)
+      (effects (font (size 1.27 1.27)) hide)
+    )
+    (pin "1")
+    (pin "2")
+    (instances
+      (project "CAN-USB RF Module"
+        (path "/05ffaa46-4df3-4c93-a015-882eb69d3f55"
+          (reference "SW2") (unit 1)
+        )
+      )
+      (project "H2 Sensor Board Lucy Rev 1"
+        (path "/61fdd4a1-2d1e-44dc-8644-252e12d35745"
+          (reference "SW2") (unit 1)
+        )
+        (path "/61fdd4a1-2d1e-44dc-8644-252e12d35745/7173564b-4ce8-4fe4-9cf3-378e96487dfe"
+          (reference "SW3") (unit 1)
+        )
+      )
+    )
+  )
   (symbol (lib_id "Device:R") (at 73.66 66.04 90) (unit 1)
     (in_bom yes) (on_board yes) (dnp no) (fields_autoplaced)
@@
         )
       )
+    )
+  )
+  (symbol (lib_id "Device:C") (at 33.528 90.424 90) (unit 1)
+    (in_bom yes) (on_board yes) (dnp no)
+    (property "Reference" "C1" (at 38.608 89.154 90)
+      (effects (font (size 1.27 1.27)) (justify left))
+    )
+    (property "Value" "100n" (at 36.068 94.234 90)
+      (effects (font (size 1.27 1.27)) (justify left))
+    )
+    (property "Footprint" "Capacitor_SMD:C_0402_1005Metric" (at 37.338 89.4588 0)
+      (effects (font (size 1.27 1.27)) hide)
+    )
+    (property "Datasheet" "~" (at 33.528 90.424 0)
+      (effects (font (size 1.27 1.27)) hide)
+    )
+    (property "Description" "100nF -20%,+80% 16V Y5V 0402 Multilayer Ceramic Capacitors MLCC - SMD/SMT RoHS" (at 33.528 90.424 0)
+      (effects (font (size 1.27 1.27)) hide)
+    )
+    (property "MPN" "" (at 33.528 90.424 0)
+      (effects (font (size 1.27 1.27)) hide)
+    )
+    (property "LCSC #" "C1525" (at 33.528 90.424 0)
+      (effects (font (size 1.27 1.27)) hide)
+    )
+    (pin "1")
+    (pin "2")
+    (instances
+      (project "CAN-USB RF Module"
+        (path "/05ffaa46-4df3-4c93-a015-882eb69d3f55"
+          (reference "C1") (unit 1)
+        )
+      )
+      (project "H2 Sensor Board Lucy Rev 1"
+        (path "/61fdd4a1-2d1e-44dc-8644-252e12d35745"
+          (reference "C2") (unit 1)
+        )
+        (path "/61fdd4a1-2d1e-44dc-8644-252e12d35745/7173564b-4ce8-4fe4-9cf3-378e96487dfe"
+          (reference "C3") (unit 1)
+        )
+      )

Commit message: Humiditiy sensor and other small cahnges
Parts:
- removed J3: Conn_01x03_Socket, symbol Connector:Conn_01x03_Socket
- removed R13: R, symbol Device:R
- added D11: BAT54C, Package_TO_SOT_SMD:SOT-23, symbol Diode:BAT54C
- added U10: ~, symbol H2_Parts:H2_Simon_Sensor_Breakout
Connections:
- net +5V: now also D11.1
- net GND: now also D5.2 (A), U10.1 (GND); no longer D5.1 (K)
- net H2Conc_3.3V: now also D5.1 (K), OP1.4 (-); no longer D5.2 (A)
- net H2Conc renamed V_SENSE
- net V_SENSE: now also U10.2 (V_SENSE)
- new net: D11.3, U10.3 (V_HEAT)
- new net VBAT_5V: D11.2
Other:
- moved on the sheet: D5
