File: H2-Sensor-Board2022_Lucy/H2 Sensor Board Lucy Rev 1/_autosave-Sensors.kicad_sch (KiCad schematic)
At the start: 17 parts, among them SW2 TARE, U11 AD8603, U9 BME280

Commit message: doN:
Parts:
- D5: value D_Zener -> MMSZ5226B-7-F; DK # (none) -> MMSZ5226B-FDICT-ND
Changed lines of the file:
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@@
       (effects (font (size 1.27 1.27)) (justify left))
     )
-    (property "Value" "D_Zener" (at 97.79 44.45 90)
+    (property "Value" "MMSZ5226B-7-F" (at 97.79 44.45 90)
       (effects (font (size 1.27 1.27)) (justify left))
     )
@@
       (effects (font (size 1.27 1.27)) hide)
     )
+    (property "DK #" "MMSZ5226B-FDICT-ND" (at 95.25 43.18 0)
+      (effects (font (size 1.27 1.27)) hide)
+    )
+    (property "Description" "MMSZ5226B-7-F" (at 95.25 43.18 0)
+      (effects (font (size 1.27 1.27)) hide)
+    )
