File: Batt-Power-Prototype-2023_Lucy_V1/untitled.kicad_sch (KiCad schematic)
At the start: 12 parts, among them U1 RPA60-2412SFW, U2 AP62250Z6

Commit message: changes from sat work session
Parts:
- removed U2: AP62250Z6, Package_TO_SOT_SMD:SOT-563, symbol Regulator_Switching:AP62250Z6
- added R3: 10, symbol Device:R
- added R4: 27, symbol Device:R
- C1: value C_Polarized -> 100u
- C2: value C -> 10u
- C3, C4: value C -> 6.8n
- F1: now not fitted
Connections:
- net -unfileredBattery: now reaches C1.2, D1.2 (A), FL1.1
- net DCDC-VIn: now reaches C2.1, C3.1, FL1.3, U1.1 (+VIN)
- net DCDC-VIn: now also R3.1
- net at C2.2, FL1.4, U1.2 (-VIN): now also C4.2; no longer C4.1
- net DCDC-CTRL: now reaches U1.3 (CTRL)
- net DCDC-CTRL: now also R3.2, R4.1
- net -12v: now reaches R2.2, U1.5 (-VOUT)
- net -12v: now also C4.1; no longer C4.2
- net +12v: now reaches C3.2, R1.1, U1.6 (+VOUT)
- net +unfileredBattery: now reaches F1.1
- new net GND: R4.2
Other:
- note added: "input: 18.5v output: 5v"
- moved on the sheet: C1, C2, C3, C4, D1, D2, FL1, R1, R2, U1
