File: Batt-Power-Prototype-2023_Lucy_V1/power.kicad_sch (KiCad schematic)
At the start: 62 parts, among them J1 Conn_01x02_Pin, U1 RPA60-2412SFW, U3 AZ1117IH-5.0, U5 AP62250Z6, U5 AZ1117-3.3

Commit message: pushing what ive done
Connections:
- net 12V Buck renamed 12V_Buck
- net 12V Unsensed renamed 12V_Unsensed
- net 12V out renamed 12V_out
- net 5V 1 renamed 5V_1
- net 5V 2 renamed 5V_2
- net 5V 3 renamed 5V_3
- net Battery Terminal 1 renamed Battery_Terminal_1
- net Battery Terminal 1 Unsensed renamed Battery_Terminal_1_Unsensed
- net Battery Terminal 2 renamed Battery_Terminal_2
- net DCDC-CTRL renamed DCDC_CTRL
- net DCDC-VIn renamed DCDC_VIn
Other:
- sheet Current & Voltage Senseing ports: added 12V_Buck, 12V_Unsensed, 12V_out, Battery_Terminal, Battery_Terminal_Unsensed; removed 12V Buck, 12V Unsensed, 12V out, Battery Terminal, Battery Terminal Unsensed
- sheet outputs ports: added 12V_out, 5V_1, 5V_2, 5V_3; removed 12V out, 5V 1, 5V 2, 5V 3
- moved on the sheet: C30
Changed lines of the file:
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@@
   (junction (at 191.77 120.65) (diameter 0) (color 0 0 0 0)
   )
-  (junction (at 119.38 158.75) (diameter 0) (color 0 0 0 0)
+  (junction (at 118.11 157.48) (diameter 0) (color 0 0 0 0)
   )
   (junction (at 238.76 95.25) (diameter 0) (color 0 0 0 0)
@@
     (stroke (width 0) (type default))
   )
-  (wire (pts (xy 87.63 153.67) (xy 93.98 153.67))
-    (stroke (width 0) (type default))
-  )
   (wire (pts (xy 105.41 93.98) (xy 99.06 93.98))
     (stroke (width 0) (type default))
@@
     (stroke (width 0) (type default))
   )
+  (wire (pts (xy 87.63 152.4) (xy 92.71 152.4))
+    (stroke (width 0) (type default))
+  )
   (wire (pts (xy 113.03 119.38) (xy 113.03 124.46))
     (stroke (width 0) (type default))
@@
     (stroke (width 0) (type default))
   )
-  (wire (pts (xy 119.38 158.75) (xy 125.73 158.75))
+  (wire (pts (xy 118.11 157.48) (xy 124.46 157.48))
     (stroke (width 0) (type default))
   )
@@
     (stroke (width 0) (type default))
   )
-  (wire (pts (xy 48.26 152.4) (xy 54.61 152.4))
+  (wire (pts (xy 48.26 151.13) (xy 54.61 151.13))
     (stroke (width 0) (type default))
   )
@@
     (stroke (width 0) (type default))
   )
-  (wire (pts (xy 87.63 161.29) (xy 93.98 161.29))
+  (wire (pts (xy 87.63 162.56) (xy 93.98 162.56))
     (stroke (width 0) (type default))
   )
@@
     (stroke (width 0) (type default))
   )
-  (wire (pts (xy 48.26 156.21) (xy 54.61 156.21))
-    (stroke (width 0) (type default))
-  )
-  (wire (pts (xy 87.63 158.75) (xy 119.38 158.75))
+  (wire (pts (xy 48.26 154.94) (xy 54.61 154.94))
     (stroke (width 0) (type default))
   )
@@
     (stroke (width 0) (type default))
   )
+  (wire (pts (xy 87.63 157.48) (xy 118.11 157.48))
+    (stroke (width 0) (type default))
+  )
   (wire (pts (xy 226.06 76.2) (xy 228.6 76.2))
     (stroke (width 0) (type default))
@@
     (effects (font (size 1.27 1.27)) (justify left bottom))
   )
-  (label "5V 1" (at 48.26 173.99 180) (fields_autoplaced)
+  (label "5V_1" (at 48.26 173.99 180) (fields_autoplaced)
     (effects (font (size 1.27 1.27)) (justify right bottom))
   )
-  (label "DCDC-VIn" (at 71.12 57.15 0) (fields_autoplaced)
+  (label "DCDC_VIn" (at 71.12 57.15 0) (fields_autoplaced)
     (effects (font (size 1.27 1.27)) (justify left bottom))
   )
-  (label "12V out" (at 48.26 185.42 180) (fields_autoplaced)
+  (label "12V_out" (at 48.26 185.42 180) (fields_autoplaced)
     (effects (font (size 1.27 1.27)) (justify right bottom))
   )
-  (label "Battery Terminal 1 Unsensed" (at 38.1 64.77 0) (fields_autoplaced)
+  (label "Battery_Terminal_1_Unsensed" (at 38.1 64.77 0) (fields_autoplaced)
     (effects (font (size 1.27 1.27)) (justify left bottom))
   )
-  (label "12V Buck" (at 180.34 29.21 0) (fields_autoplaced)
+  (label "12V_Buck" (at 180.34 29.21 0) (fields_autoplaced)
     (effects (font (size 1.27 1.27)) (justify left bottom))
   )
-  (label "Battery Terminal 1 Unsensed" (at 48.26 156.21 180) (fields_autoplaced)
+  (label "Battery_Terminal_1_Unsensed" (at 48.26 154.94 180) (fields_autoplaced)
     (effects (font (size 1.27 1.27)) (justify right bottom))
   )
-  (label "5V 1" (at 276.86 26.67 0) (fields_autoplaced)
+  (label "5V_1" (at 276.86 26.67 0) (fields_autoplaced)
     (effects (font (size 1.27 1.27)) (justify left bottom))
   )
-  (label "12V out" (at 125.73 158.75 0) (fields_autoplaced)
+  (label "12V_out" (at 124.46 157.48 0) (fields_autoplaced)
     (effects (font (size 1.27 1.27)) (justify left bottom))
   )
-  (label "5V 3" (at 48.26 181.61 180) (fields_autoplaced)
+  (label "5V_3" (at 48.26 181.61 180) (fields_autoplaced)
     (effects (font (size 1.27 1.27)) (justify right bottom))
   )
-  (label "12V Buck" (at 134.62 91.44 0) (fields_autoplaced)
+  (label "12V_Buck" (at 134.62 91.44 0) (fields_autoplaced)
     (effects (font (size 1.27 1.27)) (justify left bottom))
   )
-  (label "DCDC-CTRL" (at 85.09 66.04 0) (fields_autoplaced)
+  (label "DCDC_CTRL" (at 85.09 66.04 0) (fields_autoplaced)
     (effects (font (size 1.27 1.27)) (justify left bottom))
   )
-  (label "Battery Terminal 1" (at 33.02 35.56 180) (fields_autoplaced)
+  (label "Battery_Terminal_1" (at 33.02 35.56 180) (fields_autoplaced)
     (effects (font (size 1.27 1.27)) (justify right bottom))
   )
-  (label "Battery Terminal 2" (at 38.1 67.31 0) (fields_autoplaced)
+  (label "Battery_Terminal_2" (at 38.1 67.31 0) (fields_autoplaced)
     (effects (font (size 1.27 1.27)) (justify left bottom))
   )
-  (label "5V 2" (at 48.26 177.8 180) (fields_autoplaced)
+  (label "5V_2" (at 48.26 177.8 180) (fields_autoplaced)
     (effects (font (size 1.27 1.27)) (justify right bottom))
   )
-  (label "5V 3" (at 275.59 116.84 0) (fields_autoplaced)
+  (label "5V_3" (at 275.59 116.84 0) (fields_autoplaced)
     (effects (font (size 1.27 1.27)) (justify left bottom))
   )
-  (label "12V Unsensed" (at 161.29 24.13 180) (fields_autoplaced)
+  (label "12V_Unsensed" (at 161.29 24.13 180) (fields_autoplaced)
     (effects (font (size 1.27 1.27)) (justify right bottom))
   )
-  (label "DCDC-CTRL" (at 116.84 40.64 180) (fields_autoplaced)
+  (label "DCDC_CTRL" (at 116.84 40.64 180) (fields_autoplaced)
     (effects (font (size 1.27 1.27)) (justify right bottom))
   )
-  (label "DCDC-VIn" (at 111.76 33.02 0) (fields_autoplaced)
+  (label "DCDC_VIn" (at 111.76 33.02 0) (fields_autoplaced)
     (effects (font (size 1.27 1.27)) (justify left bottom))
   )
-  (label "12V Buck" (at 93.98 161.29 0) (fields_autoplaced)
+  (label "12V_Buck" (at 93.98 162.56 0) (fields_autoplaced)
     (effects (font (size 1.27 1.27)) (justify left bottom))
   )
-  (label "5V 2" (at 275.59 72.39 0) (fields_autoplaced)
+  (label "5V_2" (at 275.59 72.39 0) (fields_autoplaced)
     (effects (font (size 1.27 1.27)) (justify left bottom))
   )
-  (label "Battery Terminal 1" (at 93.98 153.67 0) (fields_autoplaced)
+  (label "Battery_Terminal_1" (at 92.71 152.4 0) (fields_autoplaced)
     (effects (font (size 1.27 1.27)) (justify left bottom))
   )
-  (label "12V Unsensed" (at 48.26 152.4 180) (fields_autoplaced)
+  (label "12V_Unsensed" (at 48.26 151.13 180) (fields_autoplaced)
     (effects (font (size 1.27 1.27)) (justify right bottom))
   )
-  (label "Battery Terminal 2" (at 33.02 45.72 180) (fields_autoplaced)
+  (label "Battery_Terminal_2" (at 33.02 45.72 180) (fields_autoplaced)
     (effects (font (size 1.27 1.27)) (justify right bottom))
   )
@@
     )
   )
-  (symbol (lib_id "power:GND") (at 119.38 166.37 0) (unit 1)
+  (symbol (lib_id "power:GND") (at 118.11 165.1 0) (unit 1)
     (in_bom yes) (on_board yes) (dnp no) (fields_autoplaced)
-    (property "Reference" "#PWR057" (at 119.38 172.72 0)
+    (property "Reference" "#PWR057" (at 118.11 171.45 0)
       (effects (font (size 1.27 1.27)) hide)
     )
-    (property "Value" "GND" (at 119.38 171.45 0)
+    (property "Value" "GND" (at 118.11 170.18 0)
       (effects (font (size 1.27 1.27)))
     )
-    (property "Footprint" "" (at 119.38 166.37 0)
+    (property "Footprint" "" (at 118.11 165.1 0)
       (effects (font (size 1.27 1.27)) hide)
     )
-    (property "Datasheet" "" (at 119.38 166.37 0)
+    (property "Datasheet" "" (at 118.11 165.1 0)
       (effects (font (size 1.27 1.27)) hide)
     )
@@
     )
   )
-  (symbol (lib_id "Device:C_Polarized") (at 119.38 162.56 0) (unit 1)
+  (symbol (lib_id "Device:C_Polarized") (at 118.11 161.29 0) (unit 1)
     (in_bom yes) (on_board yes) (dnp no) (fields_autoplaced)
-    (property "Reference" "C30" (at 123.19 160.401 0)
+    (property "Reference" "C30" (at 121.92 159.131 0)
       (effects (font (size 1.27 1.27)) (justify left))
     )
-    (property "Value" "1m" (at 123.19 162.941 0)
+    (property "Value" "1m" (at 121.92 161.671 0)
       (effects (font (size 1.27 1.27)) (justify left))
     )
-    (property "Footprint" "" (at 120.3452 166.37 0)
+    (property "Footprint" "" (at 119.0752 165.1 0)
       (effects (font (size 1.27 1.27)) hide)
     )
-    (property "Datasheet" "~" (at 119.38 162.56 0)
+    (property "Datasheet" "~" (at 118.11 161.29 0)
       (effects (font (size 1.27 1.27)) hide)
     )
@@
       (effects (font (size 1.27 1.27)) (justify left top))
     )
-    (pin "5V 1" input (at 54.61 173.99 180)
+    (pin "12V_out" input (at 54.61 185.42 180)
       (effects (font (size 1.27 1.27)) (justify left))
     )
-    (pin "12V out" input (at 54.61 185.42 180)
+    (pin "5V_3" input (at 54.61 181.61 180)
       (effects (font (size 1.27 1.27)) (justify left))
     )
-    (pin "5V 2" input (at 54.61 177.8 180)
+    (pin "5V_2" input (at 54.61 177.8 180)
       (effects (font (size 1.27 1.27)) (justify left))
     )
-    (pin "5V 3" input (at 54.61 181.61 180)
+    (pin "5V_1" input (at 54.61 173.99 180)
       (effects (font (size 1.27 1.27)) (justify left))
     )
@@
       (effects (font (size 1.27 1.27)) (justify left top))
     )
-    (pin "12V Unsensed" input (at 54.61 152.4 180)
-      (effects (font (size 1.27 1.27)) (justify left))
+    (pin "12V_Buck" input (at 87.63 162.56 0)
+      (effects (font (size 1.27 1.27)) (justify right))
     )
-    (pin "Battery Terminal Unsensed" input (at 54.61 156.21 180)
+    (pin "12V_Unsensed" input (at 54.61 151.13 180)
       (effects (font (size 1.27 1.27)) (justify left))
     )
-    (pin "Battery Terminal" input (at 87.63 153.67 0)
+    (pin "12V_out" input (at 87.63 157.48 0)
       (effects (font (size 1.27 1.27)) (justify right))
     )
-    (pin "12V out" input (at 87.63 158.75 0)
-      (effects (font (size 1.27 1.27)) (justify right))
+    (pin "Battery_Terminal_Unsensed" input (at 54.61 154.94 180)
+      (effects (font (size 1.27 1.27)) (justify left))
     )
-    (pin "12V Buck" input (at 87.63 161.29 0)
+    (pin "Battery_Terminal" input (at 87.63 152.4 0)
       (effects (font (size 1.27 1.27)) (justify right))
     )

Commit message: UPdated capacitor ftp and something else dont remember
Parts:
- removed D1: D_Zener, symbol Device:D_Zener
- added JP2: SolderJumper_2_Open, symbol Jumper:SolderJumper_2_Open
- C1: footprint (none) -> Capacitor_THT:CP_Radial_D8.0mm_P3.50mm
- D21: footprint (none) -> Diode_SMD:D_SMC
Connections:
- net GND: now also JP2.1 (A)
- net at C2.2, C4.2, FL1.4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: now also JP2.2 (B)
Other:
- moved on the sheet: D21
Changed lines of the file:
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@@
   (junction (at 243.84 30.48) (diameter 0) (color 0 0 0 0)
   )
+  (junction (at 55.88 45.72) (diameter 0) (color 0 0 0 0)
+  )
   (junction (at 62.23 101.6) (diameter 0) (color 0 0 0 0)
   )
@@
   (junction (at 180.34 30.48) (diameter 0) (color 0 0 0 0)
   )
-  (junction (at 62.23 45.72) (diameter 0) (color 0 0 0 0)
-  )
   (junction (at 274.32 76.2) (diameter 0) (color 0 0 0 0)
   )
@@
   (junction (at 148.59 25.4) (diameter 0) (color 0 0 0 0)
   )
-  (junction (at 62.23 35.56) (diameter 0) (color 0 0 0 0)
-  )
   (junction (at 158.75 54.61) (diameter 0) (color 0 0 0 0)
   )
@@
   (junction (at 191.77 76.2) (diameter 0) (color 0 0 0 0)
   )
+  (junction (at 55.88 35.56) (diameter 0) (color 0 0 0 0)
+  )
   (junction (at 237.49 30.48) (diameter 0) (color 0 0 0 0)
   )
+  (junction (at 102.87 54.61) (diameter 0) (color 0 0 0 0)
+  )
   (junction (at 49.53 45.72) (diameter 0) (color 0 0 0 0)
   )
@@
     (stroke (width 0) (type default))
   )
-  (wire (pts (xy 62.23 35.56) (xy 62.23 36.83))
+  (wire (pts (xy 55.88 35.56) (xy 55.88 36.83))
     (stroke (width 0) (type default))
   )
@@
     (stroke (width 0) (type default))
   )
-  (wire (pts (xy 49.53 45.72) (xy 62.23 45.72))
+  (wire (pts (xy 49.53 45.72) (xy 55.88 45.72))
     (stroke (width 0) (type default))
   )
@@
     (stroke (width 0) (type default))
   )
-  (wire (pts (xy 49.53 35.56) (xy 62.23 35.56))
+  (wire (pts (xy 49.53 35.56) (xy 55.88 35.56))
     (stroke (width 0) (type default))
   )
@@
     (stroke (width 0) (type default))
   )
+  (wire (pts (xy 55.88 45.72) (xy 74.93 45.72))
+    (stroke (width 0) (type default))
+  )
   (wire (pts (xy 237.49 30.48) (xy 243.84 30.48))
     (stroke (width 0) (type default))
@@
     (stroke (width 0) (type default))
   )
+  (wire (pts (xy 55.88 35.56) (xy 64.77 35.56))
+    (stroke (width 0) (type default))
+  )
   (wire (pts (xy 105.41 91.44) (xy 105.41 93.98))
     (stroke (width 0) (type default))
@@
     (stroke (width 0) (type default))
   )
+  (wire (pts (xy 102.87 54.61) (xy 102.87 55.88))
+    (stroke (width 0) (type default))
+  )
   (wire (pts (xy 255.27 76.2) (xy 265.43 76.2))
     (stroke (width 0) (type default))
@@
     (stroke (width 0) (type default))
   )
-  (wire (pts (xy 62.23 44.45) (xy 62.23 45.72))
+  (wire (pts (xy 55.88 44.45) (xy 55.88 45.72))
     (stroke (width 0) (type default))
   )
@@
     (stroke (width 0) (type default))
   )
+  (wire (pts (xy 102.87 63.5) (xy 102.87 64.77))
+    (stroke (width 0) (type default))
+  )
   (wire (pts (xy 255.27 120.65) (xy 255.27 124.46))
     (stroke (width 0) (type default))
@@
     (stroke (width 0) (type default))
   )
-  (wire (pts (xy 62.23 45.72) (xy 74.93 45.72))
-    (stroke (width 0) (type default))
-  )
   (wire (pts (xy 48.26 177.8) (xy 54.61 177.8))
     (stroke (width 0) (type default))
@@
     (stroke (width 0) (type default))
   )
-  (wire (pts (xy 62.23 35.56) (xy 64.77 35.56))
-    (stroke (width 0) (type default))
-  )
   (wire (pts (xy 148.59 48.26) (xy 148.59 54.61))
     (stroke (width 0) (type default))
@@
     )
   )
-  (symbol (lib_id "Device:D_Zener") (at 49.53 40.64 270) (unit 1)
-    (in_bom yes) (on_board yes) (dnp no) (fields_autoplaced)
-    (property "Reference" "D1" (at 52.07 39.37 90)
-      (effects (font (size 1.27 1.27)) (justify left))
-    )
-    (property "Value" "D_Zener" (at 52.07 41.91 90)
-      (effects (font (size 1.27 1.27)) (justify left))
-    )
-    (property "Footprint" "" (at 49.53 40.64 0)
-      (effects (font (size 1.27 1.27)) hide)
-    )
-    (property "Datasheet" "~" (at 49.53 40.64 0)
-      (effects (font (size 1.27 1.27)) hide)
-    )
-    (pin "1")
-    (pin "2")
-    (instances
-      (project "Batt-Power-Prototype-2023_Lucy_V1"
-        (path "/c58627b7-5b67-4b57-b29b-cc34a75a9096/caf32978-5421-40df-803f-f9402117c79f"
-          (reference "D1") (unit 1)
-        )
-      )
-    )
-  )
   (symbol (lib_id "Device:C_Polarized") (at 99.06 101.6 0) (mirror y) (unit 1)
     (in_bom yes) (on_board yes) (dnp no)
@@
     )
   )
+  (symbol (lib_id "Jumper:SolderJumper_2_Open") (at 102.87 59.69 90) (unit 1)
+    (in_bom yes) (on_board yes) (dnp no) (fields_autoplaced)
+    (property "Reference" "JP2" (at 105.41 58.42 90)
+      (effects (font (size 1.27 1.27)) (justify right))
+    )
+    (property "Value" "SolderJumper_2_Open" (at 105.41 60.96 90)
+      (effects (font (size 1.27 1.27)) (justify right))
+    )
+    (property "Footprint" "" (at 102.87 59.69 0)
+      (effects (font (size 1.27 1.27)) hide)
+    )
+    (property "Datasheet" "~" (at 102.87 59.69 0)
+      (effects (font (size 1.27 1.27)) hide)
+    )
+    (pin "2")
+    (pin "1")
+    (instances
+      (project "Batt-Power-Prototype-2023_Lucy_V1"
+        (path "/c58627b7-5b67-4b57-b29b-cc34a75a9096/caf32978-5421-40df-803f-f9402117c79f"
+          (reference "JP2") (unit 1)
+        )
+      )
+    )
+  )
   (symbol (lib_id "Device:L") (at 232.41 76.2 90) (unit 1)
     (in_bom yes) (on_board yes) (dnp no) (fields_autoplaced)
@@
     )
   )
-  (symbol (lib_id "Device:D") (at 62.23 40.64 270) (unit 1)
+  (symbol (lib_id "Device:D") (at 55.88 40.64 270) (unit 1)
     (in_bom yes) (on_board yes) (dnp no) (fields_autoplaced)
-    (property "Reference" "D21" (at 64.77 39.37 90)
+    (property "Reference" "D21" (at 58.42 39.37 90)
       (effects (font (size 1.27 1.27)) (justify left))
     )
-    (property "Value" "S10ML-TP" (at 64.77 41.91 90)
+    (property "Value" "S10ML-TP" (at 58.42 41.91 90)
       (effects (font (size 1.27 1.27)) (justify left))
     )
-    (property "Footprint" "" (at 62.23 40.64 0)
-      (effects (font (size 1.27 1.27)) hide)
-    )
-    (property "Datasheet" "~" (at 62.23 40.64 0)
-      (effects (font (size 1.27 1.27)) hide)
-    )
-    (property "Sim.Device" "D" (at 62.23 40.64 0)
+    (property "Footprint" "Diode_SMD:D_SMC" (at 55.88 40.64 0)
       (effects (font (size 1.27 1.27)) hide)
     )
-    (property "Sim.Pins" "1=K 2=A" (at 62.23 40.64 0)
+    (property "Datasheet" "https://www.mccsemi.com/pdf/Products/S10AL-S10ML(SMC).pdf" (at 55.88 40.64 0)
       (effects (font (size 1.27 1.27)) hide)
     )
@@
   )
   (symbol (lib_id "Regulator_Switching:AP62250Z6") (at 205.74 78.74 0) (unit 1)
-    (in_bom yes) (on_board yes) (dnp no) (fields_autoplaced)
+    (in_bom yes) (on_board yes) (dnp no)
     (property "Reference" "U5" (at 205.74 68.58 0)
       (effects (font (size 1.27 1.27)))
@@
     )
   )
+  (symbol (lib_id "power:GND") (at 102.87 64.77 0) (unit 1)
+    (in_bom yes) (on_board yes) (dnp no) (fields_autoplaced)
+    (property "Reference" "#PWR0110" (at 102.87 71.12 0)
+      (effects (font (size 1.27 1.27)) hide)
+    )
+    (property "Value" "GND" (at 102.87 69.85 0)
+      (effects (font (size 1.27 1.27)))
+    )
+    (property "Footprint" "" (at 102.87 64.77 0)
+      (effects (font (size 1.27 1.27)) hide)
+    )
+    (property "Datasheet" "" (at 102.87 64.77 0)
+      (effects (font (size 1.27 1.27)) hide)
+    )
+    (pin "1")
+    (instances
+      (project "Batt-Power-Prototype-2023_Lucy_V1"
+        (path "/c58627b7-5b67-4b57-b29b-cc34a75a9096/caf32978-5421-40df-803f-f9402117c79f"
+          (reference "#PWR0110") (unit 1)
+        )
+      )
+    )
+  )
   (symbol (lib_id "Regulator_Switching:AP62250Z6") (at 204.47 33.02 0) (unit 1)
     (in_bom yes) (on_board yes) (dnp no) (fields_autoplaced)
@@
   )
   (symbol (lib_id "Device:C") (at 129.54 54.61 270) (unit 1)
-    (in_bom yes) (on_board yes) (dnp no) (fields_autoplaced)
-    (property "Reference" "C4" (at 129.54 46.99 90)
+    (in_bom yes) (on_board yes) (dnp no)
+    (property "Reference" "C4" (at 129.54 58.42 90)
       (effects (font (size 1.27 1.27)))
     )
-    (property "Value" "6.8n" (at 129.54 49.53 90)
+    (property "Value" "6.8n" (at 129.54 60.96 90)
       (effects (font (size 1.27 1.27)))
     )
@@
       (effects (font (size 1.27 1.27)) (justify left))
     )
-    (property "Footprint" "" (at 75.8952 44.45 0)
+    (property "Footprint" "Capacitor_THT:CP_Radial_D8.0mm_P3.50mm" (at 75.8952 44.45 0)
       (effects (font (size 1.27 1.27)) hide)
     )
