File: Batt-Power-Prototype-2023_Lucy_V1/CVsense.kicad_sch (KiCad schematic)
At the start: 29 parts, among them U13 TSV912IDT, U14 TSV912IDT, U15 TSV912IDT

Commit message: as
Connections:
- net ADC_12V_Voltage_Out: now also U13.6 (-), U13.7; no longer U14.6 (-), U14.7
- net ADC_Battery_Voltage: now also U14.6 (-), U14.7; no longer U13.6 (-), U13.7
- net at C43.1, D?.1 (K), R?.1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: now also U14.5 (+); no longer U13.5 (+)
- net at C42.1, D?.1 (K), R?.1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: now also U13.5 (+); no longer U14.5 (+)
Other:
- note added: "@NOTE: The Power Indicator LEDs are before sensing and I am designing them to be only drawing a fixed 3 mA therefore they do not need to be in the current sense loop. - Abinash"
- moved on the sheet: U13B, U14B
Changed lines of the file:
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@@
   (junction (at 261.62 29.21) (diameter 0) (color 0 0 0 0)
   )
+  (junction (at 109.22 158.75) (diameter 0) (color 0 0 0 0)
+  )
   (junction (at 105.41 128.27) (diameter 0) (color 0 0 0 0)
   )
+  (junction (at 104.14 73.66) (diameter 0) (color 0 0 0 0)
+  )
   (junction (at 71.12 125.73) (diameter 0) (color 0 0 0 0)
   )
@@
   (junction (at 72.39 156.21) (diameter 0) (color 0 0 0 0)
   )
-  (junction (at 109.22 158.75) (diameter 0) (color 0 0 0 0)
-  )
   (junction (at 74.93 71.12) (diameter 0) (color 0 0 0 0)
   )
@@
   (junction (at 53.34 116.84) (diameter 0) (color 0 0 0 0)
   )
-  (junction (at 104.14 73.66) (diameter 0) (color 0 0 0 0)
-  )
   (junction (at 222.25 29.21) (diameter 0) (color 0 0 0 0)
   )
@@
     (stroke (width 0) (type default))
   )
-  (wire (pts (xy 233.68 96.52) (xy 233.68 100.33))
+  (wire (pts (xy 232.41 96.52) (xy 232.41 100.33))
     (stroke (width 0) (type default))
   )
@@
     (stroke (width 0) (type default))
   )
-  (wire (pts (xy 233.68 100.33) (xy 248.92 100.33))
+  (wire (pts (xy 232.41 100.33) (xy 248.92 100.33))
     (stroke (width 0) (type default))
   )
@@
   )
   (wire (pts (xy 109.22 158.75) (xy 114.3 158.75))
+    (stroke (width 0) (type default))
+  )
+  (wire (pts (xy 232.41 96.52) (xy 233.68 96.52))
     (stroke (width 0) (type default))
   )
@@
     (effects (font (size 1.27 1.27)) (justify left bottom))
   )
+  (text "@NOTE: The Power Indicator LEDs are before sensing and I am designing them to be only drawing a fixed 3 mA\n therefore they do not need to be in the current sense loop.\n- Abinash "
+    (at 13.97 193.04 0)
+    (effects (font (size 1.27 1.27)) (justify left bottom))
+  )
   (label "u11_unused" (at 247.65 36.83 90) (fields_autoplaced)
     (effects (font (size 1.27 1.27)) (justify left bottom))
@@
     )
   )
-  (symbol (lib_id "Amplifier_Operational:TSV912IDT") (at 101.6 158.75 0) (unit 2)
-    (in_bom yes) (on_board yes) (dnp no) (fields_autoplaced)
-    (property "Reference" "U14" (at 101.6 148.59 0)
-      (effects (font (size 1.27 1.27)))
-    )
-    (property "Value" "TSV912IDT" (at 101.6 151.13 0)
-      (effects (font (size 1.27 1.27)))
-    )
-    (property "Footprint" "BP_FTP:SO8_STM" (at 101.6 158.75 0)
-      (effects (font (size 1.27 1.27)) hide)
-    )
-    (property "Datasheet" "www.st.com/resource/en/datasheet/tsv911.pdf" (at 101.6 158.75 0)
-      (effects (font (size 1.27 1.27)) hide)
-    )
-    (property "Digikey #" "497-8165-2-ND" (at 101.6 158.75 0)
+  (symbol (lib_id "Amplifier_Operational:TSV912IDT") (at 96.52 73.66 0) (unit 2)
+    (in_bom yes) (on_board yes) (dnp no) (fields_autoplaced)
+    (property "Reference" "U14" (at 96.52 63.5 0)
+      (effects (font (size 1.27 1.27)))
+    )
+    (property "Value" "TSV912IDT" (at 96.52 66.04 0)
+      (effects (font (size 1.27 1.27)))
+    )
+    (property "Footprint" "BP_FTP:SO8_STM" (at 96.52 73.66 0)
+      (effects (font (size 1.27 1.27)) hide)
+    )
+    (property "Datasheet" "www.st.com/resource/en/datasheet/tsv911.pdf" (at 96.52 73.66 0)
+      (effects (font (size 1.27 1.27)) hide)
+    )
+    (property "Digikey #" "497-8165-2-ND" (at 96.52 73.66 0)
       (effects (font (size 1.27 1.27)) hide)
     )
@@
     )
   )
-  (symbol (lib_id "Amplifier_Operational:TSV912IDT") (at 96.52 73.66 0) (unit 2)
-    (in_bom yes) (on_board yes) (dnp no) (fields_autoplaced)
-    (property "Reference" "U13" (at 96.52 63.5 0)
-      (effects (font (size 1.27 1.27)))
-    )
-    (property "Value" "TSV912IDT" (at 96.52 66.04 0)
-      (effects (font (size 1.27 1.27)))
-    )
-    (property "Footprint" "BP_FTP:SO8_STM" (at 96.52 73.66 0)
-      (effects (font (size 1.27 1.27)) hide)
-    )
-    (property "Datasheet" "www.st.com/resource/en/datasheet/tsv911.pdf" (at 96.52 73.66 0)
-      (effects (font (size 1.27 1.27)) hide)
-    )
-    (property "Digikey #" "497-8165-2-ND" (at 96.52 73.66 0)
-      (effects (font (size 1.27 1.27)) hide)
-    )
+  (symbol (lib_id "Amplifier_Operational:TSV912IDT") (at 101.6 158.75 0) (unit 2)
+    (in_bom yes) (on_board yes) (dnp no) (fields_autoplaced)
+    (property "Reference" "U13" (at 101.6 148.59 0)
+      (effects (font (size 1.27 1.27)))
+    )
+    (property "Value" "TSV912IDT" (at 101.6 151.13 0)
+      (effects (font (size 1.27 1.27)))
+    )
+    (property "Footprint" "BP_FTP:SO8_STM" (at 101.6 158.75 0)
+      (effects (font (size 1.27 1.27)) hide)
+    )
+    (property "Datasheet" "www.st.com/resource/en/datasheet/tsv911.pdf" (at 101.6 158.75 0)
+      (effects (font (size 1.27 1.27)) hide)
+    )
+    (property "Digikey #" "497-8165-2-ND" (at 101.6 158.75 0)
+      (effects (font (size 1.27 1.27)) hide)
+    )

Commit message: j
Parts:
- added NT1: NetTie_2, NetTie:NetTie-2_THT_Pad0.3mm, symbol Device:NetTie_2
- C?: footprint Capacitor_SMD:C_0603_1608Metric -> Capacitor_SMD:C_0402_1005Metric
- R? (x4): footprint Resistor_SMD:R_0805_2012Metric -> Resistor_SMD:R_0603_1608Metric
Connections:
- net GND: now also NT1.2; no longer C42.2, C43.2, C?.2, C?.2, C?.2, D?.2 (A), D?.2 (A), D?.2 (A), D?.2 (A), D?.2 (A), D?.2 (A), R30.2, R?.2, R?.2, U13.4 (V-), U14.4 (V-), U15.4 (V-)
- new net GNDA: C42.2, C43.2, C?.2, C?.2, C?.2, D?.2 (A), D?.2 (A), D?.2 (A), D?.2 (A), D?.2 (A), D?.2 (A), NT1.1, R30.2, R?.2, R?.2, U13.4 (V-), U14.4 (V-), U15.4 (V-)
