File: Batt-Power-Prototype-2023_Lucy_V1/Batt-Power-Prototype-2023_Lucy_V1.kicad_pcb (KiCad board)
At the start: 2 copper layers, 100 x 100 mm, 155 parts, among them IC1 ESDALC6V1W5, J1 Conn_01x06_Pin, J10 STD_PWR_HEADER, J11 STD_PWR_HEADER, J12 STD_PWR_HEADER, J13 AMASS XT60-F Horizontal, J2 USB_B_Micro, J3 OLED, J4 DE9_Receptacle_MountingHoles, J5 GPIO, J6 AMASS XT60-F Vertical, J7 STD_PWR_HEADER, J8 STD_PWR_HEADER, J9 STD_PWR_HEADER, SW1 RESET, SW2 SW_SPDT, U1 8MHz, U10 AP62250Z6, U11 ACS723xLCTR-10AU, U12 ACS723xLCTR-10AU, U13 TSV912IDT, U14 TSV912IDT, U15 TSV912IDT, U16 ACS723xLCTR-10AU, U2 FT234XD-R, U3 STM32L432KCUx, U4 MCP2542FD-E/SN, U5 AZ1117-3.3, U6 AZ1117IH-5.0, U7 RPA60-2412SFW, U9 AP62250Z6

Commit message: a'
Parts:
- removed J13: AMASS XT60-F Horizontal, BP_FTP:AMASS_XT60PW-F
- removed NT1: NetTie_2, NetTie:NetTie-2_THT_Pad0.3mm
- removed needstobe50V1: 10u, BP_FTP:CAPC3225X270N
- added G***: LOGO, LOGO, F.Cu at (126.2, 117.8)
- added G***: LOGO, BP_FTP:BattBord, F.Cu at (371.5, 12.4)
- added H5: MountingHole_Pad, MountingHole:MountingHole_3.2mm_M3_Pad, F.Cu at (100.0, 64.0)
- added H6: MountingHole_Pad, MountingHole:MountingHole_3.2mm_M3_Pad, F.Cu at (190.0, 64.0)
- added H7: MountingHole_Pad, MountingHole:MountingHole_3.2mm_M3_Pad, F.Cu at (190.0, 154.0)
- added H8: MountingHole_Pad, MountingHole:MountingHole_3.2mm_M3_Pad, F.Cu at (100.0, 154.0)
- added JP3: POWER SEL, Jumper:SolderJumper-2_P1.3mm_Open_TrianglePad1.0x1.5mm, B.Cu at (107.1, 129.8)
- added JP4: POWER SEL, Jumper:SolderJumper-2_P1.3mm_Open_TrianglePad1.0x1.5mm, B.Cu at (107.0, 132.4)
- added L4: 10u, BP_FTP:CAPC3225X270N, B.Cu at (172.9, 101.7)
- added kibuzzard-65BDD721: G***, kibuzzard-65BDD721, F.Cu at (142.9, 123.5)
- added kibuzzard-65BDD72B: G***, kibuzzard-65BDD72B, F.Cu at (109.3, 123.5)
- added kibuzzard-65BDD733: G***, kibuzzard-65BDD733, F.Cu at (126.2, 123.5)
- added kibuzzard-65BDE858: G***, kibuzzard-65BDE858, B.Cu at (102.5, 129.8)
- added kibuzzard-65BDE861: G***, kibuzzard-65BDE861, B.Cu at (102.8, 132.4)
- added kibuzzard-65BDE8C6: G***, kibuzzard-65BDE8C6, B.Cu at (107.0, 127.3)
- C10, C11, C2, C9, D2, D9, R3, R4: moved to F.Cu
- C20, C23, D11, R12, U6: moved to B.Cu
- moved J5 75.4 mm to (97.2, 90.2)
- moved J1 62.7 mm to (99.8, 86.2)
- moved R20 45.7 mm to (141.9, 111.7), turned to 180 degrees
- moved R21 44.6 mm to (140.3, 110.2), turned to -90 degrees
- moved U10 42.6 mm to (141.9, 109.8), turned to -90 degrees
- moved C30 42.4 mm to (143.5, 110.2), turned to -90 degrees
- moved C17 41.2 mm to (108.3, 150.4), turned to 0 degrees
- moved C18 40.2 mm to (105.9, 151.1), turned to -90 degrees
- moved U7 39.1 mm to (166.1, 106.4), turned to 0 degrees
- moved D10 38.8 mm to (172.5, 78.8), turned to 90 degrees
- moved C53 38.4 mm to (142.1, 107.7), turned to 0 degrees
- moved R11 36.3 mm to (182.9, 112.2), turned to -90 degrees
- moved R10 36.0 mm to (179.6, 112.2), turned to 90 degrees
- moved L3 35.9 mm to (148.0, 107.8), turned to 90 degrees
- moved U5 35.3 mm to (108.3, 145.2), turned to 90 degrees
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Connections:
- C42 pad 2: GNDA -> GND
- C43 pad 2: GNDA -> GND
- C47 pad 2: GNDA -> GND
- C49 pad 2: GNDA -> GND
- C5 pad 1: +5V -> Net-(JP3-B)
- C50 pad 2: GNDA -> GND
- C7 pad 1: +5V -> Net-(JP3-B)
- D16 pad 2: GNDA -> GND
- D17 pad 2: GNDA -> GND
- D18 pad 2: GNDA -> GND
- D19 pad 2: GNDA -> GND
- D20 pad 2: GNDA -> GND
- D21 pad 2: GNDA -> GND
- R27 pad 2: GNDA -> GND
- R28 pad 2: GNDA -> GND
- R30 pad 2: GNDA -> GND
- U13 pad 4: GNDA -> GND
- U14 pad 4: GNDA -> GND
- U15 pad 4: GNDA -> GND
- U2 pad 4: +5V -> Net-(JP3-B)
Routing:
- net GND: track 227.5 -> 105.3 mm
- net +3V3: track 81.4 -> 20.7 mm, vias 5 -> 4
- net /Power/12V_Buck: track 10.5 -> 62.3 mm, vias 75 -> 40
- net /Battery_Curr: track 50.3 -> 0.00 mm, vias 4 -> 0
- net /ADC_Battery_Voltage: track 39.0 -> 0.00 mm, vias 2 -> 0
- net /12V_Current_Out: track 37.3 -> 0.00 mm, vias 4 -> 0
- net /Power/Battery_Terminal_2: track 37.1 -> 0.00 mm
- net /Power/12V_Unsensed: track 47.8 -> 18.4 mm, vias 0 -> 1
- net /ADC_12V_Voltage_Out: track 27.5 -> 0.00 mm, vias 2 -> 0
- net /12V_Current_Buck: track 26.8 -> 0.00 mm, vias 2 -> 0
- net Net-(D10-K): track 21.1 -> 0.00 mm, vias 0 -> 27
- net GNDA: track 21.0 -> 0.00 mm
- net /NRST: track 22.2 -> 2.60 mm
- net Net-(JP2-B): track 25.6 -> 6.12 mm
- net /Power/5V_2: track 0.00 -> 15.3 mm, vias 0 -> 2
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- added copper zone on B.Cu, net +3V3
- added copper zone on B.Cu, net +5V
- added copper zone on F.Cu, net /Power/Battery_Terminal_2
- added copper zone on B.Cu, net /Power/DCDC_V_{in}
- added copper zone on F.Cu, net /Power/outputs/5V_1
- added copper zone on F.Cu, net /Power/outputs/5V_2
- added copper zone on F.Cu, net /Power/outputs/5V_3
- added copper zone on F.Cu, net Net-(JP2-B)
- added copper zone on F.Cu, net Net-(U10-FB)
- added copper zone on F.Cu, net Net-(U17-FB)
- added copper zone on F.Cu, net Net-(U17-SW)
- added copper zone on F.Cu, net Net-(U9-FB)
- added copper zone on F.Cu, net Net-(U9-SW)
- removed copper zone on F.Cu, net +5V
- removed copper zone on F.Cu, net /Power/12V_PCBs
- removed copper zone on F.Cu, net /Power/Battery_Terminal_1_Unsensed
- removed copper zone on B.Cu, net /Power/Battery_Terminal_2
- removed copper zone on F.Cu, net GND
- removed copper zone on B.Cu, net GNDA
- removed copper zone on B.Cu, net Net-(D9-K)
Other:
- copper layers 2 -> 4

Commit message: a
Parts:
- removed the G*** at (371.5, 12.4)
- removed H1, H2, H3, H4: MountingHole, MountingHole:MountingHole_3.2mm_M3
- removed J3: OLED, BP_FTP:Display_128x64_096_I2C
- removed L4: 10u, BP_FTP:CAPC3225X270N
- added C54: 10u, BP_FTP:CAPC3225X270N, B.Cu at (172.9, 101.9)
- added C55: 100n, Capacitor_SMD:C_0402_1005Metric, B.Cu at (99.0, 68.8)
- added SW3: GPBTN, Button_Switch_THT:SW_PUSH_6mm_H5mm, F.Cu at (101.4, 71.0)
- added kibuzzard-65BEF952: G***, kibuzzard-65BEF952, F.Cu at (124.2, 126.8)
- added kibuzzard-65C0826A: G***, kibuzzard-65C0826A, F.Cu at (117.8, 135.8)
- added kibuzzard-65C082BD: G***, kibuzzard-65C082BD, F.Cu at (106.8, 149.6)
- added kibuzzard-65C082EE: G***, kibuzzard-65C082EE, F.Cu at (104.4, 149.1)
- added kibuzzard-65C08310: G***, kibuzzard-65C08310, F.Cu at (120.1, 134.8)
- added kibuzzard-65C08361: G***, kibuzzard-65C08361, F.Cu at (122.5, 134.4)
- added kibuzzard-65C0836E: G***, kibuzzard-65C0836E, F.Cu at (125.1, 134.8)
- added kibuzzard-65C08389: G***, kibuzzard-65C08389, F.Cu at (127.7, 136.0)
- C10, C11, C2, C9, JP1, R3, R4: moved to B.Cu
- D11: moved to F.Cu
- R12: value 560R -> 1k; moved to F.Cu
- R15: value 1k98 -> 3k3
- R16, R17, R18, R19, R20, R21: footprint Resistor_SMD:R_0402_1005Metric -> Resistor_SMD:R_0603_1608Metric
- R22, R23, R24: value 560R -> 1k
- R5, R6, R7: value 220R -> 400R
- R9: value 260R -> 400R
- moved D6 77.9 mm to (102.3, 100.6), turned to 90 degrees
- moved IC1 76.7 mm to (98.2, 111.4), turned to 180 degrees
- moved D7 72.0 mm to (97.8, 107.8)
- moved R12 42.2 mm to (104.3, 144.0), turned to 90 degrees
- moved D11 42.2 mm to (104.3, 140.2), turned to -90 degrees
- moved C18 31.4 mm to (97.9, 120.8), turned to 180 degrees
- moved C17 28.9 mm to (98.6, 123.2), turned to -90 degrees
- moved U5 22.4 mm to (103.8, 123.2), turned to 0 degrees
- moved C23 13.8 mm to (146.5, 135.0), turned to 0 degrees
- moved R29 12.8 mm to (131.8, 110.7)
- moved R30 12.7 mm to (131.8, 112.8), turned to 0 degrees
- moved C20 11.0 mm to (142.4, 134.9), turned to 180 degrees
- moved C50 9.97 mm to (133.5, 115.8)
- moved D21 9.27 mm to (125.7, 119.0), turned to -90 degrees
- moved TP1 8.07 mm to (118.4, 126.6)
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Connections:
- J1 pad 1: /GPIO6 -> unconnected-(J1-Pin_1-Pad1)
- J1 pad 2: /GPIO5 -> unconnected-(J1-Pin_2-Pad2)
- J1 pad 3: /GPIO4 -> unconnected-(J1-Pin_3-Pad3)
- J1 pad 4: /GPIO3 -> unconnected-(J1-Pin_4-Pad4)
- J1 pad 5: /GPIO2 -> unconnected-(J1-Pin_5-Pad5)
- U3 pad 12: /GPIO5 -> unconnected-(U3-PA6-Pad12)
- U3 pad 13: /GPIO6 -> unconnected-(U3-PA7-Pad13)
- U3 pad 14: /GPIO3 -> unconnected-(U3-PB0-Pad14)
- U3 pad 15: /GPIO4 -> unconnected-(U3-PB1-Pad15)
- U3 pad 19: /SCL -> unconnected-(U3-PA9-Pad19)
- U3 pad 20: /SDA -> unconnected-(U3-PA10-Pad20)
- U3 pad 3: /GPIO2 -> unconnected-(U3-PC15-Pad3)
Routing:
- net +5V: track 61.8 -> 430.2 mm, vias 2 -> 18
- net GND: track 105.3 -> 237.5 mm, vias 1 -> 447
- net +3V3: track 20.7 -> 143.4 mm, vias 4 -> 9
- net /Power/Battery_Terminal_1_Unsensed: track 0.00 -> 105.3 mm, vias 0 -> 1
- net /GPIO1: track 0.00 -> 70.3 mm, vias 0 -> 1
- net /DEBUG_SWCLK: track 0.00 -> 67.0 mm, vias 0 -> 1
- net /DEBUG_SWDIO: track 0.00 -> 65.6 mm, vias 0 -> 2
- net /NRST: track 2.60 -> 55.5 mm, vias 0 -> 3
- net /Power/12V_Unsensed: track 18.4 -> 70.3 mm, vias 1 -> 5
- net /Power/5V_3: track 15.2 -> 59.6 mm, vias 2 -> 3
- net /Power/5V_1: track 15.1 -> 57.8 mm, vias 2 -> 4
- net /CAN_STBY: track 0.00 -> 34.5 mm, vias 0 -> 1
- net /Battery_Curr: track 0.00 -> 33.7 mm, vias 0 -> 2
- net /CAN_TX: track 0.00 -> 30.7 mm, vias 0 -> 1
- net /Power/5V_2: track 15.3 -> 45.1 mm, vias 2 -> 3
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- added copper zone on F.Cu, net +5V
- added copper zone on In1.Cu, net +5V
- added copper zone on In2.Cu, net +5V
- added copper zone on B.Cu, net GND
- added copper zone on F.Cu, net GND
- added copper zone on In1.Cu, net GND
- added copper zone on In2.Cu, net GND
Other:
- board text removed: "MCU"

Commit message: final
Parts:
- removed kibuzzard-65C0826A: G***, kibuzzard-65C0826A
- removed kibuzzard-65C082BD: G***, kibuzzard-65C082BD
- removed kibuzzard-65C082EE: G***, kibuzzard-65C082EE
- removed kibuzzard-65C08310: G***, kibuzzard-65C08310
- removed kibuzzard-65C08361: G***, kibuzzard-65C08361
- removed kibuzzard-65C0836E: G***, kibuzzard-65C0836E
- removed kibuzzard-65C08389: G***, kibuzzard-65C08389
- added kibuzzard-65C1D3DC: G***, kibuzzard-65C1D3DC, F.Cu at (117.8, 135.8)
- added kibuzzard-65C1D3E6: G***, kibuzzard-65C1D3E6, F.Cu at (120.1, 135.6)
- added kibuzzard-65C1D3ED: G***, kibuzzard-65C1D3ED, F.Cu at (122.5, 135.6)
- added kibuzzard-65C1D405: G***, kibuzzard-65C1D405, F.Cu at (125.1, 135.6)
- added kibuzzard-65C1D40B: G***, kibuzzard-65C1D40B, F.Cu at (127.7, 135.9)
- added kibuzzard-65C1D412: G***, kibuzzard-65C1D412, F.Cu at (106.8, 149.6)
- added kibuzzard-65C1D419: G***, kibuzzard-65C1D419, F.Cu at (104.3, 148.3)
- C28, C29, C30: footprint Capacitor_SMD:C_0402_1005Metric -> Capacitor_SMD:C_0603_1608Metric
- C43: value 6u -> 6.8u
- U17: value ~ -> AP62250Z6
- moved U1 1.82 mm to (110.5, 120.6)
- moved C8 1.65 mm to (110.7, 118.3)
- moved L3 0.60 mm to (148.6, 107.8)
- moved L2 0.54 mm to (130.8, 107.7)
- moved L1 0.50 mm to (113.3, 107.8)
- moved C29 0.33 mm to (126.1, 110.3)
- moved C28 0.29 mm to (108.7, 110.3)
- moved C30 0.29 mm to (143.8, 110.2)
Routing:
- net Net-(U10-SW): track 7.29 -> 13.4 mm
- net GND: track 237.5 -> 243.4 mm, vias 447 -> 453
- net Net-(U9-SW): track 7.36 -> 12.6 mm
- net /Battery_Curr: track 33.7 -> 28.6 mm
- net Net-(U17-SW): track 7.33 -> 12.0 mm
- net /CAN_RX: track 24.5 -> 21.9 mm, vias 1 -> 2
- net /Power/Battery_Terminal_1_Unsensed: track 105.3 -> 107.4 mm
- net /XCLK: track 4.60 -> 6.48 mm
- net +3V3: track 143.4 -> 142.4 mm
- net /Power/5V_1: track 57.8 -> 58.5 mm, vias 4 -> 20
- net /NRST: track 55.5 -> 56.2 mm
- net /GPIO1: track 70.3 -> 69.8 mm
- net /Power/5V_3: track 59.6 -> 59.5 mm, vias 3 -> 12
- net /Power/outputs/5V_3: vias 0 -> 23
- net /Power/outputs/5V_2: vias 0 -> 14
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- added copper zone on B.Cu, net /Power/5V_1
- added copper zone on B.Cu, net /Power/5V_2
- added copper zone on B.Cu, net /Power/5V_3

Commit message: a
Parts:
- moved C21 2.00 mm to (162.0, 128.1)
Routing:
- net /Power/DCDC_V_{in}: track 31.2 -> 33.3 mm, vias 6 -> 26
- net Net-(JP2-B): track 17.4 -> 18.6 mm, vias 0 -> 32
- net GND: track 243.4 -> 243.3 mm, vias 453 -> 450
- added copper zone on B.Cu, net /Power/Battery_Terminal_2

Commit message: done layout v2
Parts:
- removed U17: AP62250Z6, Package_TO_SOT_SMD:SOT-563
- added U8: AP62250WU-7, Package_TO_SOT_SMD:TSOT-23-6, F.Cu at (105.7, 92.3)
- C12, C13, C14, FB1: moved to B.Cu
- R11: value 17k -> 18k
- R5, R6, R7, R9: value 400R -> 390R
- U10, U9: value AP62250Z6 -> AP62250WU-7; footprint Package_TO_SOT_SMD:SOT-563 -> Package_TO_SOT_SMD:TSOT-23-6
- moved C18 25.5 mm to (95.3, 95.4)
- moved U5 23.8 mm to (101.3, 99.5)
- moved C17 22.6 mm to (96.1, 100.8)
- moved C12 21.8 mm to (104.8, 105.1), turned to 90 degrees
- moved C13 21.8 mm to (103.3, 105.1), turned to 90 degrees
- moved C14 21.8 mm to (101.8, 105.1), turned to 90 degrees
- moved R20 19.6 mm to (137.1, 92.8), turned to -90 degrees
- moved R16 19.6 mm to (101.6, 92.9), turned to -90 degrees
- moved R18 19.5 mm to (119.4, 92.8), turned to -90 degrees
- moved IC1 18.9 mm to (95.2, 92.7), turned to -90 degrees
- moved C33 18.6 mm to (142.7, 80.2)
- moved kibuzzard-65BDE861 18.6 mm to (98.6, 113.5)
- moved C35 18.5 mm to (125.2, 80.2)
- moved kibuzzard-65BDE858 18.5 mm to (98.2, 111.5)
- moved C36 18.4 mm to (142.8, 83.5)
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Routing:
- net /Power/5V_1: track 58.5 -> 95.3 mm, vias 20 -> 29
- net /Power/5V_2: track 45.1 -> 75.5 mm, vias 17 -> 23
- net +5V: track 430.2 -> 404.4 mm, vias 18 -> 21
- net +3V3: track 142.4 -> 154.7 mm, vias 9 -> 12
- net Net-(U10-SW): track 13.4 -> 3.36 mm
- net GND: track 243.3 -> 250.9 mm, vias 450 -> 459
- net Net-(U9-SW): track 12.6 -> 8.60 mm
- net /Power/5V_3: track 59.5 -> 63.5 mm, vias 12 -> 28
- net /NRST: track 56.0 -> 59.8 mm, vias 3 -> 1
- net Net-(D1-K): track 1.96 -> 5.63 mm
- net /Power/12V_Buck: track 62.2 -> 65.4 mm
- net /DEBUG_SWCLK: track 67.0 -> 70.2 mm
- net /CAN_STBY: track 34.5 -> 37.7 mm
- net Net-(U2-CBUS0): track 18.0 -> 19.3 mm
- net Net-(U8-SW): track 12.0 -> 13.3 mm
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