File: Relay-Board_2023_Lucy_V1/Relay_Board_Lucy_V1/Relay_Board_Lucy_V1.kicad_sch (KiCad schematic)
At the start: 59 parts, among them J1 STD_PWR_HEADER, J10 STD_PWR_HEADER, J2 VP0265540000G, J3 VP0265540000G, J4 VP0265540000G, J5 VP0265540000G, Q1 SI2302A-TPMSCT-ND, U1 ACS770LCB-050U-PFF, U2 ACS770LCB-050B-PFF, U4 TSV914IPT, U5 TSV914IPT, U6 ACS770LCB-050U-PFF, U6 MAX14572

Commit message: update
Parts:
- added R1: 1.3, symbol Device:R_Small
Other:
- sheet CAP Charge Relay ports: added ~{RLY_ENBL}; removed RLY_ENBL
- sheet CAP Relay ports: added ~{RLY_ENBL}; removed RLY_ENBL
- sheet MOTOR Relay ports: added ~{RLY_ENBL}; removed RLY_ENBL
- sheet RES Relay ports: added ~{RLY_ENBL}; removed RLY_ENBL
- note added: "R_LOAD: - High wattage startup/cap charge/cap discharge resistor - Designed about Lucy's 28V stack - Power calculations are not dependent on capacitance Maximum FC current draw: P = I^2*R = (30)^2*1.3 = 1170W (never through R_load) Startup Current: (FC @ 20V) P = (15)^2*1.3 = 292.5W Capacitor charging current: (SC start @ 0V) P = 292.5W Capacitor discharge current: (SC max 28V) P = 28^2/1.3 = 603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"
Changed lines of the file:
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@@
     (stroke (width 0) (type default))
   )
-  (wire (pts (xy 147.32 144.78) (xy 153.67 144.78))
-    (stroke (width 0) (type default))
-  )
   (wire (pts (xy 241.3 165.1) (xy 241.3 162.56))
     (stroke (width 0) (type default))
@@
     (stroke (width 0) (type default))
   )
+  (polyline (pts (xy 119.38 133.35) (xy 105.41 133.35))
+    (stroke (width 0) (type default))
+  )
   (wire (pts (xy 241.3 132.08) (xy 241.3 139.7))
     (stroke (width 0) (type default))
@@
     (stroke (width 0) (type default))
   )
+  (wire (pts (xy 147.32 144.78) (xy 153.67 144.78))
+    (stroke (width 0) (type default))
+  )
   (wire (pts (xy 241.3 148.59) (xy 241.3 144.78))
     (stroke (width 0) (type default))
@@
     (stroke (width 0) (type default))
   )
+  (polyline (pts (xy 105.41 132.08) (xy 105.41 133.35))
+    (stroke (width 0) (type default))
+  )
   (wire (pts (xy 250.19 218.44) (xy 250.19 220.98))
     (stroke (width 0) (type default))
@@
     (stroke (width 0) (type default))
   )
+  (polyline (pts (xy 119.38 125.73) (xy 105.41 125.73))
+    (stroke (width 0) (type default))
+  )
   (wire (pts (xy 238.76 210.82) (xy 242.57 210.82))
     (stroke (width 0) (type default))
@@
     (stroke (width 0) (type default))
   )
+  (polyline (pts (xy 105.41 125.73) (xy 105.41 127))
+    (stroke (width 0) (type default))
+  )
   (wire (pts (xy 345.44 67.31) (xy 342.9 67.31))
     (stroke (width 0) (type default))
@@
   )
   (text "Note: The resistor polarity will change during use, thus they are labelled\npositive and negative solely for naming nets."
-    (at 69.85 140.97 0)
+    (at 66.04 149.86 0)
     (effects (font (size 1.27 1.27)) (justify left bottom))
   )
@@
     (effects (font (size 1.27 1.27)) (justify left bottom))
   )
-  (text "Notes:\n- Current at the supercapacitors could be positive or negative"
-    (at 48.26 116.84 0)
+  (text "Notes:\n- Current at the supercapacitors \n  could be positive or negative"
+    (at 21.59 80.01 0)
     (effects (font (size 1.27 1.27)) (justify left bottom))
   )
@@
     (effects (font (size 1.27 1.27)) (justify left bottom))
   )
+  (text "R_LOAD:\n - High wattage startup/cap charge/cap discharge resistor\n - Designed about Lucy's 28V stack\n - Power calculations are not dependent on capacitance\n\nMaximum FC current draw: P = I^2*R = (30)^2*1.3 = 1170W (never through R_load)\nStartup Current: (FC @ 20V) P = (15)^2*1.3 = 292.5W\nCapacitor charging current: (SC start @ 0V) P = 292.5W\nCapacitor discharge current: (SC max 28V) P = 28^2/1.3 = 603W\n\nResistor must be able to dissipate 603W continuous"
+    (at 16.51 139.7 0)
+    (effects (font (size 1.27 1.27)) (justify left bottom))
+  )
   (text "Fuel cell voltage\nsend to the fuel\ncell power board"
     (at 24.13 36.83 0)
@@
     )
   )
+  (symbol (lib_id "Device:R_Small") (at 105.41 129.54 180) (unit 1)
+    (in_bom no) (on_board no) (dnp no)
+    (property "Reference" "R1" (at 110.49 128.27 0)
+      (effects (font (size 1.27 1.27)))
+    )
+    (property "Value" "1.3" (at 110.49 130.81 0)
+      (effects (font (size 1.27 1.27)))
+    )
+    (property "Footprint" "" (at 105.41 129.54 0)
+      (effects (font (size 1.27 1.27)) hide)
+    )
+    (property "Datasheet" "" (at 105.41 129.54 0)
+      (effects (font (size 1.27 1.27)) hide)
+    )
+    (property "Part#" "" (at 105.41 129.54 0)
+      (effects (font (size 1.27 1.27)) hide)
+    )
+    (pin "1")
+    (pin "2")
+    (instances
+      (project "Relay_Board_Lucy_V1"
+        (path "/1f586fab-d165-4cda-895e-cc224a8182b4/d0430468-7d1b-42a2-a24e-658bd737b804"
+          (reference "R1") (unit 1)
+        )
+        (path "/1f586fab-d165-4cda-895e-cc224a8182b4"
+          (reference "R_LOAD") (unit 1)
+        )
+      )
+    )
+  )
   (symbol (lib_id "power:GNDA") (at 97.79 104.14 0) (unit 1)
     (in_bom yes) (on_board yes) (dnp no)
@@
       (effects (font (size 1.27 1.27)) (justify right))
     )
-    (pin "RLY_ENBL" input (at 245.11 72.39 0)
+    (pin "~{RLY_ENBL}" input (at 245.11 72.39 0)
       (effects (font (size 1.27 1.27)) (justify right))
     )
@@
       (effects (font (size 1.27 1.27)) (justify left))
     )
-    (pin "RLY_ENBL" input (at 153.67 144.78 180)
+    (pin "~{RLY_ENBL}" input (at 153.67 144.78 180)
       (effects (font (size 1.27 1.27)) (justify left))
     )
@@
       (effects (font (size 1.27 1.27)) (justify right))
     )
-    (pin "RLY_ENBL" input (at 163.83 86.36 0)
+    (pin "~{RLY_ENBL}" input (at 163.83 86.36 0)
       (effects (font (size 1.27 1.27)) (justify right))
     )
@@
       (effects (font (size 1.27 1.27)) (justify left))
     )
-    (pin "RLY_ENBL" input (at 153.67 118.11 180)
+    (pin "~{RLY_ENBL}" input (at 153.67 118.11 180)
       (effects (font (size 1.27 1.27)) (justify left))
     )
