File: Fuel-Cell-Testing-Board_2023_Lucy/purge.kicad_sch (KiCad schematic)
At the start: 1 part, among them U3 EL3H7(B)(TA)-VG

Commit message: quick update
Other:
- note added: "to do: - copy and paste purge and supply valve control - footprint for optocoupler"
Changed lines of the file:
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@@
 (kicad_sch (version 20230121) (generator eeschema)
   (paper "A4")
+  (text "to do:\n- copy and paste purge and supply valve control\n- footprint for optocoupler \n"
+    (at 76.2 120.65 0)
+    (effects (font (size 1.27 1.27) (color 255 0 9 1)) (justify left bottom))
+  )
   (symbol (lib_id "Isolator:LTV-356T") (at 134.62 97.79 0) (unit 1)
     (in_bom yes) (on_board yes) (dnp no) (fields_autoplaced)
