File: Fuel_Cell_Controller_Lucy_V1/Fuel_Cell_Controller_Prototype.kicad_pcb (KiCad board)
At the start: 0 parts

Commit message: Again too much to say
Parts:
- added C1: 100n, Capacitor_SMD:C_0603_1608Metric, F.Cu at (35.5, 108.6)
- added C10: 4u7, Capacitor_SMD:C_0603_1608Metric, F.Cu at (39.5, 113.6)
- added C11: 100n, Capacitor_SMD:C_0603_1608Metric, F.Cu at (39.5, 116.1)
- added C12: 100n, Capacitor_SMD:C_0603_1608Metric, F.Cu at (39.5, 118.6)
- added C13: 100n, Capacitor_SMD:C_0603_1608Metric, F.Cu at (39.5, 121.2)
- added C14: 100n, Capacitor_SMD:C_0603_1608Metric, F.Cu at (39.5, 123.7)
- added C15: 1u, Capacitor_SMD:C_0603_1608Metric, F.Cu at (43.5, 108.6)
- added C16: 1u, Capacitor_SMD:C_0603_1608Metric, F.Cu at (43.5, 111.1)
- added C17: 1u, Capacitor_SMD:C_0603_1608Metric, F.Cu at (43.5, 113.6)
- added C18: 1u, Capacitor_SMD:C_0603_1608Metric, F.Cu at (43.5, 116.1)
- added C19: 1u, Capacitor_SMD:C_0603_1608Metric, F.Cu at (43.5, 118.6)
- added C2: 1u_X5R, Capacitor_SMD:C_0603_1608Metric, F.Cu at (35.5, 111.1)
- added C20: 2u2, Capacitor_SMD:C_0603_1608Metric, F.Cu at (68.4, 79.8)
- added C21: 100n, Capacitor_SMD:C_0603_1608Metric, F.Cu at (68.4, 82.3)
- added C22: 2u2, Capacitor_SMD:C_0603_1608Metric, F.Cu at (68.4, 84.8)
- added C23: 100n, Capacitor_SMD:C_0603_1608Metric, F.Cu at (68.4, 87.3)
- added C24: 100n, Capacitor_SMD:C_0603_1608Metric, F.Cu at (68.4, 89.8)
- added C25: 100n, Capacitor_SMD:C_0603_1608Metric, F.Cu at (68.4, 92.3)
- added C26: 100n, Capacitor_SMD:C_0603_1608Metric, F.Cu at (68.4, 94.8)
- added C27: 100n, Capacitor_SMD:C_0603_1608Metric, F.Cu at (72.4, 79.8)
- added C28: 100n, Capacitor_SMD:C_0603_1608Metric, F.Cu at (72.4, 82.3)
- added C29: 100n, Capacitor_SMD:C_0603_1608Metric, F.Cu at (72.4, 84.8)
- added C3: 1u_X5R, Capacitor_SMD:C_0603_1608Metric, F.Cu at (35.5, 113.6)
- added C30: 4u7, Capacitor_SMD:CP_Elec_3x5.3, F.Cu at (36.8, 102.4)
- added C31: 100n, Capacitor_SMD:C_0603_1608Metric, F.Cu at (72.4, 87.3)
- added C32: 4u7, Capacitor_SMD:C_0603_1608Metric, F.Cu at (72.4, 89.8)
- added C33: 47p, Capacitor_SMD:C_0402_1005Metric, F.Cu at (79.9, 86.6)
- added C34: 47p, Capacitor_SMD:C_0402_1005Metric, F.Cu at (79.9, 88.6)
- added C35: 10n, Capacitor_SMD:C_0603_1608Metric, F.Cu at (72.4, 92.3)
- added C36: 100n, Capacitor_SMD:C_0603_1608Metric, F.Cu at (71.5, 108.6)
- added C4: 100n, Capacitor_SMD:C_0603_1608Metric, F.Cu at (35.5, 116.1)
- added C5: 100n, Capacitor_SMD:C_0603_1608Metric, F.Cu at (35.5, 118.6)
- added C6: 100n, Capacitor_SMD:C_0603_1608Metric, F.Cu at (35.5, 121.2)
- added C7: 1u_X5R, Capacitor_SMD:C_0603_1608Metric, F.Cu at (35.5, 123.7)
- added C8: 1u_X5R, Capacitor_SMD:C_0603_1608Metric, F.Cu at (39.5, 108.6)
- added C9: 100n, Capacitor_SMD:C_0603_1608Metric, F.Cu at (39.5, 111.1)
- added D1: BLUE, LED_SMD:LED_0805_2012Metric, F.Cu at (65.3, 108.9)
- added D10: LED, LED_SMD:LED_0805_2012Metric, F.Cu at (54.2, 101.5)
- added D11: SD0805S020S1R0, Diode_SMD:D_0805_2012Metric_Pad1.15x1.40mm_HandSolder, F.Cu at (83.6, 133.0)
- added D12: MMSZ5226B-7-F, FC.FTP:D_SOD_123_M, F.Cu at (76.4, 115.4)
- added D13: MMSZ5226B-7-F, FC.FTP:D_SOD_123_M, F.Cu at (76.4, 118.8)
- added D2: BLUE, LED_SMD:LED_0805_2012Metric, F.Cu at (65.3, 111.9)
- added D3: MMSZ5226B-7-F, FC.FTP:D_SOD_123_M, F.Cu at (64.0, 138.5)
- added D4: ESDALC6V1P5, FC.FTP:ESDALC6V1P5, F.Cu at (46.6, 137.4)
- added D5: GREEN, LED_SMD:LED_0805_2012Metric, F.Cu at (65.3, 114.9)
- added D6: GREEN, LED_SMD:LED_0805_2012Metric, F.Cu at (65.3, 118.0)
- added D7: SD0805S020S1R0, Diode_SMD:D_0805_2012Metric_Pad1.15x1.40mm_HandSolder, F.Cu at (71.9, 133.0)
- added D8: MMSZ5226B-7-F, FC.FTP:D_SOD_123_M, F.Cu at (77.6, 71.6)
- added D9: MMSZ5226B-7-F, FC.FTP:D_SOD_123_M, F.Cu at (77.6, 74.9)
- added FB1: 300R, Inductor_SMD:L_1206_3216Metric, F.Cu at (41.6, 137.5)
- added J1: STD_PWR_HEADER, RB_FTP:STD_PWR_HEADER, F.Cu at (40.8, 130.1)
- added J2: SWD_HEADER, Connector_PinSocket_2.54mm:PinSocket_1x04_P2.54mm_Vertical, F.Cu at (60.8, 109.7)
- added J3: DE9_Receptacle, Connector_Dsub:DSUB-9_Female_Horizontal_P2.77x2.84mm_EdgePinOffset7.70mm_Housed_MountingHolesOffset9.12mm, F.Cu at (55.5, 81.8)
- added J4: DA15_Receptacle_MountingHoles, Connector_Dsub:DSUB-15_Female_Horizontal_P2.77x2.84mm_EdgePinOffset7.70mm_Housed_MountingHolesOffset9.12mm, F.Cu at (63.8, 60.4)
- added J5: USB_B_Micro, RB_FTP:USB_Micro-B_Wuerth_629105150521, F.Cu at (199.9, 97.7)
- added JP1: SolderJumper_2_Open, Jumper:SolderJumper-2_P1.3mm_Open_RoundedPad1.0x1.5mm, F.Cu at (80.6, 80.3)
- added JP2: SolderJumper_2_Open, Jumper:SolderJumper-2_P1.3mm_Open_RoundedPad1.0x1.5mm, F.Cu at (80.6, 83.9)
- added L1: 600R/0.5A, Inductor_SMD:L_0805_2012Metric, F.Cu at (58.6, 101.4)
- added Q1: SI2302A-TPMSCT-ND, Package_TO_SOT_SMD:SOT-23-3, F.Cu at (63.7, 130.2)
- added Q2: SI2302A-TPMSCT-ND, Package_TO_SOT_SMD:SOT-23-3, F.Cu at (63.7, 134.6)
- added Q3: FMMT491ATA, Package_TO_SOT_SMD:SOT-23-3, F.Cu at (72.1, 129.3)
- added Q4: FMMT491ATA, Package_TO_SOT_SMD:SOT-23-3, F.Cu at (83.7, 129.3)
- added R1: 10k, Resistor_SMD:R_0603_1608Metric, F.Cu at (43.5, 121.2)
- added R10: 2.2M, Resistor_SMD:R_0402_1005Metric, F.Cu at (53.9, 133.1)
- added R11: 225k, Resistor_SMD:R_0402_1005Metric, F.Cu at (53.9, 135.1)
- added R12: 11.5k, Resistor_SMD:R_0402_1005Metric, F.Cu at (53.9, 137.1)
- added R13: 11.5k, Resistor_SMD:R_0402_1005Metric, F.Cu at (53.9, 139.1)
- added R14: 100k, Resistor_SMD:R_0603_1608Metric, F.Cu at (47.5, 111.1)
- added R15: 100k, Resistor_SMD:R_0603_1608Metric, F.Cu at (47.5, 113.6)
- added R16: 10k, Resistor_SMD:R_0603_1608Metric, F.Cu at (47.5, 116.1)
- added R17: 10k, Resistor_SMD:R_0603_1608Metric, F.Cu at (47.5, 118.6)
- added R18: 422, Resistor_SMD:R_0603_1608Metric, F.Cu at (76.7, 128.3)
- added R19: 249, Resistor_SMD:R_0603_1608Metric, F.Cu at (76.7, 130.8)
- added R2: 10k, Resistor_SMD:R_0603_1608Metric, F.Cu at (43.5, 123.7)
- added R20: 10k, Resistor_SMD:R_0603_1608Metric, F.Cu at (72.4, 94.8)
- added R21: 10k, Resistor_SMD:R_0603_1608Metric, F.Cu at (76.4, 79.8)
- added R22: 50, Resistor_SMD:R_0603_1608Metric, F.Cu at (76.4, 82.3)
- added R23: 10k, Resistor_SMD:R_0603_1608Metric, F.Cu at (76.4, 84.8)
- added R24: 10k, Resistor_SMD:R_0603_1608Metric, F.Cu at (76.4, 87.3)
- added R25: 270, Resistor_SMD:R_0603_1608Metric, F.Cu at (76.4, 89.8)
- added R26: 27, Resistor_SMD:R_0402_1005Metric, F.Cu at (186.4, 96.9)
- added R27: 27, Resistor_SMD:R_0402_1005Metric, F.Cu at (186.4, 98.9)
- added R28: 60, Resistor_SMD:R_0603_1608Metric, F.Cu at (76.4, 92.3)
- added R29: 60, Resistor_SMD:R_0603_1608Metric, F.Cu at (76.4, 94.8)
- added R3: 10k, Resistor_SMD:R_0603_1608Metric, F.Cu at (47.5, 108.6)
- added R30: 422, Resistor_SMD:R_0603_1608Metric, F.Cu at (88.3, 128.3)
- added R31: 249, Resistor_SMD:R_0603_1608Metric, F.Cu at (88.3, 130.8)
- added R32: 52.3k, Resistor_SMD:R_0603_1608Metric, F.Cu at (71.5, 111.1)
- added R33: 13.7k, Resistor_SMD:R_0603_1608Metric, F.Cu at (71.5, 113.6)
- added R34: 100k, Resistor_SMD:R_0603_1608Metric, F.Cu at (71.5, 116.1)
- added R35: 100k, Resistor_SMD:R_0603_1608Metric, F.Cu at (71.5, 118.6)
- added R4: 2.2M, Resistor_SMD:R_0402_1005Metric, F.Cu at (51.0, 131.1)
- added R5: 950k, Resistor_SMD:R_0402_1005Metric, F.Cu at (51.0, 133.1)
- added R6: 2.2M, Resistor_SMD:R_0402_1005Metric, F.Cu at (51.0, 135.1)
- added R7: 270k, Resistor_SMD:R_0402_1005Metric, F.Cu at (51.0, 137.1)
- added R8: 2.2M, Resistor_SMD:R_0402_1005Metric, F.Cu at (51.0, 139.1)
- added R9: 550k, Resistor_SMD:R_0402_1005Metric, F.Cu at (53.9, 131.1)
- added SW1: PTS815 SJM 250 SMTR LFS, Button_Switch_SMD:SW_SPST_PTS810, F.Cu at (52.9, 123.0)
- added SW2: PTS815 SJM 250 SMTR LFS, Button_Switch_SMD:SW_SPST_PTS810, F.Cu at (52.9, 127.8)
- added U1: LD39050PU33R, Package_DFN_QFN:DFN-6-1EP_3x3mm_P0.95mm_EP1.7x2.6mm, F.Cu at (58.7, 130.3)
- added U10: FT234XD-R, FC.FTP:SON45P300X300X80-13N, F.Cu at (183.6, 97.9)
- added U11: MCP2542FD-E/SN, Package_SO:SOIC-8_3.9x4.9mm_P1.27mm, F.Cu at (79.0, 66.7)
- added U12: USBLC6-2SC6, FC.FTP:USBLC6-2SC6, F.Cu at (191.0, 97.8)
- added U13: EL3H7(B)(TA)-VG, RB_FTP:SOIC_BTA-VG_EVS, F.Cu at (86.0, 124.8)
- added U14: MCP602-E/SN, Package_SO:SOIC-8_3.9x4.9mm_P1.27mm, F.Cu at (77.7, 110.6)
- added U2: LD39050PU33R, Package_DFN_QFN:DFN-6-1EP_3x3mm_P0.95mm_EP1.7x2.6mm, F.Cu at (58.7, 135.1)
- added U3: STM32L432KCUx, Package_DFN_QFN:QFN-32-1EP_5x5mm_P0.5mm_EP3.45x3.45mm, F.Cu at (59.9, 124.3)
- added U4: MAX14572, Package_SO:TSSOP-14-1EP_4.4x5mm_P0.65mm, F.Cu at (54.0, 110.7)
- added U5: MAX14572, Package_SO:TSSOP-14-1EP_4.4x5mm_P0.65mm, F.Cu at (54.0, 117.3)
- added U6: EL3H7(B)(TA)-VG, RB_FTP:SOIC_BTA-VG_EVS, F.Cu at (74.3, 124.8)
- added U7: MCP1501-33E/SN, Package_SO:SOIC-8_3.9x4.9mm_P1.27mm, F.Cu at (79.0, 60.3)
- added U8: AD8603, Package_TO_SOT_SMD:TSOT-23-5, F.Cu at (79.9, 98.3)
- added U9: AD8603, Package_TO_SOT_SMD:TSOT-23-5, F.Cu at (79.9, 102.8)
- added X1: OXETDLJANF-8MHZ, Crystal:Crystal_SMD_3225-4Pin_3.2x2.5mm, F.Cu at (36.1, 138.0)
Routing:
- net /IO /V_{BUS}: track 0.00 -> 11.1 mm
- net /IO /D-: track 0.00 -> 6.35 mm
- net /IO /D+: track 0.00 -> 6.24 mm, vias 0 -> 2
Other:
- copper layers 0 -> 2
