File: Fuel-Cell-Power-Board_2023_Lucy_V1/FCBoard.kicad_sch (KiCad schematic)
At the start: 92 parts, among them CON1 1X02, CON10 1X02, CON11 1X01, CON12 1X01, CON2 1X01, CON3 1X01, J1 DE9_Receptacle_MountingHoles, J2 DE9_Plug, J4 Fuel Cell, U1 STM32L432KCUx, U7 ADP2302ARDZ-5.0-R7

Commit message: Reworked schematic for more readability and changed symbols from EAGLE to KiCAD.
Parts:
- removed C41, C42, C43: EEU-FC2A221, FCC Power Board Aug 2022_OW:CAP_16_X_25, symbol FCC Power Board Aug 2022_OW-eagle-import:EEU-FC2A221
- removed C44, C45: 1uF, FCC Power Board Aug 2022_OW:C1210, symbol FCC Power Board Aug 2022_OW-eagle-import:C-EUC1210
- removed C46, C47, C66, C67: EEUFR1H221B, FCC Power Board Aug 2022_OW:CAP_PAN_10X16, symbol FCC Power Board Aug 2022_OW-eagle-import:EEUFR1H221B
- removed C48, C49, C62, C68, C69: 10uF, FCC Power Board Aug 2022_OW:C1210, symbol FCC Power Board Aug 2022_OW-eagle-import:C-EUC1210
- removed C50, C63, C70: 1uF, FCC Power Board Aug 2022_OW:C0805, symbol FCC Power Board Aug 2022_OW-eagle-import:C-EUC0805
- removed C51, C64, C65, C71: 0.1uF, FCC Power Board Aug 2022_OW:C0603, symbol FCC Power Board Aug 2022_OW-eagle-import:C-EUC0603
- removed C52, C72: 1nF/50V, FCC Power Board Aug 2022_OW:0805, symbol FCC Power Board Aug 2022_OW-eagle-import:CAPACITOR_0805
- removed C54, C73: 1uF/50V, FCC Power Board Aug 2022_OW:0805, symbol FCC Power Board Aug 2022_OW-eagle-import:CAPACITOR_0805
- removed C55, C60, C61, C74, C79, C80: 220uF, FCC Power Board Aug 2022_OW:CAPACITOR_220UF_63V, symbol FCC Power Board Aug 2022_OW-eagle-import:CAPACITOR_ELECTROLYTIC_220UF
- removed C56, C75: 0.1uF, FCC Power Board Aug 2022_OW:0805, symbol FCC Power Board Aug 2022_OW-eagle-import:CAPACITOR_0805
- removed C57, C58, C59, C76, C77, C78: 10uF, FCC Power Board Aug 2022_OW:0805, symbol FCC Power Board Aug 2022_OW-eagle-import:CAPACITOR_0805
- removed CON10: 1X02, FCC Power Board Aug 2022_OW:1X02, symbol FCC Power Board Aug 2022_OW-eagle-import:1X02
- removed CON11, CON12: 1X01, FCC Power Board Aug 2022_OW:1X01, symbol FCC Power Board Aug 2022_OW-eagle-import:1X01
- removed D1: SMBJ12A, FCC Power Board Aug 2022_OW:DO214AA, symbol FCC Power Board Aug 2022_OW-eagle-import:DIODE_TVS_UNI_DO-214AA
- removed D2: SMBJ5.0A, FCC Power Board Aug 2022_OW:DO214AA, symbol FCC Power Board Aug 2022_OW-eagle-import:DIODE_TVS_UNI_DO-214AA
- removed F1, F4: 7.5A, FCC Power Board Aug 2022_OW:FUSEHOLDER_VERTICAL, symbol FCC Power Board Aug 2022_OW-eagle-import:FUSEHOLDER_VERTICAL
- removed J4: Fuel Cell, Connector_Molex:Molex_Micro-Fit_3.0_43045-0612_2x03_P3.00mm_Vertical, symbol Connector_Generic:Conn_01x06
- removed LED8, LED9: RED, FCC Power Board Aug 2022_OW:0805_LED, symbol FCC Power Board Aug 2022_OW-eagle-import:LED_0805
- removed MOD4: i3A, FCC Power Board Aug 2022_OW:CONVERTER_I3A, symbol FCC Power Board Aug 2022_OW-eagle-import:CONVERTER_I3A
- removed R14: 560, FCC Power Board Aug 2022_OW:0805, symbol FCC Power Board Aug 2022_OW-eagle-import:RESISTOR_0805
- removed R2: 1.6k, FCC Power Board Aug 2022_OW:0805, symbol FCC Power Board Aug 2022_OW-eagle-import:RESISTOR_0805
- removed R3, R7: 10k, FCC Power Board Aug 2022_OW:TRIMPOT, symbol FCC Power Board Aug 2022_OW-eagle-import:RESISTOR_TRIMPOT
- removed R4: 2k, FCC Power Board Aug 2022_OW:0805, symbol FCC Power Board Aug 2022_OW-eagle-import:RESISTOR_0805
- removed R5: R-US_R0603, FCC Power Board Aug 2022_OW:R0603, symbol FCC Power Board Aug 2022_OW-eagle-import:R-US_R0603
- removed R6: 8.2k, FCC Power Board Aug 2022_OW:0805, symbol FCC Power Board Aug 2022_OW-eagle-import:RESISTOR_0805
- removed U$15: VS-15EWL06FNTR-M3, FCC Power Board Aug 2022_OW:TO252, symbol FCC Power Board Aug 2022_OW-eagle-import:VS-15EWL06FNTR-M3
- removed U$16: P4SMA51A, FCC Power Board Aug 2022_OW:SMA-DO214AC, symbol FCC Power Board Aug 2022_OW-eagle-import:P4SMA51A
- removed U$17: 47uH, FCC Power Board Aug 2022_OW:INDUCTOR_SMD_FOOTPRINT, symbol FCC Power Board Aug 2022_OW-eagle-import:PA4320
- removed U$26: DB2460500L, FCC Power Board Aug 2022_OW:SOD123, symbol FCC Power Board Aug 2022_OW-eagle-import:DB2460500L
- removed U$27: 744770112, FCC Power Board Aug 2022_OW:INDUCTOR_SMD_FOOTPRINT, symbol FCC Power Board Aug 2022_OW-eagle-import:744770112
- added C10: 0.1uF, symbol Device:C
- added C11, C12, C30, C31: 220uF, FCC Power Board Aug 2022_OW:CAP_PAN_10X16, symbol Device:C_Polarized
- added C13, C42: 1uF/50V, FCC Power Board Aug 2022_OW:0805, symbol Device:C
- added C14, C43: 1nF/50V, FCC Power Board Aug 2022_OW:0805, symbol Device:C
- added C15, C20, C21, C41, C45, C46: 220uF, FCC Power Board Aug 2022_OW:CAPACITOR_220UF_63V, symbol Device:C_Polarized
- added C16, C32: 0.1uF, FCC Power Board Aug 2022_OW:0805, symbol Device:C
- added C17, C18, C19, C33, C34, C44: 10uF, FCC Power Board Aug 2022_OW:0805, symbol Device:C
- added C2, C3: 220uF, FCC Power Board Aug 2022_OW:CAP_16_X_25, symbol Device:C
- added C22, C26, C29: 10uF, FCC Power Board Aug 2022_OW:C1210, symbol Device:C
- added C23, C27: 1uF, FCC Power Board Aug 2022_OW:C0805, symbol Device:C
- added C24, C25, C28: 0.1uF, FCC Power Board Aug 2022_OW:C0603, symbol Device:C
- added C4: 220uF, symbol Device:C
- added C5, C6: 1uF, FCC Power Board Aug 2022_OW:C1210, symbol Device:C
- added C7, C8: 10uF, symbol Device:C
- added C9: 1uF, symbol Device:C
- added CON7: 1X02, FCC Power Board Aug 2022_OW:1X02, symbol FCC Power Board Aug 2022_OW-eagle-import:1X02
- added CON8, CON9: 1X01, FCC Power Board Aug 2022_OW:1X01, symbol FCC Power Board Aug 2022_OW-eagle-import:1X01
- added D1: DB2460500L, FCC Power Board Aug 2022_OW:SOD123, symbol Device:D
- added D3: P4SMA51A, FCC Power Board Aug 2022_OW:SMA-DO214AC, symbol Device:D_Zener
- added D4: VS-15EWL06FNTR-M3, FCC Power Board Aug 2022_OW:TO252, symbol Device:D
- added D5, D7: SMBJ12A, FCC Power Board Aug 2022_OW:DO214AA, symbol Device:D_Zener
- added F2, F3: 7.5A, FCC Power Board Aug 2022_OW:FUSEHOLDER_VERTICAL, symbol FCC Power Board Aug 2022_OW-eagle-import:FUSEHOLDER_VERTICAL
- added L1: 47uH, FCC Power Board Aug 2022_OW:INDUCTOR_SMD_FOOTPRINT, symbol Device:L
- added L2: 12uH, FCC Power Board Aug 2022_OW:INDUCTOR_SMD_FOOTPRINT, symbol Device:L
- added LED1, LED3: RED, FCC Power Board Aug 2022_OW:0805_LED, symbol Device:LED
- added MOD1: i3A, FCC Power Board Aug 2022_OW:CONVERTER_I3A, symbol FCC Power Board Aug 2022_OW-eagle-import:CONVERTER_I3A
- added R1: 1.6k, FCC Power Board Aug 2022_OW:0805, symbol Device:R
- added R10: 560, FCC Power Board Aug 2022_OW:0805, symbol Device:R
- added R2: R, FCC Power Board Aug 2022_OW:R0603, symbol Device:R
- added R8: 2k, FCC Power Board Aug 2022_OW:0805, symbol Device:R
- added R9: 8.2k, FCC Power Board Aug 2022_OW:0805, symbol Device:R
- added RV1, RV2: 10k, FCC Power Board Aug 2022_OW:TRIMPOT, symbol Device:R_Potentiometer_US
Connections:
- net +12V: now also U7.2 (VIN), U7.3 (EN), C22.1, C23.1, C24.1, D5.1 (K), F2.3 (2), F2.4 (2), LED1.2 (A), R2.1
- net 12V: no longer U7.2 (VIN), U7.3 (EN)
- net 12V_PRE_FUSE: now also C16.1, C17.1, C18.1, C19.1, C20.1, C21.1, F2.1, F2.2 (1)
- net 12V_REG: now also MOD3.1 (VIN), C13.1, C14.1, C15.1
- net 5V_PRE_FUSE: now also C32.1, C33.1, C34.1, C44.1, C45.1, C46.1, CON8.1, F3.1, F3.2 (1), MOD1.7 (SENSE+), MOD1.8 (VOUT)
- net 5V_REG: now also C41.1, C42.1, C43.1, MOD1.1 (VIN)
- net FEEDBACK: now also C26.1, C27.1, C28.1, C29.1, C30.1, C31.1, L2.2
- net GND: now also SV3.3, SV4.3, C10.2, C11.2, C12.2, C13.2, C14.2, C15.2, C16.2, C17.2, C18.2, C19.2, C20.2, C21.2, C26.2, C27.2, C28.2, C29.2, C30.2, C31.2, C32.2, C33.2, C34.2, C41.2, C42.2, C43.2, C44.2, C45.2, C46.2, C7.2, C8.2, C9.2, CON7.1, CON9.1, D1.2 (A), D5.2 (A), D7.2 (A), MOD1.3 (GND), MOD1.4 (GND), R10.2, R8.2, RV1.1, RV2.1; no longer SV3.1, SV4.1
- net GND_IN: now also SV3.1, SV4.1, C2.2, C3.2, C4.2, C5.2, C6.2, D3.2 (A), D4.2 (A); no longer SV3.3, SV4.3
- net VIN: now also C2.1, D3.1 (K), D4.1 (K), L1.1; no longer MOD3.1 (VIN)
- net at U7.1 (BST): now also C25.2
- net at U7.8 (SW): now also C25.1, D1.1 (K), L2.1
- net at JP2.2, U$19.P$1 (VIN): now also C3.1, C4.1, C5.1, C6.1, L1.2
- net at U$19.P$6 (VOUT), U$22.OUT: now also C10.1, C11.1, C12.1, C7.1, C8.1, C9.1
- net at U7.4 (PGOOD): now also R2.2
- net at MOD3.6 (TRIM): now also R1.1
- new net: C22.2, C23.2, C24.2
- new net: LED3.1 (K), R10.1
- new net: MOD1.6 (TRIM), R9.1
- new net: R9.2, RV2.2, RV2.3
- new net: LED1.1 (K), R8.1
- new net: R1.2, RV1.2, RV1.3
- new net: CON7.2, MOD1.2 (ON/OFF)
- new net +5V: D7.1 (K), F3.3 (2), F3.4 (2), LED3.2 (A)
Other:
- note removed: "12uH"
- note removed: "Input Connector"
- note removed: "Output Should be clean 12V"
- note removed: "Protection System"
- note removed: "Reference Ground"
- moved on the sheet: C1, CON1, CON2, CON3, J1, J2, JP2, LED10, LED11, LED12, LED13, LED14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

Commit message: Making changes
Parts:
- removed C1: 10uF, symbol Device:C
- removed C22, C26, C29: 10uF, FCC Power Board Aug 2022_OW:C1210, symbol Device:C
- removed C23, C27: 1uF, FCC Power Board Aug 2022_OW:C0805, symbol Device:C
- removed C24, C25, C28: 0.1uF, FCC Power Board Aug 2022_OW:C0603, symbol Device:C
- removed C30, C31: 220uF, FCC Power Board Aug 2022_OW:CAP_PAN_10X16, symbol Device:C_Polarized
- removed C32: 0.1uF, FCC Power Board Aug 2022_OW:0805, symbol Device:C
- removed C33, C34, C44: 10uF, FCC Power Board Aug 2022_OW:0805, symbol Device:C
- removed C41, C45, C46: 220uF, FCC Power Board Aug 2022_OW:CAPACITOR_220UF_63V, symbol Device:C_Polarized
- removed C42: 1uF/50V, FCC Power Board Aug 2022_OW:0805, symbol Device:C
- removed C43: 1nF/50V, FCC Power Board Aug 2022_OW:0805, symbol Device:C
- removed C53: EEUFR1H221B, FCC Power Board Aug 2022_OW:CAP_PAN_10X16, symbol FCC Power Board Aug 2022_OW-eagle-import:EEUFR1H221B
- removed CON2, CON3, CON8, CON9: 1X01, FCC Power Board Aug 2022_OW:1X01, symbol FCC Power Board Aug 2022_OW-eagle-import:1X01
- removed CON7: 1X02, FCC Power Board Aug 2022_OW:1X02, symbol FCC Power Board Aug 2022_OW-eagle-import:1X02
- removed D1: DB2460500L, FCC Power Board Aug 2022_OW:SOD123, symbol Device:D
- removed D7: SMBJ12A, FCC Power Board Aug 2022_OW:DO214AA, symbol Device:D_Zener
- removed E4, E5, E6: 5555140-6, FCC Power Board Aug 2022_OW:1734723-1_RJ11, symbol FCC Power Board Aug 2022_OW-eagle-import:5555140-6
- removed F3: 7.5A, FCC Power Board Aug 2022_OW:FUSEHOLDER_VERTICAL, symbol FCC Power Board Aug 2022_OW-eagle-import:FUSEHOLDER_VERTICAL
- removed J1: DE9_Receptacle_MountingHoles, symbol Connector:DE9_Receptacle_MountingHoles
- removed J2: DE9_Plug, symbol Connector:DE9_Plug
- removed JP2: JP1E, FCC Power Board Aug 2022_OW:JP1, symbol FCC Power Board Aug 2022_OW-eagle-import:JP1E
- removed L2: 12uH, FCC Power Board Aug 2022_OW:INDUCTOR_SMD_FOOTPRINT, symbol Device:L
- removed LED10, LED13, LED14: LEDCHIPLED_0805, FCC Power Board Aug 2022_OW:CHIPLED_0805, symbol FCC Power Board Aug 2022_OW-eagle-import:LEDCHIPLED_0805
- removed LED11: Amber 1.9V, FCC Power Board Aug 2022_OW:CHIPLED_0805, symbol FCC Power Board Aug 2022_OW-eagle-import:LEDCHIPLED_0805
- removed LED12: Blue 3.3V, FCC Power Board Aug 2022_OW:CHIPLED_0805, symbol FCC Power Board Aug 2022_OW-eagle-import:LEDCHIPLED_0805
- removed LED3: RED, FCC Power Board Aug 2022_OW:0805_LED, symbol Device:LED
- removed MOD1: i3A, FCC Power Board Aug 2022_OW:CONVERTER_I3A, symbol FCC Power Board Aug 2022_OW-eagle-import:CONVERTER_I3A
- removed R10: 560, FCC Power Board Aug 2022_OW:0805, symbol Device:R
- removed R2: R, FCC Power Board Aug 2022_OW:R0603, symbol Device:R
- removed R9: 8.2k, FCC Power Board Aug 2022_OW:0805, symbol Device:R
- removed RV2: 10k, FCC Power Board Aug 2022_OW:TRIMPOT, symbol Device:R_Potentiometer_US
- removed SV3, SV4: MA03-1, FCC Power Board Aug 2022_OW:MA03-1, symbol FCC Power Board Aug 2022_OW-eagle-import:MA03-1
- removed U$19: RPA60-2412SFW_P, FCC Power Board Aug 2022_OW:RPA60-2412SFW_P, symbol FCC Power Board Aug 2022_OW-eagle-import:RPA60-2412SFW_P
- removed U$23, U$24: 2X1-CONN, FCC Power Board Aug 2022_OW:2X1-MATE-N-LOCK, symbol FCC Power Board Aug 2022_OW-eagle-import:2X1-CONN
- removed U$25: M3_SCREW_TERMINAL, FCC Power Board Aug 2022_OW:M3_SCREW_TERMINAL, symbol FCC Power Board Aug 2022_OW-eagle-import:M3_SCREW_TERMINAL
- removed U$28: SHELL2013_FUSEMINI-BLADE, FCC Power Board Aug 2022_OW:SHELL2013_MINI-BLADE-FUSE, symbol FCC Power Board Aug 2022_OW-eagle-import:SHELL2013_FUSEMINI-BLADE
- removed U$29, U$30: NSI45020AT1G, FCC Power Board Aug 2022_OW:SOD123, symbol FCC Power Board Aug 2022_OW-eagle-import:NSI45020AT1G
- removed U1: STM32L432KCUx, Package_DFN_QFN:QFN-32-1EP_5x5mm_P0.5mm_EP3.45x3.45mm, symbol MCU_ST_STM32L4:STM32L432KCUx
- removed U7: ADP2302ARDZ-5.0-R7, FCC Power Board Aug 2022_OW:RD_8_1, symbol FCC Power Board Aug 2022_OW-eagle-import:ADP2302ARDZ-5.0-R7
- added C1, C11, C20 (x4), C37, C9: 100n, Capacitor_SMD:C_0603_1608Metric, symbol Device:C_Small
- added C12, C38: 4u7, Capacitor_SMD:C_0603_1608Metric, symbol Device:C_Small
- added C19, C20, C21: 100n, Capacitor_SMD:C_0402_1005Metric, symbol Device:C_Small
- added C20 (x2): 47p, Capacitor_SMD:C_0402_1005Metric, symbol Device:C_Small
- added C22: 1u, Capacitor_SMD:C_0603_1608Metric, symbol Device:C_Small
- added C52: 4u7, Capacitor_SMD:CP_Elec_3x5.3, symbol Device:C_Polarized_Small
- added D2: MMSZ5226B-7-F, FC.FTP:D_SOD_123_M, symbol FCC_Parts:MMSZ5226B-7-F
- added D6: ESDALC6V1P5, FC.FTP:ESDALC6V1P5, symbol FCC_Parts:ESDALC6V1P5
- added D8: PINK, LED_SMD:LED_0805_2012Metric, symbol Device:LED
- added FB1: 300R, Inductor_SMD:L_0603_1608Metric, symbol Device:FerriteBead_Small
- added J3: STD_PWR_HEADER, RB_FTP:STD_PWR_HEADER, symbol RB_Parts:STD_PWR_HEADER
- added J5: DE9_Receptacle, Connector_Dsub:DSUB-9_Female_Horizontal_P2.77x2.84mm_EdgePinOffset7.70mm_Housed_MountingHolesOffset9.12mm, symbol Connector:DE9_Receptacle_MountingHoles
- added J6: SWD_HEADER, Connector_PinSocket_2.54mm:PinSocket_1x04_P2.54mm_Vertical, symbol Connector_Generic:Conn_01x04
- added J7: DA15_Receptacle_MountingHoles, Connector_Dsub:DSUB-15_Female_Horizontal_P2.77x2.84mm_EdgePinOffset7.70mm_Housed_MountingHolesOffset9.12mm, symbol Connector:DA15_Receptacle_MountingHoles
- added J7: USB_B_Micro, RB_FTP:USB_Micro-B_Wuerth_629105150521, symbol Connector:USB_B_Micro
- added JP1, JP3: SolderJumper_2_Open, Jumper:SolderJumper-2_P1.3mm_Open_RoundedPad1.0x1.5mm, symbol Jumper:SolderJumper_2_Open
- added L3: 600R/0.5A, Inductor_SMD:L_0805_2012Metric, symbol Device:L_Iron
- added NT1: NetTie_2, NetTie:NetTie-2_SMD_Pad0.5mm, symbol Device:NetTie_2
- added PS1: RPA60-2412SFW_P, FCPB_FTP:CONV_RPA60-2412SFW_P, symbol FCPB_PARTS:RPA60-2412SFW_P
- added R11, R7: 26.7, Resistor_SMD:R_0402_1005Metric, symbol Device:R_Small
- added R25: 10k, Resistor_SMD:R_0603_1608Metric, symbol Device:R_Small
- added R3, R4: 60.4, Resistor_SMD:R_0603_1608Metric, symbol Device:R_Small
- added R6: 30.1, Resistor_SMD:R_0603_1608Metric, symbol Device:R_Small
- added SW1, SW2: PTS815 SJM 250 SMTR LFS, Button_Switch_SMD:SW_SPST_PTS810, symbol Switch:SW_Push_45deg
- added TP1: MCO, TestPoint:TestPoint_Pad_D1.0mm, symbol Connector:TestPoint_Small
- added U2: STM32L432KCUx, Package_DFN_QFN:QFN-32-1EP_5x5mm_P0.5mm_EP3.45x3.45mm, symbol MCU_ST_STM32L4:STM32L432KCUx
- added U3: FT234XD-R, FC.FTP:SON45P300X300X80-13N, symbol FCC_Parts:FT234XD-R
- added U4: USBLC6-2SC6, FC.FTP:USBLC6-2SC6, symbol FCC_Parts:USBLC6-2SC6
- added U9: MCP2542FD-E/SN, Package_SO:SOIC-8_3.9x4.9mm_P1.27mm, symbol FCC_PARTS:MCP2542FD
- added X1: OXETDLJANF-8MHZ, Crystal:Crystal_SMD_3225-4Pin_3.2x2.5mm, symbol RB_PARTS:OXETDLJANF-8MHZ
Connections:
- net FC_IN is gone; now on net VIN: U$14.OUT
- net +12V: now also J7.1, J7.10 (P10), J7.2, J7.9 (P9)
- net +3V3: now also C1.1, U9.5 (VIO)
- net +5V: now also C37.2, JP3.2 (B), U9.3 (VDD)
- net CAN_H: now also J5.7, R3.2, U9.7 (CANH)
- net CAN_L: now also J5.2, R4.2, U9.6 (CANL)
- net GND: now also J5.6, PS1.5 (-VOUT)
- net V+: now also J5.9
- net V-: now also J5.3
- net VIN: no longer U$14.IN
- net at C10.1, C11.1, C12.1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: now also PS1.6 (+VOUT)
- net at C3.1, C4.1, C5.1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: now also PS1.1 (+VIN)
- net GND_IN renamed FC-
- net FC-: now also J3.1 (12V), J3.2 (GND), J3.3 (5V), PS1.2 (-VIN)
- new net: D8.1 (K), R6.1
- new net: R6.2, U3.6 (CBUS0)
- new net: C20.1, C52.1, JP3.1 (A), L3.1, U3.4 (VCC)
- new net: C38.2, R3.1, R4.1
- new net: R7.1, U3.1 (USBDM)
- new net: C21.1, C22.1, FB1.2, U2.5 (VDDA)
- new net: R11.1, U3.12 (USBDP)
- new net BOOT0: R25.1, SW2.2, U2.31 (PH3)
- new net CAN_{RXD}: U2.21 (PA11), U9.4 (RXD)
- new net CAN_{STBY}: U2.25 (PA15), U9.8 (STBY)
- new net CAN_{TXD}: U2.22 (PA12), U9.1 (TXD)
- new net D+: J7.3 (D+), U4.4
- new net D-: J7.2 (D-), U4.6
- new net DM: C20.1, R7.2, U4.1
- new net DP: C20.1, R11.2, U4.3
- new net FC+: J3.4 (12V), J3.5 (GND), J3.6 (5V), U$14.IN
- new net FTDI_{~{RST}}: C20.2, U2.15 (PB1), U3.2 (~{RESET}#)
- new net GNDA: C1.2, C11.2, C12.2, C19.2, C20.1, C20.2, C20.2, C20.2, C20.2, C20.2, C20.2, C21.2, C22.2, C37.1, C38.1, C52.2, C9.2, D2.2, D6.2, J5.0 (PAD), J6.3 (Pin_3), J7.0 (PAD), J7.14 (P14), J7.15 (P15), J7.6 (Shield), J7.7, J7.8, JP1.1 (A), NT1.1, SW1.1, SW2.1, U2.16 (VSS), U2.32 (VSS), U2.33 (VSS), U3.13 (GND__1), U3.5 (GND), U9.2 (VSS), X1.2 (GND)
- new net GND_{1}: J7.5 (GND), NT1.2, U4.2
- new net MCU_3V3: C12.1, C19.1, C20.1, C9.1, D2.1, FB1.1, J6.1 (Pin_1), R25.2, U2.1 (VDD), U2.17 (VDD), X1.1 (Tri-State), X1.4 (VDD)
- new net PA0: U2.6 (PA0), X1.3 (OUT)
- new net PA1: U2.7 (PA1)
- new net PA10: U2.20 (PA10), U3.7 (TXD)
- new net PA13: D6.3, J6.4 (Pin_4), U2.23 (PA13)
- new net PA14: D6.1, J6.2 (Pin_2), U2.24 (PA14)
- new net PA2: U2.8 (PA2)
- new net PA3: U2.9 (PA3)
- new net PA4: U2.10 (PA4)
- new net PA5: U2.11 (PA5)
- new net PA6: U2.12 (PA6)
- new net PA7: U2.13 (PA7)
- new net PA8: TP1.1, U2.18 (PA8)
- new net PA9: U2.19 (PA9), U3.10 (RXD)
- new net PB0: U2.14 (PB0)
- new net PB3: U2.26 (PB3), U3.11 (CTS#)
- new net PB4: U2.27 (PB4), U3.8 (RTS#)
- new net PB5: U2.28 (PB5)
- new net PB6: U2.29 (PB6)
- new net PB7: U2.30 (PB7)
- new net PC14: U2.2 (PC14)
- new net PC15: U2.3 (PC15)
- new net PWM_{1}: J7.3
- new net PWM_{2}: J7.11 (P111)
- new net SHIELD: J5.5, JP1.2 (B)
- new net TACH_{1}: J7.4
- new net TACH_{2}: J7.12 (P12)
- new net TACH_{3}: J7.5
- new net TACH_{4}: J7.13 (P13)
- new net VCCIO: C20.1, D8.2 (A), U3.3 (3V3OUT), U3.9 (VCCIO)
- new net V_{BUS}: C20.1, J7.1 (VBUS), L3.2, U4.5
- new net ~{RST}: C11.1, SW1.2, U2.4 (NRST)
- no-connect marks 7 -> 9
Other:
- note added: "BOOT0 and ~{RST}"
- note added: "CANBus Transciever and Receptacle"
- note added: "CLOCK"
- note added: "FB1: - 300 Ohms @ 100MHz - DCR 300 mOhms"
- note added: "FTDI - TTL to USB"
- note added: "FTDI VCP DRIVERS"
- note added: "Power in from FC"
- note added: "Run V_{BUS} under the IC close to GND pin for optimal protection"
- note added: "Serial Wire Debug"
- note added: "Shield should only be connected at one point. This will likely be on one of the power boards. Do not attach V+ or V- or GND to anything since we are supplying power via other means between borns and we need to avoid ground loops."
- note added: "Should be 5MHz with proper code config"
- note added: "V_{F} = 3.0V"
- note removed: "20mA Current Source"
- note removed: "2A FUSE"
- note removed: "5V DC-DC"
- note removed: "5V DC-DC Converter"
- note removed: "5V Regulator"
- note removed: "CAN Connection"
- note removed: "FAN"
- note removed: "LED Test"
- note removed: "Note: 1) Vout can be increased by adjusting the trimpot clockwise. 2) The resistor in series with the trimpot limits the output voltage. 3) D8 is a TVS diode to protect devices on the 5V rail."
- note removed: "Output Connectors"
- note removed: "PA8 is TIM1_CH1 which has integrated PWM capability"
- note removed: "To isolate? Or not to isolate? That is the question"
