File: Fuel-Cell-Power-Board-WIP/diffAmp.kicad_sch (KiCad schematic)
At the start: 5 parts, among them U10 TSV912IDT

Commit message: some small changes
Parts:
- removed R34, R36, R37, R38: R, symbol Device:R
- removed U10: TSV912IDT, symbol Amplifier_Operational:TSV912IDT
Changed lines of the file:
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@@
 (kicad_sch (version 20230121) (generator eeschema)
   (paper "A4")
-  (junction (at 119.38 110.49) (diameter 0) (color 0 0 0 0)
-  )
-  (junction (at 148.59 100.33) (diameter 0) (color 0 0 0 0)
-  )
-  (junction (at 119.38 92.71) (diameter 0) (color 0 0 0 0)
-  )
-  (wire (pts (xy 127 73.66) (xy 127 68.58))
-    (stroke (width 0) (type default))
-  )
-  (wire (pts (xy 95.25 92.71) (xy 104.14 92.71))
-    (stroke (width 0) (type default))
-  )
-  (wire (pts (xy 148.59 121.92) (xy 148.59 100.33))
-    (stroke (width 0) (type default))
-  )
-  (wire (pts (xy 119.38 92.71) (xy 127 92.71))
-    (stroke (width 0) (type default))
-  )
-  (wire (pts (xy 119.38 92.71) (xy 119.38 97.79))
-    (stroke (width 0) (type default))
-  )
-  (wire (pts (xy 148.59 100.33) (xy 161.29 100.33))
-    (stroke (width 0) (type default))
-  )
-  (wire (pts (xy 127 68.58) (xy 138.43 68.58))
-    (stroke (width 0) (type default))
-  )
-  (wire (pts (xy 127 92.71) (xy 127 81.28))
-    (stroke (width 0) (type default))
-  )
-  (wire (pts (xy 95.25 110.49) (xy 104.14 110.49))
-    (stroke (width 0) (type default))
-  )
-  (wire (pts (xy 138.43 68.58) (xy 138.43 71.12))
-    (stroke (width 0) (type default))
-  )
-  (wire (pts (xy 111.76 110.49) (xy 119.38 110.49))
-    (stroke (width 0) (type default))
-  )
-  (wire (pts (xy 119.38 97.79) (xy 127 97.79))
-    (stroke (width 0) (type default))
-  )
-  (wire (pts (xy 119.38 121.92) (xy 119.38 110.49))
-    (stroke (width 0) (type default))
-  )
-  (wire (pts (xy 148.59 100.33) (xy 142.24 100.33))
-    (stroke (width 0) (type default))
-  )
-  (wire (pts (xy 125.73 121.92) (xy 119.38 121.92))
-    (stroke (width 0) (type default))
-  )
-  (wire (pts (xy 119.38 102.87) (xy 127 102.87))
-    (stroke (width 0) (type default))
-  )
-  (wire (pts (xy 119.38 110.49) (xy 119.38 102.87))
-    (stroke (width 0) (type default))
-  )
-  (wire (pts (xy 133.35 121.92) (xy 148.59 121.92))
-    (stroke (width 0) (type default))
-  )
-  (wire (pts (xy 111.76 92.71) (xy 119.38 92.71))
-    (stroke (width 0) (type default))
-  )
-  (label "CurrToVolt" (at 161.29 100.33 180) (fields_autoplaced)
-    (effects (font (size 1.27 1.27)) (justify right bottom))
-  )
-  (hierarchical_label "V_{HI}" (shape input) (at 95.25 92.71 180) (fields_autoplaced)
-    (effects (font (size 1.27 1.27)) (justify right))
-  )
-  (hierarchical_label "V_{LO}" (shape input) (at 95.25 110.49 180) (fields_autoplaced)
-    (effects (font (size 1.27 1.27)) (justify right))
-  )
-  (symbol (lib_id "Device:R") (at 127 77.47 180) (unit 1)
-    (in_bom yes) (on_board yes) (dnp no) (fields_autoplaced)
-    (property "Reference" "R38" (at 129.54 76.835 0)
-      (effects (font (size 1.27 1.27)) (justify right))
-    )
-    (property "Value" "R" (at 129.54 79.375 0)
-      (effects (font (size 1.27 1.27)) (justify right))
-    )
-    (property "Footprint" "" (at 128.778 77.47 90)
-      (effects (font (size 1.27 1.27)) hide)
-    )
-    (property "Datasheet" "~" (at 127 77.47 0)
-      (effects (font (size 1.27 1.27)) hide)
-    )
-    (pin "1")
-    (pin "2")
-    (instances
-      (project "FCBoard"
-        (path "/7aefa7f6-8562-49e0-9457-229f56bba97d/483ed529-0998-43e9-b404-75e6d31b159c"
-          (reference "R38") (unit 1)
-        )
-      )
-    )
-  )
-  (symbol (lib_id "Amplifier_Operational:TSV912IDT") (at 134.62 100.33 0) (unit 1)
-    (in_bom yes) (on_board yes) (dnp no)
-    (property "Reference" "U10" (at 134.62 91.44 0)
-      (effects (font (size 1.27 1.27)))
-    )
-    (property "Value" "TSV912IDT" (at 134.62 93.98 0)
-      (effects (font (size 1.27 1.27)))
-    )
-    (property "Footprint" "" (at 134.62 100.33 0)
-      (effects (font (size 1.27 1.27)) hide)
-    )
-    (property "Datasheet" "www.st.com/resource/en/datasheet/tsv911.pdf" (at 134.62 100.33 0)
-      (effects (font (size 1.27 1.27)) hide)
-    )
-    (pin "1")
-    (pin "2")
-    (pin "3")
-    (pin "5")
-    (pin "6")
-    (pin "7")
-    (pin "4")
-    (pin "8")
-    (instances
-      (project "FCBoard"
-        (path "/7aefa7f6-8562-49e0-9457-229f56bba97d/5be85d44-b1c4-47a6-b267-9e3b1f3657e3"
-          (reference "U10") (unit 1)
-        )
-        (path "/7aefa7f6-8562-49e0-9457-229f56bba97d/59d9b0c4-d4f4-4be3-8a94-d2e2577f3ec5"
-          (reference "U12") (unit 1)
-        )
-        (path "/7aefa7f6-8562-49e0-9457-229f56bba97d/fe3123b0-dc9c-4c12-a57a-891411bdcffa"
-          (reference "U7") (unit 1)
-        )
-        (path "/7aefa7f6-8562-49e0-9457-229f56bba97d/483ed529-0998-43e9-b404-75e6d31b159c"
-          (reference "U12") (unit 1)
-        )
-      )
-    )
-  )
-  (symbol (lib_id "Device:R") (at 107.95 110.49 90) (unit 1)
-    (in_bom yes) (on_board yes) (dnp no) (fields_autoplaced)
-    (property "Reference" "R36" (at 107.95 105.41 90)
-      (effects (font (size 1.27 1.27)))
-    )
-    (property "Value" "R" (at 107.95 107.95 90)
-      (effects (font (size 1.27 1.27)))
-    )
-    (property "Footprint" "" (at 107.95 112.268 90)
-      (effects (font (size 1.27 1.27)) hide)
-    )
-    (property "Datasheet" "~" (at 107.95 110.49 0)
-      (effects (font (size 1.27 1.27)) hide)
-    )
-    (pin "1")
-    (pin "2")
-    (instances
-      (project "FCBoard"
-        (path "/7aefa7f6-8562-49e0-9457-229f56bba97d/483ed529-0998-43e9-b404-75e6d31b159c"
-          (reference "R36") (unit 1)
-        )
-      )
-    )
-  )
-  (symbol (lib_id "Device:R") (at 107.95 92.71 90) (unit 1)
-    (in_bom yes) (on_board yes) (dnp no) (fields_autoplaced)
-    (property "Reference" "R34" (at 107.95 87.63 90)
-      (effects (font (size 1.27 1.27)))
-    )
-    (property "Value" "R" (at 107.95 90.17 90)
-      (effects (font (size 1.27 1.27)))
-    )
-    (property "Footprint" "" (at 107.95 94.488 90)
-      (effects (font (size 1.27 1.27)) hide)
-    )
-    (property "Datasheet" "~" (at 107.95 92.71 0)
-      (effects (font (size 1.27 1.27)) hide)
-    )
-    (pin "1")
-    (pin "2")
-    (instances
-      (project "FCBoard"
-        (path "/7aefa7f6-8562-49e0-9457-229f56bba97d/483ed529-0998-43e9-b404-75e6d31b159c"
-          (reference "R34") (unit 1)
-        )
-      )
-    )
-  )
-  (symbol (lib_id "power:GND") (at 138.43 71.12 0) (unit 1)
-    (in_bom yes) (on_board yes) (dnp no) (fields_autoplaced)
-    (property "Reference" "#PWR01" (at 138.43 77.47 0)
-      (effects (font (size 1.27 1.27)) hide)
-    )
-    (property "Value" "GND" (at 138.43 76.2 0)
-      (effects (font (size 1.27 1.27)))
-    )
-    (property "Footprint" "" (at 138.43 71.12 0)
-      (effects (font (size 1.27 1.27)) hide)
-    )
-    (property "Datasheet" "" (at 138.43 71.12 0)
-      (effects (font (size 1.27 1.27)) hide)
-    )
-    (pin "1")
-    (instances
-      (project "FCBoard"
-        (path "/7aefa7f6-8562-49e0-9457-229f56bba97d/483ed529-0998-43e9-b404-75e6d31b159c"
-          (reference "#PWR01") (unit 1)
-        )
-      )
-    )
-  )
-  (symbol (lib_id "Device:R") (at 129.54 121.92 90) (unit 1)
-    (in_bom yes) (on_board yes) (dnp no) (fields_autoplaced)
-    (property "Reference" "R37" (at 129.54 116.84 90)
-      (effects (font (size 1.27 1.27)))
-    )
-    (property "Value" "R" (at 129.54 119.38 90)
-      (effects (font (size 1.27 1.27)))
-    )
-    (property "Footprint" "" (at 129.54 123.698 90)
-      (effects (font (size 1.27 1.27)) hide)
-    )
-    (property "Datasheet" "~" (at 129.54 121.92 0)
-      (effects (font (size 1.27 1.27)) hide)
-    )
-    (pin "1")
-    (pin "2")
-    (instances
-      (project "FCBoard"
-        (path "/7aefa7f6-8562-49e0-9457-229f56bba97d/483ed529-0998-43e9-b404-75e6d31b159c"
-          (reference "R37") (unit 1)
-        )
-      )
-    )
-  )
 )

Commit message: All values calculated, next step is to pick parts.
Parts:
- added C45: C, symbol Device:C
- added R20: 1k, symbol Device:R
- added U12: INA190A1IDCKR, DCK0006A-IPC_A, symbol FCPB_Parts:INA190A1IDCKR
- added U18: INA169, Package_TO_SOT_SMD:SOT-23-5, symbol Amplifier_Current:INA169
Connections:
- new net FC_5V_B2: C45.1, U12.3 (VS)
- new net FC_Meas: R20.1, U12.6 (OUT), U18.1
- new net GND: C45.2, R20.2, U12.1 (REF), U12.2 (GND), U18.2 (GND)
- new net V_{HI}: U12.4 (IN+), U18.3 (+), U18.5 (V+)
- new net V_{LO}: U12.5 (IN-), U18.4 (-)
Other:
- note added: "The sense resistor must be 1k or less for best performance. We will go with R_sense = 1k meaning we run 28V/1k=28mA max. R_sense should be rated for AT LEAST 784mW"
- note added: "V_out = (I_load*R_sense*GAIN) The GAIN is 25V/V The maximum voltage output is thus 28mA * 1k * 25V/V = 700V????"
